File: Connectors.sch (KiCad schematic (older format))
At the start: 12 parts, among them J10 JST-PH, J11 USB_C_Receptacle_USB2.0, J9 Micro_SD_Card_Det, U8 USBLC6-2SC6

Commit message: Fix BOM ref
Parts:
- R71: MPN (none) -> RC0603JR-0710KL; Mfr. (none) -> Yageo
- U8: MPN (none) -> USBLC6-2SC6Y; Mfr. (none) -> STMicroelectronics
Changed lines of the file:
@@
 $Descr A4 11693 8268
 encoding utf-8
-Sheet 14 15
+Sheet 14 17
 Title "Kleinvoet"
 Date "2020-06-11"
@@
 F 2 "Package_TO_SOT_SMD:SOT-23-6" H 3800 4900 50  0001 C CNN
 F 3 "https://www.st.com/resource/en/datasheet/usblc6-2.pdf" H 4000 5750 50  0001 C CNN
+F 4 "USBLC6-2SC6Y" H 3800 5400 50  0001 C CNN "MPN"
+F 5 "STMicroelectronics" H 3800 5400 50  0001 C CNN "Mfr."
 	1    3800 5400
 	1    0    0    -1
@@
 F 2 "Resistor_SMD:R_0603_1608Metric_Pad1.05x0.95mm_HandSolder" H 4350 2650 50  0001 C CNN
 F 3 "~" H 4350 2650 50  0001 C CNN
+F 4 "RC0603JR-0710KL" H 4350 2650 50  0001 C CNN "MPN"
+F 5 "Yageo" H 4350 2650 50  0001 C CNN "Mfr."
 	1    4350 2650
 	-1   0    0    1

Commit message: PCB Layout Checkpoint
Parts:
- J13: renamed from J11; footprint grootvoet:USB_C_Receptacle_Amphenol_12401610E4-2A -> grootvoet:USB_C_Recepetacle_JAE_DX07S016JA1; MPN 12401610E4#2A -> DX07S016JA1R1500; Mfr. Amphenol Commercial Products -> JAE Electronics
- renumbered CB29 to CB39, J9 to J11, J10 to J12, R71 to R89, R72 to R90, R73 to R91, U8 to U10
Connections:
- net USB_CONN_D+: now also U10.4 (I/O2); no longer U10.6 (I/O1)
- net USB_CONN_D-: now also U10.6 (I/O1); no longer U10.4 (I/O2)
- net USB_D+: now also U10.3 (I/O2); no longer U10.1 (I/O1)
- net USB_D-: now also U10.1 (I/O1); no longer U10.3 (I/O2)
Changed lines of the file:
@@
 $EndDescr
 $Comp
-L power:GND #PWR0124
+L power:GND #PWR0130
 U 1 1 5EF579E9
 P 7200 4000
-F 0 "#PWR0124" H 7200 3750 50  0001 C CNN
+F 0 "#PWR0130" H 7200 3750 50  0001 C CNN
 F 1 "GND" H 7205 3827 50  0000 C CNN
 F 2 "" H 7200 4000 50  0001 C CNN
@@
 $EndComp
 $Comp
-L power:Earth #PWR0123
+L power:Earth #PWR0129
 U 1 1 5EF579EF
 P 6900 4000
-F 0 "#PWR0123" H 6900 3750 50  0001 C CNN
+F 0 "#PWR0129" H 6900 3750 50  0001 C CNN
 F 1 "Earth" H 6900 3850 50  0001 C CNN
 F 2 "" H 6900 4000 50  0001 C CNN
@@
 $EndComp
 $Comp
-L power:VBUS #PWR0125
+L power:VBUS #PWR0131
 U 1 1 5EF579F5
 P 7900 2500
-F 0 "#PWR0125" H 7900 2350 50  0001 C CNN
+F 0 "#PWR0131" H 7900 2350 50  0001 C CNN
 F 1 "VBUS" H 7915 2673 50  0000 C CNN
 F 2 "" H 7900 2500 50  0001 C CNN
@@
 	7900 3000 7800 3000
 $Comp
-L Connector:USB_C_Receptacle_USB2.0 J11
+L Connector:USB_C_Receptacle_USB2.0 J13
 U 1 1 5EF57A02
 P 7200 3100
-F 0 "J11" H 7307 3967 50  0000 C CNN
+F 0 "J13" H 7307 3967 50  0000 C CNN
 F 1 "USB_C_Receptacle_USB2.0" H 7150 3900 50  0000 C CNN
-F 2 "grootvoet:USB_C_Receptacle_Amphenol_12401610E4-2A" H 7350 3100 50  0001 C CNN
+F 2 "grootvoet:USB_C_Recepetacle_JAE_DX07S016JA1" H 7350 3100 50  0001 C CNN
 F 3 "https://www.usb.org/sites/default/files/documents/usb_type-c.zip" H 7350 3100 50  0001 C CNN
-F 4 "Amphenol Commercial Products" H 7200 3100 50  0001 C CNN "Mfr."
-F 5 "12401610E4#2A" H 7200 3100 50  0001 C CNN "MPN"
+F 4 "JAE Electronics" H 7200 3100 50  0001 C CNN "Mfr."
+F 5 "DX07S016JA1R1500" H 7200 3100 50  0001 C CNN "MPN"
 	1    7200 3100
 	1    0    0    -1
@@
 NoConn ~ 7800 3600
 $Comp
-L Device:R_Small R72
+L Device:R_Small R90
 U 1 1 5EF57A0A
 P 8500 3050
-F 0 "R72" H 8441 3004 50  0000 R CNN
+F 0 "R90" H 8441 3004 50  0000 R CNN
 F 1 "5.1k" H 8441 3095 50  0000 R CNN
 F 2 "Resistor_SMD:R_0603_1608Metric_Pad1.05x0.95mm_HandSolder" H 8500 3050 50  0001 C CNN
@@
 $EndComp
 $Comp
-L Device:R_Small R73
+L Device:R_Small R91
 U 1 1 5EF57A10
 P 8800 3050
-F 0 "R73" H 8741 3004 50  0000 R CNN
+F 0 "R91" H 8741 3004 50  0000 R CNN
 F 1 "5.1k" H 8741 3095 50  0000 R CNN
 F 2 "Resistor_SMD:R_0603_1608Metric_Pad1.05x0.95mm_HandSolder" H 8800 3050 50  0001 C CNN
@@
 	8800 2700 7800 2700
 $Comp
-L power:GND #PWR0126
+L power:GND #PWR0132
 U 1 1 5EF57A1A
 P 8650 3300
-F 0 "#PWR0126" H 8650 3050 50  0001 C CNN
+F 0 "#PWR0132" H 8650 3050 50  0001 C CNN
 F 1 "GND" H 8655 3127 50  0000 C CNN
 F 2 "" H 8650 3300 50  0001 C CNN
@@
 	9550 3500 9550 3450
 $Comp
-L power:Earth #PWR0127
+L power:Earth #PWR0133
 U 1 1 5EF57A38
 P 9550 3500
-F 0 "#PWR0127" H 9550 3250 50  0001 C CNN
+F 0 "#PWR0133" H 9550 3250 50  0001 C CNN
 F 1 "Earth" H 9550 3350 50  0001 C CNN
 F 2 "" H 9550 3500 50  0001 C CNN
@@
 USB-C Connection
 $Comp
-L power:Earth #PWR0122
+L power:Earth #PWR0128
 U 1 1 5EF59730
 P 6200 3750
-F 0 "#PWR0122" H 6200 3500 50  0001 C CNN
+F 0 "#PWR0128" H 6200 3500 50  0001 C CNN
 F 1 "Earth" H 6200 3600 50  0001 C CNN
 F 2 "" H 6200 3750 50  0001 C CNN
@@
 	1    0    0    -1
 $EndComp
-Text HLabel 3400 5500 0    50   BiDi ~ 0
-USB_D+
-Text HLabel 4200 5500 2    50   BiDi ~ 0
-USB_D-
 Text HLabel 3300 3550 0    50   BiDi ~ 0
 SDIO_D1
@@
 SDIO_WP
 $Comp
-L power:GND #PWR0117
+L power:GND #PWR0123
 U 1 1 5EFBCDAD
 P 4350 3850
-F 0 "#PWR0117" H 4350 3600 50  0001 C CNN
+F 0 "#PWR0123" H 4350 3600 50  0001 C CNN
 F 1 "GND" H 4355 3677 50  0000 C CNN
 F 2 "" H 4350 3850 50  0001 C CNN
@@
 SD Card Holder
 $Comp
-L Connector_Generic:Conn_01x02 J10
+L Connector_Generic:Conn_01x02 J12
 U 1 1 5EE0C945
 P 6200 5400
-F 0 "J10" H 6280 5392 50  0000 L CNN
+F 0 "J12" H 6280 5392 50  0000 L CNN
 F 1 "JST-PH" H 6280 5301 50  0000 L CNN
 F 2 "Connector_JST:JST_PH_S2B-PH-SM4-TB_1x02-1MP_P2.00mm_Horizontal" H 6200 5400 50  0001 C CNN
@@
 $EndComp
 $Comp
-L power:+BATT #PWR0120
+L power:+BATT #PWR0126
 U 1 1 5EE0C94B
 P 6000 5200
-F 0 "#PWR0120" H 6000 5050 50  0001 C CNN
+F 0 "#PWR0126" H 6000 5050 50  0001 C CNN
 F 1 "+BATT" H 6015 5373 50  0000 C CNN
 F 2 "" H 6000 5200 50  0001 C CNN
@@
 $EndComp
 $Comp
-L power:GND #PWR0121
+L power:GND #PWR0127
 U 1 1 5EE0C951
 P 6000 5700
-F 0 "#PWR0121" H 6000 5450 50  0001 C CNN
+F 0 "#PWR0127" H 6000 5450 50  0001 C CNN
 F 1 "GND" H 6005 5527 50  0000 C CNN
 F 2 "" H 6000 5700 50  0001 C CNN
@@
 LIPO Battery Connector
 $Comp
-L Power_Protection:USBLC6-2SC6 U8
+L Power_Protection:USBLC6-2SC6 U10
 U 1 1 5EF91333
 P 3800 5400
-F 0 "U8" H 3550 5750 50  0000 C CNN
+F 0 "U10" H 3550 5750 50  0000 C CNN
 F 1 "USBLC6-2SC6" H 4150 5750 50  0000 C CNN
 F 2 "Package_TO_SOT_SMD:SOT-23-6" H 3800 4900 50  0001 C CNN
@@
 $EndComp
 $Comp
-L power:GND #PWR0115
+L power:GND #PWR0121
 U 1 1 5EF9E21E
 P 3800 5800
-F 0 "#PWR0115" H 3800 5550 50  0001 C CNN
+F 0 "#PWR0121" H 3800 5550 50  0001 C CNN
 F 1 "GND" H 3805 5627 50  0000 C CNN
 F 2 "" H 3800 5800 50  0001 C CNN
@@
 $EndComp
 $Comp
-L power:VBUS #PWR0114
+L power:VBUS #PWR0120
 U 1 1 5EF9EE8C
 P 3800 5000
-F 0 "#PWR0114" H 3800 4850 50  0001 C CNN
+F 0 "#PWR0120" H 3800 4850 50  0001 C CNN
 F 1 "VBUS" H 3815 5173 50  0000 C CNN
 F 2 "" H 3800 5000 50  0001 C CNN
@@
 	1    0    0    -1
 $EndComp
-Text Label 4200 5300 0    50   ~ 0
-USB_CONN_D-
-Text Label 3400 5300 2    50   ~ 0
-USB_CONN_D+
 Text Label 7900 3200 0    50   ~ 0
 USB_CONN_D+
@@
 USB ESD Protection
 $Comp
-L Device:C_Small CB29
+L Device:C_Small CB39
 U 1 1 5EFBCA6D
 P 4950 5400
-F 0 "CB29" H 5042 5446 50  0000 L CNN
+F 0 "CB39" H 5042 5446 50  0000 L CNN
 F 1 "100n" H 5042 5355 50  0000 L CNN
 F 2 "Capacitor_SMD:C_0603_1608Metric_Pad1.05x0.95mm_HandSolder" H 4950 5400 50  0001 C CNN
@@
 $EndComp
 $Comp
-L power:VBUS #PWR0118
+L power:VBUS #PWR0124
 U 1 1 5EFBD2C9
 P 4950 5200
-F 0 "#PWR0118" H 4950 5050 50  0001 C CNN
+F 0 "#PWR0124" H 4950 5050 50  0001 C CNN
 F 1 "VBUS" H 4965 5373 50  0000 C CNN
 F 2 "" H 4950 5200 50  0001 C CNN
@@
 $EndComp
 $Comp
-L power:GND #PWR0119
+L power:GND #PWR0125
 U 1 1 5EFBD729
 P 4950 5600
-F 0 "#PWR0119" H 4950 5350 50  0001 C CNN
+F 0 "#PWR0125" H 4950 5350 50  0001 C CNN
 F 1 "GND" H 4955 5427 50  0000 C CNN
 F 2 "" H 4950 5600 50  0001 C CNN
@@
 	2750 4750 5400 4750
 $Comp
-L Device:R_Small R71
+L Device:R_Small R89
 U 1 1 5EF7DC5F
 P 4350 2650
-F 0 "R71" H 4291 2604 50  0000 R CNN
+F 0 "R89" H 4291 2604 50  0000 R CNN
 F 1 "10k" H 4291 2695 50  0000 R CNN
 F 2 "Resistor_SMD:R_0603_1608Metric_Pad1.05x0.95mm_HandSolder" H 4350 2650 50  0001 C CNN
@@
 $EndComp
 $Comp
-L Connector:Micro_SD_Card_Det J9
+L Connector:Micro_SD_Card_Det J11
 U 1 1 5EF580BF
 P 5400 3250
-F 0 "J9" H 5350 4067 50  0000 C CNN
+F 0 "J11" H 5350 4067 50  0000 C CNN
 F 1 "Micro_SD_Card_Det" H 5350 3976 50  0000 C CNN
 F 2 "Connector_Card:microSD_HC_Hirose_DM3D-SF" H 7450 3950 50  0001 C CNN
@@
 $EndComp
 $Comp
-L power:+3V3 #PWR0116
+L power:+3V3 #PWR0122
 U 1 1 5EF922F3
 P 4250 2450
-F 0 "#PWR0116" H 4250 2300 50  0001 C CNN
+F 0 "#PWR0122" H 4250 2300 50  0001 C CNN
 F 1 "+3V3" H 4265 2623 50  0000 C CNN
 F 2 "" H 4250 2450 50  0001 C CNN
@@
 Wire Wire Line
 	4150 3150 4500 3150
+Text Label 3400 5300 2    50   ~ 0
+USB_CONN_D-
+Text HLabel 3400 5500 0    50   BiDi ~ 0
+USB_D-
+Text HLabel 4200 5500 2    50   BiDi ~ 0
+USB_D+
+Text Label 4200 5300 0    50   ~ 0
+USB_CONN_D+
 $EndSCHEMATC

Commit message: Major Commit with Final PCB Design
Parts:
- removed H1: MountingHole_Pad, MountingHole:MountingHole_4.3mm_M4_Pad_Via, symbol Mechanical:MountingHole_Pad
- J11: footprint Connector_Card:microSD_HC_Hirose_DM3D-SF -> grootvoet:microSD_HC_Molex_5031821852; MPN DM3D-SF -> 503182-1852; Mfr. Hirose Connector -> Molex
- J12: footprint Connector_JST:JST_PH_S2B-PH-SM4-TB_1x02-1MP_P2.00mm_Horizontal -> grootvoet:JST_PH_S2B-PH-SM4-TB_1x02-1MP_P2.00mm_Horizontal
- U10: footprint Package_TO_SOT_SMD:SOT-23-6 -> grootvoet:SOT-666_Handsoldering; MPN USBLC6-2SC6Y -> USBLC6-2P6
Changed lines of the file:
@@
 Connect shield to all external mounting and \nthen to GND at a single point close to the \nconnector. Place all IO connectors (with shields) \nclose to each other.
 Wire Wire Line
-	9400 3450 9100 3450
-Connection ~ 9400 3450
-Wire Wire Line
-	9100 3450 9100 3400
-Connection ~ 9550 3450
-Wire Wire Line
 	9400 3450 9400 3400
-Wire Wire Line
-	9550 3450 9400 3450
 Connection ~ 9700 3450
 Wire Wire Line
@@
 Wire Wire Line
 	9700 3450 9700 3400
-Wire Wire Line
-	9550 3450 9700 3450
-Wire Wire Line
-	9550 3500 9550 3450
 $Comp
 L power:Earth #PWR0133
 U 1 1 5EF57A38
-P 9550 3500
-F 0 "#PWR0133" H 9550 3250 50  0001 C CNN
-F 1 "Earth" H 9550 3350 50  0001 C CNN
-F 2 "" H 9550 3500 50  0001 C CNN
-F 3 "~" H 9550 3500 50  0001 C CNN
-	1    9550 3500
+P 9700 3450
+F 0 "#PWR0133" H 9700 3200 50  0001 C CNN
+F 1 "Earth" H 9700 3300 50  0001 C CNN
+F 2 "" H 9700 3450 50  0001 C CNN
+F 3 "~" H 9700 3450 50  0001 C CNN
+	1    9700 3450
 	1    0    0    -1
 $EndComp
@@
 F 3 "~" H 9400 3300 50  0001 C CNN
 	1    9400 3300
-	1    0    0    -1
-$EndComp
-$Comp
-L Mechanical:MountingHole_Pad H1
-U 1 1 5EF57A50
-P 9100 3300
-F 0 "H1" H 9200 3303 50  0000 L CNN
-F 1 "MountingHole_Pad" H 9200 3258 50  0001 L CNN
-F 2 "MountingHole:MountingHole_4.3mm_M4_Pad_Via" H 9100 3300 50  0001 C CNN
-F 3 "~" H 9100 3300 50  0001 C CNN
-	1    9100 3300
 	1    0    0    -1
 $EndComp
@@
 F 0 "J12" H 6280 5392 50  0000 L CNN
 F 1 "JST-PH" H 6280 5301 50  0000 L CNN
-F 2 "Connector_JST:JST_PH_S2B-PH-SM4-TB_1x02-1MP_P2.00mm_Horizontal" H 6200 5400 50  0001 C CNN
+F 2 "grootvoet:JST_PH_S2B-PH-SM4-TB_1x02-1MP_P2.00mm_Horizontal" H 6200 5400 50  0001 C CNN
 F 3 "~" H 6200 5400 50  0001 C CNN
 F 4 "1769" H 6200 5400 50  0001 C CNN "MPN"
@@
 F 0 "U10" H 3550 5750 50  0000 C CNN
 F 1 "USBLC6-2SC6" H 4150 5750 50  0000 C CNN
-F 2 "Package_TO_SOT_SMD:SOT-23-6" H 3800 4900 50  0001 C CNN
+F 2 "grootvoet:SOT-666_Handsoldering" H 3800 4900 50  0001 C CNN
 F 3 "https://www.st.com/resource/en/datasheet/usblc6-2.pdf" H 4000 5750 50  0001 C CNN
-F 4 "USBLC6-2SC6Y" H 3800 5400 50  0001 C CNN "MPN"
+F 4 "USBLC6-2P6" H 3800 5400 50  0001 C CNN "MPN"
 F 5 "STMicroelectronics" H 3800 5400 50  0001 C CNN "Mfr."
 	1    3800 5400
@@
 F 0 "J11" H 5350 4067 50  0000 C CNN
 F 1 "Micro_SD_Card_Det" H 5350 3976 50  0000 C CNN
-F 2 "Connector_Card:microSD_HC_Hirose_DM3D-SF" H 7450 3950 50  0001 C CNN
+F 2 "grootvoet:microSD_HC_Molex_5031821852" H 7450 3950 50  0001 C CNN
 F 3 "https://www.hirose.com/product/en/download_file/key_name/DM3/category/Catalog/doc_file_id/49662/?file_category_id=4&item_id=195&is_series=1" H 5400 3350 50  0001 C CNN
-F 4 "DM3D-SF" H 5400 3250 50  0001 C CNN "MPN"
-F 5 "Hirose Connector" H 5400 3250 50  0001 C CNN "Mfr."
+F 4 "503182-1852" H 5400 3250 50  0001 C CNN "MPN"
+F 5 "Molex" H 5400 3250 50  0001 C CNN "Mfr."
 	1    5400 3250
 	1    0    0    -1
@@
 Text Label 4200 5300 0    50   ~ 0
 USB_CONN_D+
+Wire Wire Line
+	9400 3450 9700 3450
 $EndSCHEMATC

Commit message: CHange to single 3 designs to save cost
Parts:
- H2, H3, H4: footprint MountingHole:MountingHole_4.3mm_M4_Pad_Via -> MountingHole:MountingHole_3.2mm_M3_Pad_Via
Changed lines of the file:
@@
 F 0 "H4" H 10100 3303 50  0000 L CNN
 F 1 "MountingHole_Pad" H 10100 3258 50  0001 L CNN
-F 2 "MountingHole:MountingHole_4.3mm_M4_Pad_Via" H 10000 3300 50  0001 C CNN
+F 2 "MountingHole:MountingHole_3.2mm_M3_Pad_Via" H 10000 3300 50  0001 C CNN
 F 3 "~" H 10000 3300 50  0001 C CNN
 	1    10000 3300
@@
 F 0 "H3" H 9800 3303 50  0000 L CNN
 F 1 "MountingHole_Pad" H 9800 3258 50  0001 L CNN
-F 2 "MountingHole:MountingHole_4.3mm_M4_Pad_Via" H 9700 3300 50  0001 C CNN
+F 2 "MountingHole:MountingHole_3.2mm_M3_Pad_Via" H 9700 3300 50  0001 C CNN
 F 3 "~" H 9700 3300 50  0001 C CNN
 	1    9700 3300
@@
 F 0 "H2" H 9500 3303 50  0000 L CNN
 F 1 "MountingHole_Pad" H 9500 3258 50  0001 L CNN
-F 2 "MountingHole:MountingHole_4.3mm_M4_Pad_Via" H 9400 3300 50  0001 C CNN
+F 2 "MountingHole:MountingHole_3.2mm_M3_Pad_Via" H 9400 3300 50  0001 C CNN
 F 3 "~" H 9400 3300 50  0001 C CNN
 	1    9400 3300

Commit message: Try split up project to multiboard
NOTE: There was a warning about libs being out of date and the USB-C
connector. This was partly due to the 'libs' dir not being up to date
but the USB-C looks like a global update.
Parts:
- J13: symbol Connector:USB_C_Receptacle_USB2.0 -> kleinvoet-rescue:USB_C_Receptacle_USB2.0-Connector
Changed lines of the file:
@@
 	7900 3000 7800 3000
 $Comp
-L Connector:USB_C_Receptacle_USB2.0 J13
+L kleinvoet-rescue:USB_C_Receptacle_USB2.0-Connector J13
 U 1 1 5EF57A02
 P 7200 3100

Commit message: Misc. TODOs
Parts:
- added C3: 1u, Capacitor_SMD:C_0603_1608Metric_Pad1.08x0.95mm_HandSolder, symbol Device:C_Small
- CB39: footprint Capacitor_SMD:C_0603_1608Metric_Pad1.05x0.95mm_HandSolder -> Capacitor_SMD:C_0603_1608Metric_Pad1.08x0.95mm_HandSolder
Connections:
- net +3V3: now also C3.1
- net GND: now also C3.2
Changed lines of the file:
@@
 $Descr A4 11693 8268
 encoding utf-8
-Sheet 16 13
+Sheet 12 13
 Title "Kleinvoet"
 Date "2020-06-11"
@@
 F 0 "CB39" H 5042 5446 50  0000 L CNN
 F 1 "100n" H 5042 5355 50  0000 L CNN
-F 2 "Capacitor_SMD:C_0603_1608Metric_Pad1.05x0.95mm_HandSolder" H 4950 5400 50  0001 C CNN
+F 2 "Capacitor_SMD:C_0603_1608Metric_Pad1.08x0.95mm_HandSolder" H 4950 5400 50  0001 C CNN
 F 3 "~" H 4950 5400 50  0001 C CNN
 F 4 "C0603C104M5RACTU" H 4950 5400 50  0001 C CNN "MPN"
@@
 Wire Wire Line
 	9400 3450 9700 3450
+$Comp
+L Device:C_Small C?
+U 1 1 5F937BF5
+P 3150 2450
+AR Path="/5F937BF5" Ref="C?"  Part="1"
+AR Path="/5EF53A66/5F937BF5" Ref="C3"  Part="1"
+F 0 "C3" H 3242 2496 50  0000 L CNN
+F 1 "1u" H 3242 2405 50  0000 L CNN
+F 2 "Capacitor_SMD:C_0603_1608Metric_Pad1.08x0.95mm_HandSolder" H 3150 2450 50  0001 C CNN
+F 3 "~" H 3150 2450 50  0001 C CNN
+F 4 "C0603C105K8RACTU" H 3150 2450 50  0001 C CNN "MPN"
+F 5 "KEMET" H 3150 2450 50  0001 C CNN "Mfr."
+	1    3150 2450
+	1    0    0    -1
+$EndComp
+$Comp
+L power:+3V3 #PWR03
+U 1 1 5F938578
+P 3150 2350
+F 0 "#PWR03" H 3150 2200 50  0001 C CNN
+F 1 "+3V3" H 3165 2523 50  0000 C CNN
+F 2 "" H 3150 2350 50  0001 C CNN
+F 3 "" H 3150 2350 50  0001 C CNN
+	1    3150 2350
+	1    0    0    -1
+$EndComp
+$Comp
+L power:GND #PWR07
+U 1 1 5F9387A8
+P 3150 2550
+F 0 "#PWR07" H 3150 2300 50  0001 C CNN
+F 1 "GND" H 3155 2377 50  0000 C CNN
+F 2 "" H 3150 2550 50  0001 C CNN
+F 3 "" H 3150 2550 50  0001 C CNN
+	1    3150 2550
+	1    0    0    -1
+$EndComp
 $EndSCHEMATC
