File: Sensor_Connector.sch (KiCad schematic (older format))
At the start: 6 parts, among them J3 Sensor_Conn

Commit message: Start layout
Connections:
- net SIG_N: now also C18.2, FB4.1; no longer FB4.2, J3.3 (Pin_3), TP19.1
- net SIG_P: now also C19.1, FB3.1; no longer FB3.2, J3.1 (Pin_1), TP19.2
- new net SIG_CONN_N: FB4.2, J3.1 (Pin_1), TP19.1
- new net SIG_CONN_P: FB3.2, J3.3 (Pin_3), TP19.2
Changed lines of the file:
@@
 $Descr A4 11693 8268
 encoding utf-8
-Sheet 6 9
+Sheet 5 9
 Title "Kleinvoet"
 Date "2020-06-11"
@@
 Text Notes 6250 3050 0    50   ~ 0
 PIN LAYOUT\n----------------\n1 | Enable\n2 | Calibration Enable\n3 | Calibration Signal\n4 | Signal (N)\n5 | GND\n6 | Signal (P)\n7 | GND\n8 | Power Supply (+3v3)
-Text HLabel 1800 5300 0    50   Input ~ 0
+Text HLabel 2550 5300 2    50   Input ~ 0
 SIG_P
-Text HLabel 1800 5750 0    50   Input ~ 0
+Text HLabel 2550 5750 2    50   Input ~ 0
 SIG_N
 Text Notes 7450 5600 0    50   ~ 0
@@
 AR Path="/5EE5ECAD/5EFF6D57/5EEA2252" Ref="C30"  Part="1"
 AR Path="/5EE5ECAD/5EFFC4F7/5EEA2252" Ref="C32"  Part="1"
-F 0 "C30" H 2542 5946 50  0000 L CNN
+F 0 "C18" H 2542 5946 50  0000 L CNN
 F 1 "220p" H 2542 5855 50  0000 L CNN
 F 2 "Capacitor_SMD:C_0603_1608Metric_Pad1.08x0.95mm_HandSolder" H 2450 5900 50  0001 C CNN
@@
 AR Path="/5EE5ECAD/5EFF6D57/5EEA248A" Ref="C31"  Part="1"
 AR Path="/5EE5ECAD/5EFFC4F7/5EEA248A" Ref="C33"  Part="1"
-F 0 "C31" H 2542 5046 50  0000 L CNN
+F 0 "C19" H 2542 5046 50  0000 L CNN
 F 1 "220p" H 2542 4955 50  0000 L CNN
 F 2 "Capacitor_SMD:C_0603_1608Metric_Pad1.08x0.95mm_HandSolder" H 2450 5000 50  0001 C CNN
@@
 	1    0    0    1
 $EndComp
-Text Notes 1400 4550 0    50   ~ 10
+Text Notes 1300 4600 0    50   ~ 10
 Signal Conditioning
 Wire Notes Line
@@
 AR Path="/5EE5ECAD/5EFF6D57/5EFE739C" Ref="#PWR079"  Part="1"
 AR Path="/5EE5ECAD/5EFFC4F7/5EFE739C" Ref="#PWR085"  Part="1"
-F 0 "#PWR079" H 1850 3400 50  0001 C CNN
+F 0 "#PWR067" H 1850 3400 50  0001 C CNN
 F 1 "GND" V 1850 3450 50  0000 C CNN
 F 2 "" H 1850 3650 50  0001 C CNN
@@
 	0    1    -1   0
 $EndComp
-Text HLabel 4050 4000 0    50   Output ~ 0
-SIG_N
 $Comp
 L power:+3V3 #PWR065
@@
 AR Path="/5EE5ECAD/5EFF6D57/5EE5C6A5" Ref="#PWR077"  Part="1"
 AR Path="/5EE5ECAD/5EFFC4F7/5EE5C6A5" Ref="#PWR083"  Part="1"
-F 0 "#PWR077" H 2350 3500 50  0001 C CNN
+F 0 "#PWR065" H 2350 3500 50  0001 C CNN
 F 1 "+3V3" V 2350 3850 50  0000 C CNN
 F 2 "" H 2350 3650 50  0001 C CNN
@@
 	0    1    -1   0
 $EndComp
-Text HLabel 4450 4000 2    50   Output ~ 0
-SIG_P
 $Comp
 L power:GND #PWR?
@@
 AR Path="/5EE5ECAD/5EFF6D57/5EF00E56" Ref="#PWR0146"  Part="1"
 AR Path="/5EE5ECAD/5EFFC4F7/5EF00E56" Ref="#PWR0147"  Part="1"
-F 0 "#PWR0146" H 2350 3200 50  0001 C CNN
+F 0 "#PWR0144" H 2350 3200 50  0001 C CNN
 F 1 "GND" V 2350 3250 50  0000 C CNN
 F 2 "" H 2350 3450 50  0001 C CNN
@@
 AR Path="/5EE5ECAD/5EFF6D57/5F997D5D" Ref="FB7"  Part="1"
 AR Path="/5EE5ECAD/5EFFC4F7/5F997D5D" Ref="FB12"  Part="1"
-F 0 "FB7" V 1913 5300 50  0000 C CNN
+F 0 "FB3" V 1913 5300 50  0000 C CNN
 F 1 "Ferrite_Bead_Small" V 2004 5300 50  0000 C CNN
 F 2 "Inductor_SMD:L_0603_1608Metric_Pad1.05x0.95mm_HandSolder" V 2080 5300 50  0001 C CNN
@@
 AR Path="/5EE5ECAD/5EFF6D57/5F999474" Ref="FB11"  Part="1"
 AR Path="/5EE5ECAD/5EFFC4F7/5F999474" Ref="FB13"  Part="1"
-F 0 "FB11" V 1913 5750 50  0000 C CNN
+F 0 "FB4" V 1913 5750 50  0000 C CNN
 F 1 "Ferrite_Bead_Small" V 2004 5750 50  0000 C CNN
 F 2 "Inductor_SMD:L_0603_1608Metric_Pad1.05x0.95mm_HandSolder" V 2080 5750 50  0001 C CNN
@@
 AR Path="/5EE5ECAD/5EFF6D57/5EEA4A0A" Ref="#PWR080"  Part="1"
 AR Path="/5EE5ECAD/5EFFC4F7/5EEA4A0A" Ref="#PWR086"  Part="1"
-F 0 "#PWR080" H 2450 5750 50  0001 C CNN
+F 0 "#PWR068" H 2450 5750 50  0001 C CNN
 F 1 "GND" H 2455 5827 50  0000 C CNN
 F 2 "" H 2450 6000 50  0001 C CNN
@@
 AR Path="/5EE5ECAD/5EFF6D57/5F99FD60" Ref="#PWR0189"  Part="1"
 AR Path="/5EE5ECAD/5EFFC4F7/5F99FD60" Ref="#PWR0191"  Part="1"
-F 0 "#PWR0189" H 2450 4650 50  0001 C CNN
+F 0 "#PWR0185" H 2450 4650 50  0001 C CNN
 F 1 "GND" H 2455 4727 50  0000 C CNN
 F 2 "" H 2450 4900 50  0001 C CNN
@@
 	2050 5300 1800 5300
 Wire Notes Line
-	1450 4600 1450 6300
-Wire Notes Line
-	1450 6300 2850 6300
-Wire Notes Line
 	2850 6300 2850 4600
-Wire Notes Line
-	1450 4600 2850 4600
 $Comp
 L power:GND #PWR?
@@
 AR Path="/5EE5ECAD/5EFF6D57/5F9A54A7" Ref="#PWR0188"  Part="1"
 AR Path="/5EE5ECAD/5EFFC4F7/5F9A54A7" Ref="#PWR0190"  Part="1"
-F 0 "#PWR0188" H 2350 3300 50  0001 C CNN
+F 0 "#PWR0184" H 2350 3300 50  0001 C CNN
 F 1 "GND" V 2350 3350 50  0000 C CNN
 F 2 "" H 2350 3550 50  0001 C CNN
@@
 AR Path="/5EE5ECAD/5EFF6D57/5EDAD860" Ref="J6"  Part="1"
 AR Path="/5EE5ECAD/5EFFC4F7/5EDAD860" Ref="J7"  Part="1"
-F 0 "J6" H 2100 3750 50  0000 C CNN
+F 0 "J3" H 2100 3750 50  0000 C CNN
 F 1 "Sensor_Conn" H 2100 3850 50  0000 C CNN
 F 2 "grootvoet:TE_7-215079-8" H 2050 3550 50  0001 C CNN
@@
 AR Path="/5EE5ECAD/5EFF6D57/5F9E0F6D" Ref="TP21"  Part="1"
 AR Path="/5EE5ECAD/5EFFC4F7/5F9E0F6D" Ref="TP22"  Part="1"
-F 0 "TP21" H 4250 4195 50  0000 C CNN
+F 0 "TP19" H 4250 4195 50  0000 C CNN
 F 1 "SIG" H 4250 4104 50  0000 C CNN
 F 2 "TestPoint:TestPoint_2Pads_Pitch2.54mm_Drill0.8mm" H 4250 4000 50  0001 C CNN
@@
 	1    0    0    -1
 $EndComp
-Text HLabel 1850 3550 0    50   Output ~ 0
-SIG_N
-Text HLabel 1850 3450 0    50   Output ~ 0
-SIG_P
+Wire Wire Line
+	2550 5300 2450 5300
+Connection ~ 2450 5300
+Wire Wire Line
+	2550 5750 2450 5750
+Connection ~ 2450 5750
+Text Label 1850 3450 2    50   ~ 0
+SIG_CONN_N
+Text Label 1850 3550 2    50   ~ 0
+SIG_CONN_P
+Text Label 1800 5300 2    50   ~ 0
+SIG_CONN_P
+Text Label 1800 5750 2    50   ~ 0
+SIG_CONN_N
+Wire Notes Line
+	1300 4600 1300 6300
+Wire Notes Line
+	1300 6300 2850 6300
+Wire Notes Line
+	1300 4600 2850 4600
+Text Label 4450 4000 0    50   ~ 0
+SIG_CONN_P
+Text Label 4050 4000 2    50   ~ 0
+SIG_CONN_N
 $EndSCHEMATC
