File: kleinvoet.sch (KiCad schematic (older format))
At the start: 37 parts, among them J1 Conn_ST_STDC14, SW1 RESET, SW2 USER, U1 STM32F446RETx, Y1 12 MHz, Y2 32.768 kHz

Commit message: Route analog section
Parts:
- R1: value 100k -> 10k; MPN RC0603FR-07100KL -> (none)
Changed lines of the file:
@@
 P 3450 1850
 F 0 "R1" H 3509 1896 50  0000 L CNN
-F 1 "100k" H 3509 1805 50  0000 L CNN
+F 1 "10k" H 3509 1805 50  0000 L CNN
 F 2 "Resistor_SMD:R_0603_1608Metric_Pad0.98x0.95mm_HandSolder" H 3450 1850 50  0001 C CNN
 F 3 "~" H 3450 1850 50  0001 C CNN
-F 4 "RC0603FR-07100KL" H 3450 1850 50  0001 C CNN "MPN"
+F 4 "" H 3450 1850 50  0001 C CNN "MPN"
 F 5 "Yageo" H 3450 1850 50  0001 C CNN "Mfr."
 	1    3450 1850

Commit message: Major layout update
Changed lines of the file:
@@
 $EndDescr
 $Sheet
-S 1400 2100 1000 600
+S 1400 2100 1000 500
 U 5EE5ECAD
 F0 "ADC_Interface" 50
@@
 F8 "SCL" I L 1400 2300 50
 F9 "EN_XO" I L 1400 2500 50
-F10 "MCLK" I R 2400 2600 50
 $EndSheet
 $Sheet
@@
 Wire Wire Line
 	5450 4050 6200 4050
-Text Label 3250 3050 2    50   ~ 0
-ADC_SAI_MCLK
-Wire Wire Line
-	3250 3050 4050 3050
 Text Label 3250 3150 2    50   ~ 0
 ADC_SAI_SD_A
@@
 Wire Wire Line
 	2550 2400 2400 2400
-Text Label 2550 2600 0    50   ~ 0
-ADC_SAI_MCLK
-Wire Wire Line
-	2550 2600 2400 2600
 Text Label 6150 2450 0    50   ~ 0
 ADC_XO_EN
@@
 Wire Wire Line
 	5450 1950 6150 1950
+Wire Wire Line
+	4050 3050 3850 3050
 Text Label 2550 2500 0    50   ~ 0
 ADC_SAI_SD_A

Commit message: Change ST-LINk loc.
Connections:
- net ADC_XO_EN renamed D2
Changed lines of the file:
@@
 Wire Wire Line
 	2550 2400 2400 2400
-Text Label 6150 2450 0    50   ~ 0
-ADC_XO_EN
-Wire Wire Line
-	6150 2450 5450 2450
-Text Label 1200 2500 2    50   ~ 0
-ADC_XO_EN
-Wire Wire Line
-	1200 2500 1400 2500
 $Comp
 L Device:R_Small R6

Commit message: Route out GND planes
Parts:
- added FB5: BLM15HD102SN1, Inductor_SMD:L_0402_1005Metric, symbol Device:Ferrite_Bead_Small
- J1: footprint grootvoet:SAMTEC-FTSH-107-01-X-D -> grootvoet:SAMTEC-FTSH-107-01-X-DV; MPN M50-055023W0445 -> FTSH-107-01-F-DV-K; Mfr. Harwin -> Samtec
Connections:
- net RTC_CAL: now also FB5.2
- new net GNSS_Module/GPS_SYNC: FB5.1
Changed lines of the file:
@@
 F 0 "J1" H 1207 6696 50  0000 R CNN
 F 1 "Conn_ST_STDC14" H 1207 6605 50  0000 R CNN
-F 2 "grootvoet:SAMTEC-FTSH-107-01-X-D" H 1650 6650 50  0001 C CNN
+F 2 "grootvoet:SAMTEC-FTSH-107-01-X-DV" H 1650 6650 50  0001 C CNN
 F 3 "https://www.st.com/content/ccc/resource/technical/document/user_manual/group1/99/49/91/b6/b2/3a/46/e5/DM00526767/files/DM00526767.pdf/jcr:content/translations/en.DM00526767.pdf" V 1300 5400 50  0001 C CNN
-F 4 "M50-055023W0445" H 1650 6650 50  0001 C CNN "MPN"
-F 5 "Harwin" H 1650 6650 50  0001 C CNN "Mfr."
+F 4 "FTSH-107-01-F-DV-K" H 1650 6650 50  0001 C CNN "MPN"
+F 5 "Samtec" H 1650 6650 50  0001 C CNN "Mfr."
 	1    1650 6650
 	1    0    0    -1
@@
 Text Label 10100 5400 2    50   ~ 0
 OSC_LSE_OUT
-Text Label 1200 1550 2    50   ~ 0
+Text Label 1000 1550 2    50   ~ 0
 RTC_CAL
 Wire Wire Line
@@
 Text Label 2550 2400 0    50   ~ 0
 ADC_SAI_SD_B
+$Comp
+L Device:Ferrite_Bead_Small FB5
+U 1 1 5F9E7EDF
+P 1100 1550
+AR Path="/5F9E7EDF" Ref="FB5"  Part="1"
+AR Path="/5EDF3693/5F9E7EDF" Ref="FB?"  Part="1"
+F 0 "FB5" V 1000 1650 50  0000 C CNN
+F 1 "BLM15HD102SN1" V 1150 1900 50  0001 C CNN
+F 2 "Inductor_SMD:L_0402_1005Metric" V 1030 1550 50  0001 C CNN
+F 3 "~" H 1100 1550 50  0001 C CNN
+F 4 "BLM15HD102SN1D" V 1100 1550 50  0001 C CNN "MPN"
+F 5 "Murata Electronics" H 1100 1550 50  0001 C CNN "Mfr."
+	1    1100 1550
+	0    1    1    0
+$EndComp
 $EndSCHEMATC

Commit message: (WIP) SD config
Changed lines of the file:
@@
 Wire Wire Line
 	1200 1750 1400 1750
-Text Label 5650 2250 0    50   ~ 0
+Text Label 3850 3050 2    50   ~ 0
 SDIO_CD
-Wire Wire Line
-	5650 2250 5450 2250
 Text Label 1200 5200 2    50   ~ 0
 SDIO_CD
@@
 Text Label 3850 3150 2    50   ~ 0
 SAI1_SD_A
-Text Label 3850 3050 2    50   ~ 0
-SAI_MCLK_B
 NoConn ~ 4050 3450
 NoConn ~ 4050 3550

Commit message: Route USR BTN
Connections:
- net D12: now also CB9.1, SW2.1
- net D15: no longer CB9.1, SW2.1
Changed lines of the file:
@@
 Text Label 5400 6800 0    50   ~ 0
 LED_STATUS
-Text Label 6200 3950 0    50   ~ 0
+Text Label 6150 2050 0    50   ~ 0
 USR_BTN
-Wire Wire Line
-	6200 3950 5450 3950
 NoConn ~ 5450 3350
 Wire Wire Line
@@
 	5450 1850 6150 1850
 Wire Wire Line
-	5650 2050 5450 2050
-Wire Wire Line
 	5650 2150 5450 2150
 Text Label 6150 1950 0    50   ~ 0
@@
 	0    1    1    0
 $EndComp
+Wire Wire Line
+	5450 2050 6150 2050
 $EndSCHEMATC

Commit message: Route ADC rst
Connections:
- net D9 renamed ADC_~RST
Changed lines of the file:
@@
 	1200 2200 1400 2200
 Text Label 1200 2400 2    50   ~ 0
-~RST
+ADC_~RST
 Wire Wire Line
 	1200 2400 1400 2400
@@
 Wire Wire Line
 	5450 2050 6150 2050
+Text Label 3850 3750 2    50   ~ 0
+ADC_~RST
+Wire Wire Line
+	3850 3750 4050 3750
 $EndSCHEMATC
