File: Power.sch (KiCad schematic (older format))
At the start: 22 parts, among them Q1 PMOS, U8 MCP73831-2-OT, U9 TPS73733QDRBRQ1

Commit message: New ADC board layout
Merge feature/kv-new-adc

Squashed commit of the following:
===============================================

commit d560af3129baffdc71a13a7fa7beda6d7e4b1bbe
Author: CM Geldenhuys <20198329@sun.ac.za>
Date:   Mon Nov 2 10:16:05 2020 +0200

    Change board layout

commit e0e102b1b715915958904bd07514080422fcc802
Author: CM Geldenhuys <20198329@sun.ac.za>
Date:   Mon Nov 2 08:42:49 2020 +0200

    Route ADC rst

commit dbc5adba55d665b163eedfb4150514fe2b5b8ec8
Author: CM Geldenhuys <20198329@sun.ac.za>
Date:   Mon Nov 2 08:37:27 2020 +0200

    Fix GPS conn.

commit 0f139c20ac4bbbbfd2ab5507f187a5ddf70be7a1
Author: CM Geldenhuys <20198329@sun.ac.za>
Date:   Mon Nov 2 08:23:01 2020 +0200

    Route USR BTN

commit f6bd16c8e79a9fc3047a82e3e1abb388a579a1e4
Author: CM Geldenhuys <20198329@sun.ac.za>
Date:   Sun Nov 1 07:41:20 2020 +0200

    Route GPS Conn

commit 016e6e7ba1ce602e3233b00102ced6621a380f78
Author: CM Geldenhuys <20198329@sun.ac.za>
Date:   Fri Oct 30 17:31:13 2020 +0200

    Route Misc.

commit 6a809ae2e129821f12cca4ec3806ebf69337c268
Author: CM Geldenhuys <20198329@sun.ac.za>
Date:   Fri Oct 30 11:40:29 2020 +0200

    (WIP) SD config

commit b5d79f248cd283a71c5ab746a4afc4eb96850216
Author: CM Geldenhuys <20198329@sun.ac.za>
Date:   Fri Oct 30 11:24:56 2020 +0200

    Route ST-Link

commit dba35a7554c0c60ddd581dd4b7cbdf28445f26a1
Author: CM Geldenhuys <20198329@sun.ac.za>
Date:   Fri Oct 30 11:03:44 2020 +0200

    Route out GND planes

commit ee78e0f947a8edc358d3e2ec17c7ddf8f87e82dd
Author: CM Geldenhuys <20198329@sun.ac.za>
Date:   Thu Oct 29 16:17:03 2020 +0200

    Change ST-LINk loc.

commit b281a3fe16ed9d80db1964422c72eaf6acbfd9f3
Author: CM Geldenhuys <20198329@sun.ac.za>
Date:   Thu Oct 29 15:43:37 2020 +0200

    Major layout update

commit 655eae6cd0c7e79d683f16c4706ab989a6952fc5
Author: CM Geldenhuys <20198329@sun.ac.za>
Date:   Thu Oct 29 12:05:26 2020 +0200

    Route analog section

commit 0aa4140e89fcb36b0e9f339e25cad0a47a5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
Parts:
- C58, C59, C60, C62, C63: footprint Capacitor_SMD:C_0805_2012Metric_Pad1.15x1.40mm_HandSolder -> Capacitor_SMD:C_0805_2012Metric_Pad1.18x1.45mm_HandSolder
- R84, R85, R86, R87, R88: footprint Resistor_SMD:R_0603_1608Metric_Pad1.05x0.95mm_HandSolder -> Resistor_SMD:R_0603_1608Metric_Pad0.98x0.95mm_HandSolder
Changed lines of the file:
@@
 $Descr A4 11693 8268
 encoding utf-8
-Sheet 11 13
+Sheet 7 9
 Title "Kleinvoet"
 Date "2020-06-11"
@@
 F 0 "R84" H 3759 4196 50  0000 L CNN
 F 1 "100k" H 3759 4105 50  0000 L CNN
-F 2 "Resistor_SMD:R_0603_1608Metric_Pad1.05x0.95mm_HandSolder" H 3700 4150 50  0001 C CNN
+F 2 "Resistor_SMD:R_0603_1608Metric_Pad0.98x0.95mm_HandSolder" H 3700 4150 50  0001 C CNN
 F 3 "~" H 3700 4150 50  0001 C CNN
 F 4 "RC0603FR-07100KL" H 3700 4150 50  0001 C CNN "MPN"
@@
 F 0 "R86" V 5100 1650 50  0000 C CNN
 F 1 "10k" V 5300 1700 50  0000 C CNN
-F 2 "Resistor_SMD:R_0603_1608Metric_Pad1.05x0.95mm_HandSolder" H 5200 1650 50  0001 C CNN
+F 2 "Resistor_SMD:R_0603_1608Metric_Pad0.98x0.95mm_HandSolder" H 5200 1650 50  0001 C CNN
 F 3 "~" H 5200 1650 50  0001 C CNN
 F 4 "RC0603JR-0710KL" H 5200 1650 50  0001 C CNN "MPN"
@@
 F 0 "C58" H 4492 4296 50  0000 L CNN
 F 1 "10u" H 4492 4205 50  0000 L CNN
-F 2 "Capacitor_SMD:C_0805_2012Metric_Pad1.15x1.40mm_HandSolder" H 4400 4250 50  0001 C CNN
+F 2 "Capacitor_SMD:C_0805_2012Metric_Pad1.18x1.45mm_HandSolder" H 4400 4250 50  0001 C CNN
 F 3 "~" H 4400 4250 50  0001 C CNN
 F 4 "C0805C106K9PACTU" H 4400 4250 50  0001 C CNN "MPN"
@@
 F 0 "C63" H 7292 1796 50  0000 L CNN
 F 1 "10u" H 7292 1705 50  0000 L CNN
-F 2 "Capacitor_SMD:C_0805_2012Metric_Pad1.15x1.40mm_HandSolder" H 7200 1750 50  0001 C CNN
+F 2 "Capacitor_SMD:C_0805_2012Metric_Pad1.18x1.45mm_HandSolder" H 7200 1750 50  0001 C CNN
 F 3 "~" H 7200 1750 50  0001 C CNN
 F 4 "C0805C106K9PACTU" H 7200 1750 50  0001 C CNN "MPN"
@@
 F 0 "R87" V 5400 5800 50  0000 C CNN
 F 1 "2.2k" V 5600 5800 50  0000 C CNN
-F 2 "Resistor_SMD:R_0603_1608Metric_Pad1.05x0.95mm_HandSolder" H 5500 5800 50  0001 C CNN
+F 2 "Resistor_SMD:R_0603_1608Metric_Pad0.98x0.95mm_HandSolder" H 5500 5800 50  0001 C CNN
 F 3 "~" H 5500 5800 50  0001 C CNN
 F 4 "RC0603FR-072K2L" H 5500 5800 50  0001 C CNN "MPN"
@@
 F 0 "R85" H 4450 5900 50  0000 C CNN
 F 1 "5.1k" H 4450 5800 50  0000 C CNN
-F 2 "Resistor_SMD:R_0603_1608Metric_Pad1.05x0.95mm_HandSolder" H 4550 5900 50  0001 C CNN
+F 2 "Resistor_SMD:R_0603_1608Metric_Pad0.98x0.95mm_HandSolder" H 4550 5900 50  0001 C CNN
 F 3 "~" H 4550 5900 50  0001 C CNN
 F 4 "AC0603FR-135K1L" H 4550 5900 50  0001 C CNN "MPN"
@@
 F 0 "R88" H 7659 1746 50  0000 L CNN
 F 1 "2.2k" H 7659 1655 50  0000 L CNN
-F 2 "Resistor_SMD:R_0603_1608Metric_Pad1.05x0.95mm_HandSolder" H 7600 1700 50  0001 C CNN
+F 2 "Resistor_SMD:R_0603_1608Metric_Pad0.98x0.95mm_HandSolder" H 7600 1700 50  0001 C CNN
 F 3 "~" H 7600 1700 50  0001 C CNN
 F 4 "RC0603FR-072K2L" H 7600 1700 50  0001 C CNN "MPN"
@@
 F 0 "C60" H 6392 5696 50  0000 L CNN
 F 1 "10u" H 6392 5605 50  0000 L CNN
-F 2 "Capacitor_SMD:C_0805_2012Metric_Pad1.15x1.40mm_HandSolder" H 6300 5650 50  0001 C CNN
+F 2 "Capacitor_SMD:C_0805_2012Metric_Pad1.18x1.45mm_HandSolder" H 6300 5650 50  0001 C CNN
 F 3 "~" H 6300 5650 50  0001 C CNN
 F 4 "C0805C106K9PACTU" H 6300 5650 50  0001 C CNN "MPN"
@@
 F 0 "C62" H 6892 5696 50  0000 L CNN
 F 1 "10u" H 6892 5605 50  0000 L CNN
-F 2 "Capacitor_SMD:C_0805_2012Metric_Pad1.15x1.40mm_HandSolder" H 6800 5650 50  0001 C CNN
+F 2 "Capacitor_SMD:C_0805_2012Metric_Pad1.18x1.45mm_HandSolder" H 6800 5650 50  0001 C CNN
 F 3 "~" H 6800 5650 50  0001 C CNN
 F 4 "C0805C106K9PACTU" H 6800 5650 50  0001 C CNN "MPN"
@@
 F 0 "C59" H 4892 1746 50  0000 L CNN
 F 1 "10u" H 4892 1655 50  0000 L CNN
-F 2 "Capacitor_SMD:C_0805_2012Metric_Pad1.15x1.40mm_HandSolder" H 4800 1700 50  0001 C CNN
+F 2 "Capacitor_SMD:C_0805_2012Metric_Pad1.18x1.45mm_HandSolder" H 4800 1700 50  0001 C CNN
 F 3 "~" H 4800 1700 50  0001 C CNN
 F 4 "C0805C106K9PACTU" H 4800 1700 50  0001 C CNN "MPN"
