File: panel.kicad_pcb (KiCad board)
At the start: 4 copper layers, 0 parts

Commit message: Reference panel
Parts:
- added REF**: Fiducial_1.5mm_Mask4.5mm, Fiducial:Fiducial_1.5mm_Mask4.5mm, F.Cu at (236.2, 119.0)
- added REF**: Fiducial_1.5mm_Mask4.5mm, Fiducial:Fiducial_1.5mm_Mask4.5mm, F.Cu at (164.2, 273.8)
- added REF**: Fiducial_1.5mm_Mask4.5mm, Fiducial:Fiducial_1.5mm_Mask4.5mm, F.Cu at (236.2, 273.8)
- added Ref**: Mousebites_Panel_Single_5x2mm, grootvoet:Mousebites_Panel_Single_5x2mm, F.Cu at (234.2, 270.0)
- added Ref**: Mousebites_Panel_Double_5x5mm, grootvoet:Mousebites_Panel_Double_5x5mm, F.Cu at (146.2, 247.0)
- added Ref**: Mousebites_Panel_Double_5x5mm, grootvoet:Mousebites_Panel_Double_5x5mm, F.Cu at (146.2, 177.8)
- added Ref**: Mousebites_Panel_Double_4x2mm, grootvoet:Mousebites_Panel_Double_4x2mm, F.Cu at (216.2, 254.0)
- added Ref**: Mousebites_Panel_Double_4x2mm, grootvoet:Mousebites_Panel_Double_4x2mm, F.Cu at (216.2, 220.0)
- added Ref**: Mousebites_Panel_Double_4x2mm, grootvoet:Mousebites_Panel_Double_4x2mm, F.Cu at (162.2, 230.0)
- added Ref**: Mousebites_Panel_Double_4x2mm, grootvoet:Mousebites_Panel_Double_4x2mm, F.Cu at (196.2, 230.0)
- added Ref**: Mousebites_Panel_Double_4x2mm, grootvoet:Mousebites_Panel_Double_4x2mm, F.Cu at (162.2, 190.0)
- added Ref**: Mousebites_Panel_Double_4x2mm, grootvoet:Mousebites_Panel_Double_4x2mm, F.Cu at (196.2, 190.0)
- added Ref**: Mousebites_Panel_Double_4x2mm, grootvoet:Mousebites_Panel_Double_4x2mm, F.Cu at (216.2, 172.0)
- added Ref**: Mousebites_Panel_Double_5x7mm, grootvoet:Mousebites_Panel_Double_5x7mm, F.Cu at (216.2, 121.0)
- added Ref**: Mousebites_Panel_Double_4x2mm, grootvoet:Mousebites_Panel_Double_4x2mm, F.Cu at (234.2, 200.0)
- added Ref**: Mousebites_Panel_Double_5x7mm, grootvoet:Mousebites_Panel_Double_5x7mm, F.Cu at (216.2, 59.0)
- added Ref**: Mousebites_Panel_Single_5x2mm, grootvoet:Mousebites_Panel_Single_5x2mm, F.Cu at (234.2, 96.0)
- added Ref**: Mousebites_Panel_Single_5x2mm, grootvoet:Mousebites_Panel_Single_5x2mm, F.Cu at (238.2, 130.0)
- added Ref**: Mousebites_Panel_Double_5x8mm, grootvoet:Mousebites_Panel_Double_5x8mm, F.Cu at (149.2, 121.0)
- added Ref**: Mousebites_Panel_Double_5x8mm, grootvoet:Mousebites_Panel_Double_5x8mm, F.Cu at (149.2, 59.0)
- added Ref**: Mousebites_Panel_Double_4x2mm, grootvoet:Mousebites_Panel_Double_4x2mm, F.Cu at (132.2, 212.0)
- added Ref**: Mousebites_Panel_Double_4x2mm, grootvoet:Mousebites_Panel_Double_4x2mm, F.Cu at (92.2, 212.0)
- added Ref**: Mousebites_Panel_Double_4x2mm, grootvoet:Mousebites_Panel_Double_4x2mm, F.Cu at (196.2, 150.0)
- added Ref**: Mousebites_Panel_Double_4x2mm, grootvoet:Mousebites_Panel_Double_4x2mm, F.Cu at (162.2, 150.0)
- added Ref**: Mousebites_Panel_Double_4x2mm, grootvoet:Mousebites_Panel_Double_4x2mm, F.Cu at (132.2, 150.0)
- added Ref**: Mousebites_Panel_Single_5x2mm, grootvoet:Mousebites_Panel_Single_5x2mm, F.Cu at (196.2, 270.0)
- added Ref**: Mousebites_Panel_Double_4x2mm, grootvoet:Mousebites_Panel_Double_4x2mm, F.Cu at (92.2, 150.0)
- added Ref**: Mousebites_Panel_Double_4x2mm, grootvoet:Mousebites_Panel_Double_4x2mm, F.Cu at (200.2, 88.0)
- added Ref**: Mousebites_Panel_Double_4x2mm, grootvoet:Mousebites_Panel_Double_4x2mm, F.Cu at (92.2, 88.0)
- added Ref**: Mousebites_Panel_Double_4x2mm, grootvoet:Mousebites_Panel_Double_4x2mm, F.Cu at (160.2, 88.0)
- added Ref**: Mousebites_Panel_Double_4x2mm, grootvoet:Mousebites_Panel_Double_4x2mm, F.Cu at (132.2, 88.0)
- added Ref**: Mousebites_Panel_Single_5x2mm, grootvoet:Mousebites_Panel_Single_5x2mm, F.Cu at (162.2, 270.0)
- added Ref**: Mousebites_Panel_Single_5x2mm, grootvoet:Mousebites_Panel_Single_5x2mm, F.Cu at (238.2, 26.0)
- added Ref**: Mousebites_Panel_Single_5x2mm, grootvoet:Mousebites_Panel_Single_5x2mm, F.Cu at (201.2, 26.0)
- added Ref**: Mousebites_Panel_Single_5x2mm, grootvoet:Mousebites_Panel_Single_5x2mm, F.Cu at (164.2, 26.0)
- added Ref**: Mousebites_Panel_Single_5x2mm, grootvoet:Mousebites_Panel_Single_5x2mm, F.Cu at (133.2, 26.0)
- added Ref**: Mousebites_Panel_Single_5x2mm, grootvoet:Mousebites_Panel_Single_5x2mm, F.Cu at (96.2, 26.0)
Other:
- board outline added: 179 x 255 mm
- rule trace_min: 0.15 -> 0.2
