File: panel.kicad_pcb (KiCad board)
At the start: 4 copper layers, 179 x 255 mm, 37 parts

Commit message: Add layer info
Other:
- board text added: "Layer Info ===== Dwgs.User - Individual Board Outline Eco1.User - Router Cutout layer Edge.Cuts - Panel Outline"
