File: ADC_Frontend.sch (KiCad schematic (older format))
At the start: 22 parts, among them U3 THS4551

Commit message: Update pinout
Changed lines of the file:
@@
 $Descr A4 11693 8268
 encoding utf-8
-Sheet 4 9
+Sheet 3 9
 Title "Kleinvoet"
 Date "2020-06-11"
@@
 AR Path="/5EE5ECAD/5EE91C90/5F9B6C0C" Ref="R41"  Part="1"
 AR Path="/5EE5ECAD/5EE9492B/5F9B6C0C" Ref="R53"  Part="1"
-F 0 "R41" V 3204 4000 50  0000 C CNN
+F 0 "R17" V 3204 4000 50  0000 C CNN
 F 1 "310" V 3295 4000 50  0000 C CNN
 F 2 "Resistor_SMD:R_0603_1608Metric_Pad0.98x0.95mm_HandSolder" H 3400 4000 50  0001 C CNN
@@
 AR Path="/5EE5ECAD/5EE91C90/5F9B6FF8" Ref="R45"  Part="1"
 AR Path="/5EE5ECAD/5EE9492B/5F9B6FF8" Ref="R57"  Part="1"
-F 0 "R45" V 3954 4000 50  0000 C CNN
+F 0 "R21" V 3954 4000 50  0000 C CNN
 F 1 "330" V 4045 4000 50  0000 C CNN
 F 2 "Resistor_SMD:R_0603_1608Metric_Pad0.98x0.95mm_HandSolder" H 4150 4000 50  0001 C CNN
@@
 AR Path="/5EE5ECAD/5EE91C90/5F9B71F6" Ref="R47"  Part="1"
 AR Path="/5EE5ECAD/5EE9492B/5F9B71F6" Ref="R59"  Part="1"
-F 0 "R47" V 4654 3500 50  0000 C CNN
+F 0 "R23" V 4654 3500 50  0000 C CNN
 F 1 "360" V 4745 3500 50  0000 C CNN
 F 2 "Resistor_SMD:R_0603_1608Metric_Pad0.98x0.95mm_HandSolder" H 4850 3500 50  0001 C CNN
@@
 AR Path="/5EE5ECAD/5EE91C90/5F9B9E62" Ref="R49"  Part="1"
 AR Path="/5EE5ECAD/5EE9492B/5F9B9E62" Ref="R61"  Part="1"
-F 0 "R49" V 6096 4000 50  0000 C CNN
+F 0 "R25" V 6096 4000 50  0000 C CNN
 F 1 "15" V 6005 4000 50  0000 C CNN
 F 2 "Resistor_SMD:R_0603_1608Metric_Pad0.98x0.95mm_HandSolder" H 5900 4000 50  0001 C CNN
@@
 AR Path="/5EE5ECAD/5EE91C90/5F9BB14B" Ref="C72"  Part="1"
 AR Path="/5EE5ECAD/5EE9492B/5F9BB14B" Ref="C85"  Part="1"
-F 0 "C72" V 5429 4000 50  0000 C CNN
+F 0 "C38" V 5429 4000 50  0000 C CNN
 F 1 "3.9n" V 5338 4000 50  0000 C CNN
 F 2 "Capacitor_SMD:C_0603_1608Metric_Pad1.08x0.95mm_HandSolder" H 5200 4000 50  0001 C CNN
@@
 AR Path="/5EE5ECAD/5EE91C90/5F9BD251" Ref="C61"  Part="1"
 AR Path="/5EE5ECAD/5EE9492B/5F9BD251" Ref="C79"  Part="1"
-F 0 "C61" V 3171 3500 50  0000 C CNN
+F 0 "C26" V 3171 3500 50  0000 C CNN
 F 1 "220p" V 3262 3500 50  0000 C CNN
 F 2 "Capacitor_SMD:C_0603_1608Metric_Pad1.08x0.95mm_HandSolder" H 3400 3500 50  0001 C CNN
@@
 AR Path="/5EE5ECAD/5EE91C90/5F9DD374" Ref="R42"  Part="1"
 AR Path="/5EE5ECAD/5EE9492B/5F9DD374" Ref="R54"  Part="1"
-F 0 "R42" V 3596 5400 50  0000 C CNN
+F 0 "R18" V 3596 5400 50  0000 C CNN
 F 1 "310" V 3505 5400 50  0000 C CNN
 F 2 "Resistor_SMD:R_0603_1608Metric_Pad0.98x0.95mm_HandSolder" H 3400 5400 50  0001 C CNN
@@
 AR Path="/5EE5ECAD/5EE91C90/5F9DD37A" Ref="R46"  Part="1"
 AR Path="/5EE5ECAD/5EE9492B/5F9DD37A" Ref="R58"  Part="1"
-F 0 "R46" V 4346 5400 50  0000 C CNN
+F 0 "R22" V 4346 5400 50  0000 C CNN
 F 1 "330" V 4255 5400 50  0000 C CNN
 F 2 "Resistor_SMD:R_0603_1608Metric_Pad0.98x0.95mm_HandSolder" H 4150 5400 50  0001 C CNN
@@
 AR Path="/5EE5ECAD/5EE91C90/5F9DD380" Ref="R48"  Part="1"
 AR Path="/5EE5ECAD/5EE9492B/5F9DD380" Ref="R60"  Part="1"
-F 0 "R48" V 5046 5900 50  0000 C CNN
+F 0 "R24" V 5046 5900 50  0000 C CNN
 F 1 "360" V 4955 5900 50  0000 C CNN
 F 2 "Resistor_SMD:R_0603_1608Metric_Pad0.98x0.95mm_HandSolder" H 4850 5900 50  0001 C CNN
@@
 AR Path="/5EE5ECAD/5EE91C90/5F9DD386" Ref="U5"  Part="1"
 AR Path="/5EE5ECAD/5EE9492B/5F9DD386" Ref="U6"  Part="1"
-F 0 "U5" H 5467 4261 50  0000 C CNN
+F 0 "U3" H 5467 4261 50  0000 C CNN
 F 1 "THS4551" H 5450 4400 50  0000 C CNN
 F 2 "grootvoet:WQFN-10_RUN" H 5400 4450 50  0001 C CNN
@@
 AR Path="/5EE5ECAD/5EE91C90/5F9DD398" Ref="R50"  Part="1"
 AR Path="/5EE5ECAD/5EE9492B/5F9DD398" Ref="R62"  Part="1"
-F 0 "R50" V 6096 5400 50  0000 C CNN
+F 0 "R26" V 6096 5400 50  0000 C CNN
 F 1 "15" V 6005 5400 50  0000 C CNN
 F 2 "Resistor_SMD:R_0603_1608Metric_Pad0.98x0.95mm_HandSolder" H 5900 5400 50  0001 C CNN
@@
 AR Path="/5EE5ECAD/5EE91C90/5F9DD39E" Ref="C73"  Part="1"
 AR Path="/5EE5ECAD/5EE9492B/5F9DD39E" Ref="C86"  Part="1"
-F 0 "C73" V 5429 5400 50  0000 C CNN
+F 0 "C39" V 5429 5400 50  0000 C CNN
 F 1 "3.9n" V 5050 5400 50  0000 C CNN
 F 2 "Capacitor_SMD:C_0603_1608Metric_Pad1.08x0.95mm_HandSolder" H 5200 5400 50  0001 C CNN
@@
 AR Path="/5EE5ECAD/5EE91C90/5F9DD3A4" Ref="C69"  Part="1"
 AR Path="/5EE5ECAD/5EE9492B/5F9DD3A4" Ref="C82"  Part="1"
-F 0 "C69" H 4308 4654 50  0000 R CNN
+F 0 "C35" H 4308 4654 50  0000 R CNN
 F 1 "OPEN" H 4308 4745 50  0000 R CNN
 F 2 "Capacitor_SMD:C_0603_1608Metric_Pad1.08x0.95mm_HandSolder" H 4400 4700 50  0001 C CNN
@@
 AR Path="/5EE5ECAD/5EE91C90/5F9DD3AA" Ref="C68"  Part="1"
 AR Path="/5EE5ECAD/5EE9492B/5F9DD3AA" Ref="C81"  Part="1"
-F 0 "C68" H 3658 4654 50  0000 R CNN
+F 0 "C34" H 3658 4654 50  0000 R CNN
 F 1 "27n" H 3658 4745 50  0000 R CNN
 F 2 "Capacitor_SMD:C_0603_1608Metric_Pad1.08x0.95mm_HandSolder" H 3750 4700 50  0001 C CNN
@@
 AR Path="/5EE5ECAD/5EE91C90/5F9DD3B0" Ref="C67"  Part="1"
 AR Path="/5EE5ECAD/5EE9492B/5F9DD3B0" Ref="C80"  Part="1"
-F 0 "C67" V 3629 5900 50  0000 C CNN
+F 0 "C27" V 3629 5900 50  0000 C CNN
 F 1 "220p" V 3538 5900 50  0000 C CNN
 F 2 "Capacitor_SMD:C_0603_1608Metric_Pad1.08x0.95mm_HandSolder" H 3400 5900 50  0001 C CNN
@@
 AR Path="/5EE5ECAD/5EE91C90/5F9E915F" Ref="C77"  Part="1"
 AR Path="/5EE5ECAD/5EE9492B/5F9E915F" Ref="C90"  Part="1"
-F 0 "C77" H 7092 4746 50  0000 L CNN
+F 0 "C43" H 7092 4746 50  0000 L CNN
 F 1 "100n" H 7092 4655 50  0000 L CNN
 F 2 "Capacitor_SMD:C_0603_1608Metric_Pad1.08x0.95mm_HandSolder" H 7000 4700 50  0001 C CNN
@@
 AR Path="/5EE5ECAD/5EE91C90/5F9EA7A7" Ref="R51"  Part="1"
 AR Path="/5EE5ECAD/5EE9492B/5F9EA7A7" Ref="R63"  Part="1"
-F 0 "R51" V 6596 4000 50  0000 C CNN
+F 0 "R27" V 6596 4000 50  0000 C CNN
 F 1 "47" V 6505 4000 50  0000 C CNN
 F 2 "Resistor_SMD:R_0603_1608Metric_Pad0.98x0.95mm_HandSolder" H 6400 4000 50  0001 C CNN
@@
 AR Path="/5EE5ECAD/5EE91C90/5F9EB4CC" Ref="R52"  Part="1"
 AR Path="/5EE5ECAD/5EE9492B/5F9EB4CC" Ref="R64"  Part="1"
-F 0 "R52" V 6646 5400 50  0000 C CNN
+F 0 "R28" V 6646 5400 50  0000 C CNN
 F 1 "47" V 6555 5400 50  0000 C CNN
 F 2 "Resistor_SMD:R_0603_1608Metric_Pad0.98x0.95mm_HandSolder" H 6450 5400 50  0001 C CNN
@@
 AR Path="/5EE5ECAD/5EE91C90/5F9EC0A0" Ref="C76"  Part="1"
 AR Path="/5EE5ECAD/5EE9492B/5F9EC0A0" Ref="C89"  Part="1"
-F 0 "C76" H 7092 3746 50  0000 L CNN
+F 0 "C42" H 7092 3746 50  0000 L CNN
 F 1 "10n" H 7092 3655 50  0000 L CNN
 F 2 "Capacitor_SMD:C_0603_1608Metric_Pad1.08x0.95mm_HandSolder" H 7000 3700 50  0001 C CNN
@@
 AR Path="/5EE5ECAD/5EE91C90/5F9EC966" Ref="C78"  Part="1"
 AR Path="/5EE5ECAD/5EE9492B/5F9EC966" Ref="C91"  Part="1"
-F 0 "C78" H 7092 5746 50  0000 L CNN
+F 0 "C44" H 7092 5746 50  0000 L CNN
 F 1 "10n" H 7092 5655 50  0000 L CNN
 F 2 "Capacitor_SMD:C_0603_1608Metric_Pad1.08x0.95mm_HandSolder" H 7000 5700 50  0001 C CNN
@@
 AR Path="/5EE5ECAD/5EE91C90/5F9F8674" Ref="C71"  Part="1"
 AR Path="/5EE5ECAD/5EE9492B/5F9F8674" Ref="C84"  Part="1"
-F 0 "C71" H 4908 2204 50  0000 R CNN
+F 0 "C37" H 4908 2204 50  0000 R CNN
 F 1 "100n" H 4908 2295 50  0000 R CNN
 F 2 "Capacitor_SMD:C_0603_1608Metric_Pad1.08x0.95mm_HandSolder" H 5000 2250 50  0001 C CNN
@@
 AR Path="/5EE5ECAD/5EE91C90/5FA07028" Ref="C74"  Part="1"
 AR Path="/5EE5ECAD/5EE9492B/5FA07028" Ref="C87"  Part="1"
-F 0 "C74" H 5558 2104 50  0000 R CNN
+F 0 "C40" H 5558 2104 50  0000 R CNN
 F 1 "100n" H 5558 2195 50  0000 R CNN
 F 2 "Capacitor_SMD:C_0603_1608Metric_Pad1.08x0.95mm_HandSolder" H 5650 2150 50  0001 C CNN

Commit message: BOM
Parts:
- C26, C27: MPN (none) -> C0603C221J5GACTU; Mfr. (none) -> KEMET
- C34: MPN (none) -> CC0603JRX7R9BB273; Mfr. (none) -> Yageo
- C37, C40, C43: MPN (none) -> C0603C104M5RACTU; Mfr. (none) -> KEMET
- C38, C39: MPN (none) -> CC0603JRX7R9BB392; Mfr. (none) -> Yageo
- C42, C44: MPN (none) -> C0603C103J5RACTU; Mfr. (none) -> KEMET
- R17, R18: MPN (none) -> ERJ-3EKF3090V; Mfr. (none) -> Panasonic
- R21, R22: MPN (none) -> ERJ-3EKF3300V; Mfr. (none) -> Panasonic
- R23, R24: MPN (none) -> ERJ-3EKF3600V; Mfr. (none) -> Panasonic
- R25, R26: MPN (none) -> ERJ-3EKF15R0V; Mfr. (none) -> Panasonic
- R27, R28: MPN (none) -> ERJ-3EKF47R0V; Mfr. (none) -> Panasonic
- U3: MPN (none) -> THS4551IRUNR; Mfr. (none) -> Texas Instruments
Changed lines of the file:
@@
 F 2 "Resistor_SMD:R_0603_1608Metric_Pad0.98x0.95mm_HandSolder" H 3400 4000 50  0001 C CNN
 F 3 "~" H 3400 4000 50  0001 C CNN
+F 4 "ERJ-3EKF3090V" H 3400 4000 50  0001 C CNN "MPN"
+F 5 "Panasonic" H 3400 4000 50  0001 C CNN "Mfr."
 	1    3400 4000
 	0    1    1    0
@@
 F 2 "Resistor_SMD:R_0603_1608Metric_Pad0.98x0.95mm_HandSolder" H 4150 4000 50  0001 C CNN
 F 3 "~" H 4150 4000 50  0001 C CNN
+F 4 "ERJ-3EKF3300V" H 4150 4000 50  0001 C CNN "MPN"
+F 5 "Panasonic" H 4150 4000 50  0001 C CNN "Mfr."
 	1    4150 4000
 	0    1    1    0
@@
 F 2 "Resistor_SMD:R_0603_1608Metric_Pad0.98x0.95mm_HandSolder" H 4850 3500 50  0001 C CNN
 F 3 "~" H 4850 3500 50  0001 C CNN
+F 4 "ERJ-3EKF3600V" H 4850 3500 50  0001 C CNN "MPN"
+F 5 "Panasonic" H 4850 3500 50  0001 C CNN "Mfr."
 	1    4850 3500
 	0    1    1    0
@@
 F 2 "Resistor_SMD:R_0603_1608Metric_Pad0.98x0.95mm_HandSolder" H 5900 4000 50  0001 C CNN
 F 3 "~" H 5900 4000 50  0001 C CNN
+F 4 "ERJ-3EKF15R0V" H 5900 4000 50  0001 C CNN "MPN"
+F 5 "Panasonic" H 5900 4000 50  0001 C CNN "Mfr."
 	1    5900 4000
 	0    1    -1   0
@@
 F 2 "Capacitor_SMD:C_0603_1608Metric_Pad1.08x0.95mm_HandSolder" H 5200 4000 50  0001 C CNN
 F 3 "~" H 5200 4000 50  0001 C CNN
+F 4 "CC0603JRX7R9BB392" H 5200 4000 50  0001 C CNN "MPN"
+F 5 "Yageo" H 5200 4000 50  0001 C CNN "Mfr."
 	1    5200 4000
 	0    1    -1   0
@@
 F 2 "Capacitor_SMD:C_0603_1608Metric_Pad1.08x0.95mm_HandSolder" H 3400 3500 50  0001 C CNN
 F 3 "~" H 3400 3500 50  0001 C CNN
+F 4 "C0603C221J5GACTU" H 3400 3500 50  0001 C CNN "MPN"
+F 5 "KEMET" H 3400 3500 50  0001 C CNN "Mfr."
 	1    3400 3500
 	0    1    1    0
@@
 F 2 "Resistor_SMD:R_0603_1608Metric_Pad0.98x0.95mm_HandSolder" H 3400 5400 50  0001 C CNN
 F 3 "~" H 3400 5400 50  0001 C CNN
+F 4 "ERJ-3EKF3090V" H 3400 5400 50  0001 C CNN "MPN"
+F 5 "Panasonic" H 3400 5400 50  0001 C CNN "Mfr."
 	1    3400 5400
 	0    1    -1   0
@@
 F 2 "Resistor_SMD:R_0603_1608Metric_Pad0.98x0.95mm_HandSolder" H 4150 5400 50  0001 C CNN
 F 3 "~" H 4150 5400 50  0001 C CNN
+F 4 "ERJ-3EKF3300V" H 4150 5400 50  0001 C CNN "MPN"
+F 5 "Panasonic" H 4150 5400 50  0001 C CNN "Mfr."
 	1    4150 5400
 	0    1    -1   0
@@
 F 2 "Resistor_SMD:R_0603_1608Metric_Pad0.98x0.95mm_HandSolder" H 4850 5900 50  0001 C CNN
 F 3 "~" H 4850 5900 50  0001 C CNN
+F 4 "ERJ-3EKF3600V" H 4850 5900 50  0001 C CNN "MPN"
+F 5 "Panasonic" H 4850 5900 50  0001 C CNN "Mfr."
 	1    4850 5900
 	0    1    -1   0
@@
 F 2 "grootvoet:WQFN-10_RUN" H 5400 4450 50  0001 C CNN
 F 3 "" H 5400 4450 50  0001 C CNN
+F 4 "THS4551IRUNR" H 5000 4700 50  0001 C CNN "MPN"
+F 5 "Texas Instruments" H 5000 4700 50  0001 C CNN "Mfr."
 	1    5000 4700
 	1    0    0    -1
@@
 F 2 "Resistor_SMD:R_0603_1608Metric_Pad0.98x0.95mm_HandSolder" H 5900 5400 50  0001 C CNN
 F 3 "~" H 5900 5400 50  0001 C CNN
+F 4 "ERJ-3EKF15R0V" H 5900 5400 50  0001 C CNN "MPN"
+F 5 "Panasonic" H 5900 5400 50  0001 C CNN "Mfr."
 	1    5900 5400
 	0    1    -1   0
@@
 F 2 "Capacitor_SMD:C_0603_1608Metric_Pad1.08x0.95mm_HandSolder" H 5200 5400 50  0001 C CNN
 F 3 "~" H 5200 5400 50  0001 C CNN
+F 4 "CC0603JRX7R9BB392" H 5200 5400 50  0001 C CNN "MPN"
+F 5 "Yageo" H 5200 5400 50  0001 C CNN "Mfr."
 	1    5200 5400
 	0    1    -1   0
@@
 F 2 "Capacitor_SMD:C_0603_1608Metric_Pad1.08x0.95mm_HandSolder" H 3750 4700 50  0001 C CNN
 F 3 "~" H 3750 4700 50  0001 C CNN
+F 4 "CC0603JRX7R9BB273" H 3750 4700 50  0001 C CNN "MPN"
+F 5 "Yageo" H 3750 4700 50  0001 C CNN "Mfr."
 	1    3750 4700
 	1    0    0    1
@@
 F 2 "Capacitor_SMD:C_0603_1608Metric_Pad1.08x0.95mm_HandSolder" H 3400 5900 50  0001 C CNN
 F 3 "~" H 3400 5900 50  0001 C CNN
+F 4 "C0603C221J5GACTU" H 3400 5900 50  0001 C CNN "MPN"
+F 5 "KEMET" H 3400 5900 50  0001 C CNN "Mfr."
 	1    3400 5900
 	0    1    -1   0
@@
 AR Path="/5EE5ECAD/5EE91C90/5F9B8E94" Ref="#PWR0165"  Part="1"
 AR Path="/5EE5ECAD/5EE9492B/5F9B8E94" Ref="#PWR0177"  Part="1"
-F 0 "#PWR0165" H 5200 4800 50  0001 C CNN
+F 0 "#PWR062" H 5200 4800 50  0001 C CNN
 F 1 "GND" H 5205 4877 50  0000 C CNN
 F 2 "" H 5200 5050 50  0001 C CNN
@@
 AR Path="/5EE5ECAD/5EE91C90/5F9E515B" Ref="#PWR0160"  Part="1"
 AR Path="/5EE5ECAD/5EE9492B/5F9E515B" Ref="#PWR0172"  Part="1"
-F 0 "#PWR0160" H 3300 3250 50  0001 C CNN
+F 0 "#PWR055" H 3300 3250 50  0001 C CNN
 F 1 "GND" V 3305 3372 50  0000 R CNN
 F 2 "" H 3300 3500 50  0001 C CNN
@@
 AR Path="/5EE5ECAD/5EE91C90/5F9E5687" Ref="#PWR0161"  Part="1"
 AR Path="/5EE5ECAD/5EE9492B/5F9E5687" Ref="#PWR0173"  Part="1"
-F 0 "#PWR0161" H 3300 5650 50  0001 C CNN
+F 0 "#PWR056" H 3300 5650 50  0001 C CNN
 F 1 "GND" V 3305 5772 50  0000 R CNN
 F 2 "" H 3300 5900 50  0001 C CNN
@@
 F 2 "Capacitor_SMD:C_0603_1608Metric_Pad1.08x0.95mm_HandSolder" H 7000 4700 50  0001 C CNN
 F 3 "~" H 7000 4700 50  0001 C CNN
+F 4 "C0603C104M5RACTU" H 7000 4700 50  0001 C CNN "MPN"
+F 5 "KEMET" H 7000 4700 50  0001 C CNN "Mfr."
 	1    7000 4700
 	1    0    0    -1
@@
 F 2 "Resistor_SMD:R_0603_1608Metric_Pad0.98x0.95mm_HandSolder" H 6400 4000 50  0001 C CNN
 F 3 "~" H 6400 4000 50  0001 C CNN
+F 4 "ERJ-3EKF47R0V" H 6400 4000 50  0001 C CNN "MPN"
+F 5 "Panasonic" H 6400 4000 50  0001 C CNN "Mfr."
 	1    6400 4000
 	0    1    -1   0
@@
 F 2 "Resistor_SMD:R_0603_1608Metric_Pad0.98x0.95mm_HandSolder" H 6450 5400 50  0001 C CNN
 F 3 "~" H 6450 5400 50  0001 C CNN
+F 4 "ERJ-3EKF47R0V" H 6450 5400 50  0001 C CNN "MPN"
+F 5 "Panasonic" H 6450 5400 50  0001 C CNN "Mfr."
 	1    6450 5400
 	0    1    -1   0
@@
 F 2 "Capacitor_SMD:C_0603_1608Metric_Pad1.08x0.95mm_HandSolder" H 7000 3700 50  0001 C CNN
 F 3 "~" H 7000 3700 50  0001 C CNN
+F 4 "C0603C103J5RACTU" H 7000 3700 50  0001 C CNN "MPN"
+F 5 "KEMET" H 7000 3700 50  0001 C CNN "Mfr."
 	1    7000 3700
 	1    0    0    -1
@@
 F 2 "Capacitor_SMD:C_0603_1608Metric_Pad1.08x0.95mm_HandSolder" H 7000 5700 50  0001 C CNN
 F 3 "~" H 7000 5700 50  0001 C CNN
+F 4 "C0603C103J5RACTU" H 7000 5700 50  0001 C CNN "MPN"
+F 5 "KEMET" H 7000 5700 50  0001 C CNN "Mfr."
 	1    7000 5700
 	1    0    0    -1
@@
 AR Path="/5EE5ECAD/5EE91C90/5F9ED440" Ref="#PWR0171"  Part="1"
 AR Path="/5EE5ECAD/5EE9492B/5F9ED440" Ref="#PWR0183"  Part="1"
-F 0 "#PWR0171" H 7000 5550 50  0001 C CNN
+F 0 "#PWR072" H 7000 5550 50  0001 C CNN
 F 1 "GND" H 7005 5627 50  0000 C CNN
 F 2 "" H 7000 5800 50  0001 C CNN
@@
 AR Path="/5EE5ECAD/5EE91C90/5F9ED994" Ref="#PWR0170"  Part="1"
 AR Path="/5EE5ECAD/5EE9492B/5F9ED994" Ref="#PWR0182"  Part="1"
-F 0 "#PWR0170" H 7000 3350 50  0001 C CNN
+F 0 "#PWR070" H 7000 3350 50  0001 C CNN
 F 1 "GND" H 7005 3427 50  0000 C CNN
 F 2 "" H 7000 3600 50  0001 C CNN
@@
 F 2 "Capacitor_SMD:C_0603_1608Metric_Pad1.08x0.95mm_HandSolder" H 5000 2250 50  0001 C CNN
 F 3 "~" H 5000 2250 50  0001 C CNN
+F 4 "C0603C104M5RACTU" H 5000 2250 50  0001 C CNN "MPN"
+F 5 "KEMET" H 5000 2250 50  0001 C CNN "Mfr."
 	1    5000 2250
 	1    0    0    1
@@
 F 2 "Capacitor_SMD:C_0603_1608Metric_Pad1.08x0.95mm_HandSolder" H 5650 2150 50  0001 C CNN
 F 3 "~" H 5650 2150 50  0001 C CNN
+F 4 "C0603C104M5RACTU" H 5650 2150 50  0001 C CNN "MPN"
+F 5 "KEMET" H 5650 2150 50  0001 C CNN "Mfr."
 	1    5650 2150
 	1    0    0    1
@@
 AR Path="/5EE5ECAD/5EE91C90/5FA077A0" Ref="#PWR0167"  Part="1"
 AR Path="/5EE5ECAD/5EE9492B/5FA077A0" Ref="#PWR0179"  Part="1"
-F 0 "#PWR0167" H 5650 2000 50  0001 C CNN
+F 0 "#PWR064" H 5650 2000 50  0001 C CNN
 F 1 "GND" H 5655 2077 50  0000 C CNN
 F 2 "" H 5650 2250 50  0001 C CNN
@@
 AR Path="/5EE5ECAD/5EE91C90/5FBFEE2A" Ref="#PWR0148"  Part="1"
 AR Path="/5EE5ECAD/5EE62BAF/5FBFEE2A" Ref="#PWR0147"  Part="1"
-F 0 "#PWR0148" H 5350 4300 50  0001 C CNN
+F 0 "#PWR0147" H 5350 4300 50  0001 C CNN
 F 1 "+3.3VADC" H 5215 4523 50  0000 C CNN
 F 2 "" H 5200 4350 50  0001 C CNN
@@
 AR Path="/5EE5ECAD/5EE91C90/5F9FA478" Ref="#PWR0163"  Part="1"
 AR Path="/5EE5ECAD/5EE9492B/5F9FA478" Ref="#PWR0175"  Part="1"
-F 0 "#PWR0163" H 5000 2150 50  0001 C CNN
+F 0 "#PWR058" H 5000 2150 50  0001 C CNN
 F 1 "GND" H 5005 2227 50  0000 C CNN
 F 2 "" H 5000 2400 50  0001 C CNN
@@
 AR Path="/5EE5ECAD/5EE91C90/5FC930A6" Ref="#PWR066"  Part="1"
 AR Path="/5EE5ECAD/5EE62BAF/5FC930A6" Ref="#PWR063"  Part="1"
-F 0 "#PWR066" H 5800 2000 50  0001 C CNN
+F 0 "#PWR063" H 5800 2000 50  0001 C CNN
 F 1 "+3.3VADC" H 5665 2223 50  0000 C CNN
 F 2 "" H 5650 2050 50  0001 C CNN
