File: buffer.kicad_sch (KiCad schematic)
At the start: 35 parts, among them U1501 OPA1662AIDGKRQ1, U1502 OPA2387

Commit message: (sch) change passives to 0402
Parts:
- C1504, C1505, C1506: MPN (none) -> C0603C105K8RACTU; Mfr. (none) -> KEMET
- R1512, R1513, R1514, R1517, R1518, R1519, R1521: footprint Resistor_SMD:R_0603_1608Metric_Pad0.98x0.95mm_HandSolder -> Resistor_SMD:R_0402_1005Metric; MPN (none) -> RT0402FRE071KL; Mfr. Panasonic -> Yageo
- R1516, R1522, R1523: footprint Resistor_SMD:R_0603_1608Metric_Pad0.98x0.95mm_HandSolder -> Resistor_SMD:R_0402_1005Metric; MPN (none) -> RT0402FRE07100KL; Mfr. Panasonic -> Yageo
Changed lines of the file:
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@@
       (effects (font (size 1.27 1.27)) (justify left))
     )
-    (property "Footprint" "Resistor_SMD:R_0603_1608Metric_Pad0.98x0.95mm_HandSolder" (at 233.68 85.725 0)
+    (property "Footprint" "Resistor_SMD:R_0402_1005Metric" (at 233.68 85.725 0)
       (effects (font (size 1.27 1.27)) hide)
     )
@@
       (effects (font (size 1.27 1.27)) hide)
     )
-    (property "MPN" "" (at 233.68 85.725 0)
-      (effects (font (size 1.27 1.27)) hide)
-    )
-    (property "Mfr." "Panasonic" (at 233.68 85.725 0)
+    (property "MPN" "RT0402FRE07100KL" (at 233.68 85.725 0)
+      (effects (font (size 1.27 1.27)) hide)
+    )
+    (property "Mfr." "Yageo" (at 233.68 85.725 0)
       (effects (font (size 1.27 1.27)) hide)
     )
@@
       (effects (font (size 1.27 1.27)) hide)
     )
+    (property "MPN" "C0603C105K8RACTU" (at 152.4 77.47 0)
+      (effects (font (size 1.27 1.27)) hide)
+    )
+    (property "Mfr." "KEMET" (at 152.4 77.47 0)
+      (effects (font (size 1.27 1.27)) hide)
+    )
     (pin "1")
     (pin "2")
@@
       (effects (font (size 1.27 1.27)) hide)
     )
+    (property "MPN" "C0603C105K8RACTU" (at 150.495 42.545 0)
+      (effects (font (size 1.27 1.27)) hide)
+    )
+    (property "Mfr." "KEMET" (at 150.495 42.545 0)
+      (effects (font (size 1.27 1.27)) hide)
+    )
     (pin "1")
     (pin "2")
@@
       (effects (font (size 1.27 1.27)) (justify left))
     )
-    (property "Footprint" "Resistor_SMD:R_0603_1608Metric_Pad0.98x0.95mm_HandSolder" (at 198.755 47.625 0)
+    (property "Footprint" "Resistor_SMD:R_0402_1005Metric" (at 198.755 47.625 0)
       (effects (font (size 1.27 1.27)) hide)
     )
@@
       (effects (font (size 1.27 1.27)) hide)
     )
-    (property "MPN" "" (at 198.755 47.625 0)
-      (effects (font (size 1.27 1.27)) hide)
-    )
-    (property "Mfr." "Panasonic" (at 198.755 47.625 0)
+    (property "MPN" "RT0402FRE071KL" (at 198.755 47.625 0)
+      (effects (font (size 1.27 1.27)) hide)
+    )
+    (property "Mfr." "Yageo" (at 198.755 47.625 0)
       (effects (font (size 1.27 1.27)) hide)
     )
@@
       (effects (font (size 1.27 1.27)) (justify left))
     )
-    (property "Footprint" "Resistor_SMD:R_0603_1608Metric_Pad0.98x0.95mm_HandSolder" (at 198.12 38.1 0)
+    (property "Footprint" "Resistor_SMD:R_0402_1005Metric" (at 198.12 38.1 0)
       (effects (font (size 1.27 1.27)) hide)
     )
@@
       (effects (font (size 1.27 1.27)) hide)
     )
-    (property "MPN" "" (at 198.12 38.1 0)
-      (effects (font (size 1.27 1.27)) hide)
-    )
-    (property "Mfr." "Panasonic" (at 198.12 38.1 0)
+    (property "MPN" "RT0402FRE071KL" (at 198.12 38.1 0)
+      (effects (font (size 1.27 1.27)) hide)
+    )
+    (property "Mfr." "Yageo" (at 198.12 38.1 0)
       (effects (font (size 1.27 1.27)) hide)
     )
@@
       (effects (font (size 1.27 1.27)) (justify left))
     )
-    (property "Footprint" "Resistor_SMD:R_0603_1608Metric_Pad0.98x0.95mm_HandSolder" (at 76.2 50.8 0)
+    (property "Footprint" "Resistor_SMD:R_0402_1005Metric" (at 76.2 50.8 0)
       (effects (font (size 1.27 1.27)) hide)
     )
@@
       (effects (font (size 1.27 1.27)) hide)
     )
-    (property "MPN" "" (at 76.2 50.8 0)
-      (effects (font (size 1.27 1.27)) hide)
-    )
-    (property "Mfr." "Panasonic" (at 76.2 50.8 0)
+    (property "MPN" "RT0402FRE071KL" (at 76.2 50.8 0)
+      (effects (font (size 1.27 1.27)) hide)
+    )
+    (property "Mfr." "Yageo" (at 76.2 50.8 0)
       (effects (font (size 1.27 1.27)) hide)
     )
@@
       (effects (font (size 1.27 1.27)) (justify left))
     )
-    (property "Footprint" "Resistor_SMD:R_0603_1608Metric_Pad0.98x0.95mm_HandSolder" (at 213.36 26.035 0)
+    (property "Footprint" "Resistor_SMD:R_0402_1005Metric" (at 213.36 26.035 0)
       (effects (font (size 1.27 1.27)) hide)
     )
@@
       (effects (font (size 1.27 1.27)) hide)
     )
-    (property "MPN" "" (at 213.36 26.035 0)
-      (effects (font (size 1.27 1.27)) hide)
-    )
-    (property "Mfr." "Panasonic" (at 213.36 26.035 0)
+    (property "MPN" "RT0402FRE071KL" (at 213.36 26.035 0)
+      (effects (font (size 1.27 1.27)) hide)
+    )
+    (property "Mfr." "Yageo" (at 213.36 26.035 0)
       (effects (font (size 1.27 1.27)) hide)
     )
@@
       (effects (font (size 1.27 1.27)) hide)
     )
+    (property "MPN" "C0603C105K8RACTU" (at 207.645 67.31 0)
+      (effects (font (size 1.27 1.27)) hide)
+    )
+    (property "Mfr." "KEMET" (at 207.645 67.31 0)
+      (effects (font (size 1.27 1.27)) hide)
+    )
     (pin "1")
     (pin "2")
@@
       (effects (font (size 1.27 1.27)) (justify left))
     )
-    (property "Footprint" "Resistor_SMD:R_0603_1608Metric_Pad0.98x0.95mm_HandSolder" (at 95.25 33.02 0)
+    (property "Footprint" "Resistor_SMD:R_0402_1005Metric" (at 95.25 33.02 0)
       (effects (font (size 1.27 1.27)) hide)
     )
@@
       (effects (font (size 1.27 1.27)) hide)
     )
-    (property "MPN" "" (at 95.25 33.02 0)
-      (effects (font (size 1.27 1.27)) hide)
-    )
-    (property "Mfr." "Panasonic" (at 95.25 33.02 0)
+    (property "MPN" "RT0402FRE071KL" (at 95.25 33.02 0)
+      (effects (font (size 1.27 1.27)) hide)
+    )
+    (property "Mfr." "Yageo" (at 95.25 33.02 0)
       (effects (font (size 1.27 1.27)) hide)
     )
@@
       (effects (font (size 1.27 1.27)) (justify left))
     )
-    (property "Footprint" "Resistor_SMD:R_0603_1608Metric_Pad0.98x0.95mm_HandSolder" (at 233.68 93.345 0)
+    (property "Footprint" "Resistor_SMD:R_0402_1005Metric" (at 233.68 93.345 0)
       (effects (font (size 1.27 1.27)) hide)
     )
@@
       (effects (font (size 1.27 1.27)) hide)
     )
-    (property "MPN" "" (at 233.68 93.345 0)
-      (effects (font (size 1.27 1.27)) hide)
-    )
-    (property "Mfr." "Panasonic" (at 233.68 93.345 0)
+    (property "MPN" "RT0402FRE07100KL" (at 233.68 93.345 0)
+      (effects (font (size 1.27 1.27)) hide)
+    )
+    (property "Mfr." "Yageo" (at 233.68 93.345 0)
       (effects (font (size 1.27 1.27)) hide)
     )
@@
       (effects (font (size 1.27 1.27)) (justify left))
     )
-    (property "Footprint" "Resistor_SMD:R_0603_1608Metric_Pad0.98x0.95mm_HandSolder" (at 80.01 56.515 0)
+    (property "Footprint" "Resistor_SMD:R_0402_1005Metric" (at 80.01 56.515 0)
       (effects (font (size 1.27 1.27)) hide)
     )
@@
       (effects (font (size 1.27 1.27)) hide)
     )
-    (property "MPN" "" (at 80.01 56.515 0)
-      (effects (font (size 1.27 1.27)) hide)
-    )
-    (property "Mfr." "Panasonic" (at 80.01 56.515 0)
+    (property "MPN" "RT0402FRE071KL" (at 80.01 56.515 0)
+      (effects (font (size 1.27 1.27)) hide)
+    )
+    (property "Mfr." "Yageo" (at 80.01 56.515 0)
       (effects (font (size 1.27 1.27)) hide)
     )
@@
       (effects (font (size 1.27 1.27)) (justify left))
     )
-    (property "Footprint" "Resistor_SMD:R_0603_1608Metric_Pad0.98x0.95mm_HandSolder" (at 113.03 99.695 0)
+    (property "Footprint" "Resistor_SMD:R_0402_1005Metric" (at 113.03 99.695 0)
       (effects (font (size 1.27 1.27)) hide)
     )
@@
       (effects (font (size 1.27 1.27)) hide)
     )
-    (property "MPN" "" (at 113.03 99.695 0)
-      (effects (font (size 1.27 1.27)) hide)
-    )
-    (property "Mfr." "Panasonic" (at 113.03 99.695 0)
+    (property "MPN" "RT0402FRE07100KL" (at 113.03 99.695 0)
+      (effects (font (size 1.27 1.27)) hide)
+    )
+    (property "Mfr." "Yageo" (at 113.03 99.695 0)
       (effects (font (size 1.27 1.27)) hide)
     )
@@
       (effects (font (size 1.27 1.27)) (justify left))
     )
-    (property "Footprint" "Resistor_SMD:R_0603_1608Metric_Pad0.98x0.95mm_HandSolder" (at 198.755 43.18 0)
+    (property "Footprint" "Resistor_SMD:R_0402_1005Metric" (at 198.755 43.18 0)
       (effects (font (size 1.27 1.27)) hide)
     )
@@
       (effects (font (size 1.27 1.27)) hide)
     )
-    (property "MPN" "" (at 198.755 43.18 0)
-      (effects (font (size 1.27 1.27)) hide)
-    )
-    (property "Mfr." "Panasonic" (at 198.755 43.18 0)
-      (effects (font (size 1.27 1.27)) hide)
-    )
+    (property "MPN" "RT0402FRE071KL" (at 198.755 43.18 0)
+      (effects (font (size 1.27 1.27)) hide)
+    )
+    (property "Mfr." "Yageo" (at 198.755 43.18 0)
+      (effects (font (size 1.27 1.27)) hide)
+    )
