File: compass.kicad_sch (KiCad schematic)
At the start: 6 parts, among them U6 LIS2MDL

Commit message: (bc) changes for the day
Parts:
- C2, C47, CB1, R1: now not fitted
- U6: now not fitted; now left out of the parts list
Changed lines of the file:
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@@
   )
   (symbol (lib_id "Device:C_Small") (at 145.415 77.47 0) (unit 1)
-    (in_bom yes) (on_board yes) (dnp no)
+    (in_bom yes) (on_board yes) (dnp yes)
     (property "Reference" "CB1" (at 147.7518 76.3016 0)
       (effects (font (size 1.27 1.27)) (justify left))
@@
   )
   (symbol (lib_id "Device:C_Small") (at 156.845 77.47 0) (unit 1)
-    (in_bom yes) (on_board yes) (dnp no)
+    (in_bom yes) (on_board yes) (dnp yes)
     (property "Reference" "CB1" (at 159.1818 76.3016 0)
       (effects (font (size 1.27 1.27)) (justify left))
@@
   )
   (symbol (lib_id "grootvoet:LIS2MDL") (at 99.06 78.105 0) (unit 1)
-    (in_bom yes) (on_board yes) (dnp no) (fields_autoplaced)
+    (in_bom no) (on_board yes) (dnp yes) (fields_autoplaced)
     (property "Reference" "U6" (at 101.0159 90.551 0)
       (effects (font (size 1.27 1.27)) (justify left))
@@
   )
   (symbol (lib_id "Device:R_Small") (at 82.55 69.85 0) (mirror y) (unit 1)
-    (in_bom yes) (on_board yes) (dnp no)
+    (in_bom yes) (on_board yes) (dnp yes)
     (property "Reference" "R1" (at 81.0514 68.6816 0)
       (effects (font (size 1.27 1.27)) (justify left))
@@
   )
   (symbol (lib_id "Device:C_Small") (at 168.275 77.47 0) (unit 1)
-    (in_bom yes) (on_board yes) (dnp no)
+    (in_bom yes) (on_board yes) (dnp yes)
     (property "Reference" "C2" (at 171.45 76.2 0)
       (effects (font (size 1.27 1.27)) (justify left))
@@
   )
   (symbol (lib_id "Device:C_Small") (at 83.185 85.09 0) (mirror x) (unit 1)
-    (in_bom yes) (on_board yes) (dnp no)
+    (in_bom yes) (on_board yes) (dnp yes)
     (property "Reference" "C47" (at 80.01 84.4486 0)
       (effects (font (size 1.27 1.27)) (justify right))

Commit message: (sch) relabel
Parts:
- renumbered C47 to C1101, U6 to U1101
Changed lines of the file:
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@@
   (symbol (lib_id "power:+3.3V") (at 99.06 62.865 0) (unit 1)
     (in_bom yes) (on_board yes) (dnp no) (fields_autoplaced)
-    (property "Reference" "#PWR0194" (at 99.06 66.675 0)
+    (property "Reference" "#PWR01103" (at 99.06 66.675 0)
       (effects (font (size 1.27 1.27)) hide)
     )
@@
       (project "kleinvoet"
         (path "/4185c36c-c66e-4dbd-be5d-841e551f4885/3579cd31-f7d1-4b38-82cc-1314e00d3f8a"
-          (reference "#PWR0194") (unit 1)
+          (reference "#PWR01103") (unit 1)
         )
       )
@@
   (symbol (lib_id "power:GND") (at 145.415 84.455 0) (unit 1)
     (in_bom yes) (on_board yes) (dnp no) (fields_autoplaced)
-    (property "Reference" "#PWR0199" (at 145.415 90.805 0)
+    (property "Reference" "#PWR01106" (at 145.415 90.805 0)
       (effects (font (size 1.27 1.27)) hide)
     )
@@
       (project "kleinvoet"
         (path "/4185c36c-c66e-4dbd-be5d-841e551f4885/3579cd31-f7d1-4b38-82cc-1314e00d3f8a"
-          (reference "#PWR0199") (unit 1)
+          (reference "#PWR01106") (unit 1)
         )
       )
@@
         )
         (path "/4185c36c-c66e-4dbd-be5d-841e551f4885/3579cd31-f7d1-4b38-82cc-1314e00d3f8a"
-          (reference "CB10") (unit 1)
+          (reference "CB1101") (unit 1)
         )
       )
@@
   (symbol (lib_id "power:GND") (at 99.06 90.805 0) (unit 1)
     (in_bom yes) (on_board yes) (dnp no) (fields_autoplaced)
-    (property "Reference" "#PWR0193" (at 99.06 97.155 0)
+    (property "Reference" "#PWR01104" (at 99.06 97.155 0)
       (effects (font (size 1.27 1.27)) hide)
     )
@@
       (project "kleinvoet"
         (path "/4185c36c-c66e-4dbd-be5d-841e551f4885/3579cd31-f7d1-4b38-82cc-1314e00d3f8a"
-          (reference "#PWR0193") (unit 1)
+          (reference "#PWR01104") (unit 1)
         )
       )
@@
         )
         (path "/4185c36c-c66e-4dbd-be5d-841e551f4885/3579cd31-f7d1-4b38-82cc-1314e00d3f8a"
-          (reference "CB11") (unit 1)
+          (reference "CB1102") (unit 1)
         )
       )
@@
   (symbol (lib_id "power:+3.3V") (at 82.55 62.865 0) (unit 1)
     (in_bom yes) (on_board yes) (dnp no) (fields_autoplaced)
-    (property "Reference" "#PWR0196" (at 82.55 66.675 0)
+    (property "Reference" "#PWR01101" (at 82.55 66.675 0)
       (effects (font (size 1.27 1.27)) hide)
     )
@@
       (project "kleinvoet"
         (path "/4185c36c-c66e-4dbd-be5d-841e551f4885/3579cd31-f7d1-4b38-82cc-1314e00d3f8a"
-          (reference "#PWR0196") (unit 1)
+          (reference "#PWR01101") (unit 1)
         )
       )
@@
   (symbol (lib_id "power:GND") (at 168.275 85.09 0) (unit 1)
     (in_bom yes) (on_board yes) (dnp no) (fields_autoplaced)
-    (property "Reference" "#PWR0202" (at 168.275 91.44 0)
+    (property "Reference" "#PWR01110" (at 168.275 91.44 0)
       (effects (font (size 1.27 1.27)) hide)
     )
@@
       (project "kleinvoet"
         (path "/4185c36c-c66e-4dbd-be5d-841e551f4885/3579cd31-f7d1-4b38-82cc-1314e00d3f8a"
-          (reference "#PWR0202") (unit 1)
+          (reference "#PWR01110") (unit 1)
         )
       )
@@
   (symbol (lib_id "power:+3.3V") (at 156.845 69.85 0) (unit 1)
     (in_bom yes) (on_board yes) (dnp no) (fields_autoplaced)
-    (property "Reference" "#PWR0198" (at 156.845 73.66 0)
+    (property "Reference" "#PWR01107" (at 156.845 73.66 0)
       (effects (font (size 1.27 1.27)) hide)
     )
@@
       (project "kleinvoet"
         (path "/4185c36c-c66e-4dbd-be5d-841e551f4885/3579cd31-f7d1-4b38-82cc-1314e00d3f8a"
-          (reference "#PWR0198") (unit 1)
+          (reference "#PWR01107") (unit 1)
         )
       )
@@
   (symbol (lib_id "power:GND") (at 83.185 92.075 0) (unit 1)
     (in_bom yes) (on_board yes) (dnp no) (fields_autoplaced)
-    (property "Reference" "#PWR0195" (at 83.185 98.425 0)
+    (property "Reference" "#PWR01102" (at 83.185 98.425 0)
       (effects (font (size 1.27 1.27)) hide)
     )
@@
       (project "kleinvoet"
         (path "/4185c36c-c66e-4dbd-be5d-841e551f4885/3579cd31-f7d1-4b38-82cc-1314e00d3f8a"
-          (reference "#PWR0195") (unit 1)
+          (reference "#PWR01102") (unit 1)
         )
       )
@@
   (symbol (lib_id "grootvoet:LIS2MDL") (at 99.06 78.105 0) (unit 1)
     (in_bom no) (on_board yes) (dnp yes) (fields_autoplaced)
-    (property "Reference" "U6" (at 101.0159 90.551 0)
+    (property "Reference" "U1101" (at 101.0159 90.551 0)
       (effects (font (size 1.27 1.27)) (justify left))
     )
@@
       (project "kleinvoet"
         (path "/4185c36c-c66e-4dbd-be5d-841e551f4885/3579cd31-f7d1-4b38-82cc-1314e00d3f8a"
-          (reference "U6") (unit 1)
+          (reference "U1101") (unit 1)
         )
       )
@@
   (symbol (lib_id "power:GND") (at 156.845 84.455 0) (unit 1)
     (in_bom yes) (on_board yes) (dnp no) (fields_autoplaced)
-    (property "Reference" "#PWR0200" (at 156.845 90.805 0)
+    (property "Reference" "#PWR01108" (at 156.845 90.805 0)
       (effects (font (size 1.27 1.27)) hide)
     )
@@
       (project "kleinvoet"
         (path "/4185c36c-c66e-4dbd-be5d-841e551f4885/3579cd31-f7d1-4b38-82cc-1314e00d3f8a"
-          (reference "#PWR0200") (unit 1)
+          (reference "#PWR01108") (unit 1)
         )
       )
@@
         )
         (path "/4185c36c-c66e-4dbd-be5d-841e551f4885/3579cd31-f7d1-4b38-82cc-1314e00d3f8a"
-          (reference "R20") (unit 1)
+          (reference "R1101") (unit 1)
         )
       )
@@
   (symbol (lib_id "power:+3.3V") (at 145.415 70.485 0) (unit 1)
     (in_bom yes) (on_board yes) (dnp no) (fields_autoplaced)
-    (property "Reference" "#PWR0197" (at 145.415 74.295 0)
+    (property "Reference" "#PWR01105" (at 145.415 74.295 0)
       (effects (font (size 1.27 1.27)) hide)
     )
@@
       (project "kleinvoet"
         (path "/4185c36c-c66e-4dbd-be5d-841e551f4885/3579cd31-f7d1-4b38-82cc-1314e00d3f8a"
-          (reference "#PWR0197") (unit 1)
+          (reference "#PWR01105") (unit 1)
         )
       )
@@
         )
         (path "/4185c36c-c66e-4dbd-be5d-841e551f4885/3579cd31-f7d1-4b38-82cc-1314e00d3f8a"
-          (reference "C48") (unit 1)
+          (reference "C1102") (unit 1)
         )
       )
@@
   (symbol (lib_id "Device:C_Small") (at 83.185 85.09 0) (mirror x) (unit 1)
     (in_bom yes) (on_board yes) (dnp yes)
-    (property "Reference" "C47" (at 80.01 84.4486 0)
+    (property "Reference" "C1101" (at 80.01 84.4486 0)
       (effects (font (size 1.27 1.27)) (justify right))
     )
@@
       (project "kleinvoet"
         (path "/4185c36c-c66e-4dbd-be5d-841e551f4885/3579cd31-f7d1-4b38-82cc-1314e00d3f8a"
-          (reference "C47") (unit 1)
+          (reference "C1101") (unit 1)
         )
       )
@@
   (symbol (lib_id "power:+3.3V") (at 168.275 69.85 0) (unit 1)
     (in_bom yes) (on_board yes) (dnp no) (fields_autoplaced)
-    (property "Reference" "#PWR0201" (at 168.275 73.66 0)
+    (property "Reference" "#PWR01109" (at 168.275 73.66 0)
       (effects (font (size 1.27 1.27)) hide)
     )
@@
       (project "kleinvoet"
         (path "/4185c36c-c66e-4dbd-be5d-841e551f4885/3579cd31-f7d1-4b38-82cc-1314e00d3f8a"
-          (reference "#PWR0201") (unit 1)
-        )
-      )
+          (reference "#PWR01109") (unit 1)
+        )
+      )

Commit message: (hk) asign footprints
Parts:
- C1201: renamed from C1101; footprint (none) -> Capacitor_SMD:C_0603_1608Metric_Pad1.08x0.95mm_HandSolder
- renumbered U1101 to U1201
Changed lines of the file:
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@@
   (symbol (lib_id "power:+3.3V") (at 99.06 62.865 0) (unit 1)
     (in_bom yes) (on_board yes) (dnp no) (fields_autoplaced)
-    (property "Reference" "#PWR01103" (at 99.06 66.675 0)
+    (property "Reference" "#PWR01203" (at 99.06 66.675 0)
       (effects (font (size 1.27 1.27)) hide)
     )
@@
       (project "kleinvoet"
         (path "/4185c36c-c66e-4dbd-be5d-841e551f4885/3579cd31-f7d1-4b38-82cc-1314e00d3f8a"
-          (reference "#PWR01103") (unit 1)
+          (reference "#PWR01203") (unit 1)
         )
       )
@@
   (symbol (lib_id "power:GND") (at 145.415 84.455 0) (unit 1)
     (in_bom yes) (on_board yes) (dnp no) (fields_autoplaced)
-    (property "Reference" "#PWR01106" (at 145.415 90.805 0)
+    (property "Reference" "#PWR01206" (at 145.415 90.805 0)
       (effects (font (size 1.27 1.27)) hide)
     )
@@
       (project "kleinvoet"
         (path "/4185c36c-c66e-4dbd-be5d-841e551f4885/3579cd31-f7d1-4b38-82cc-1314e00d3f8a"
-          (reference "#PWR01106") (unit 1)
+          (reference "#PWR01206") (unit 1)
         )
       )
@@
         )
         (path "/4185c36c-c66e-4dbd-be5d-841e551f4885/3579cd31-f7d1-4b38-82cc-1314e00d3f8a"
-          (reference "CB1101") (unit 1)
+          (reference "CB1201") (unit 1)
         )
       )
@@
   (symbol (lib_id "power:GND") (at 99.06 90.805 0) (unit 1)
     (in_bom yes) (on_board yes) (dnp no) (fields_autoplaced)
-    (property "Reference" "#PWR01104" (at 99.06 97.155 0)
+    (property "Reference" "#PWR01204" (at 99.06 97.155 0)
       (effects (font (size 1.27 1.27)) hide)
     )
@@
       (project "kleinvoet"
         (path "/4185c36c-c66e-4dbd-be5d-841e551f4885/3579cd31-f7d1-4b38-82cc-1314e00d3f8a"
-          (reference "#PWR01104") (unit 1)
+          (reference "#PWR01204") (unit 1)
         )
       )
@@
         )
         (path "/4185c36c-c66e-4dbd-be5d-841e551f4885/3579cd31-f7d1-4b38-82cc-1314e00d3f8a"
-          (reference "CB1102") (unit 1)
+          (reference "CB1202") (unit 1)
         )
       )
@@
   (symbol (lib_id "power:+3.3V") (at 82.55 62.865 0) (unit 1)
     (in_bom yes) (on_board yes) (dnp no) (fields_autoplaced)
-    (property "Reference" "#PWR01101" (at 82.55 66.675 0)
+    (property "Reference" "#PWR01201" (at 82.55 66.675 0)
       (effects (font (size 1.27 1.27)) hide)
     )
@@
       (project "kleinvoet"
         (path "/4185c36c-c66e-4dbd-be5d-841e551f4885/3579cd31-f7d1-4b38-82cc-1314e00d3f8a"
-          (reference "#PWR01101") (unit 1)
+          (reference "#PWR01201") (unit 1)
         )
       )
@@
   (symbol (lib_id "power:GND") (at 168.275 85.09 0) (unit 1)
     (in_bom yes) (on_board yes) (dnp no) (fields_autoplaced)
-    (property "Reference" "#PWR01110" (at 168.275 91.44 0)
+    (property "Reference" "#PWR01210" (at 168.275 91.44 0)
       (effects (font (size 1.27 1.27)) hide)
     )
@@
       (project "kleinvoet"
         (path "/4185c36c-c66e-4dbd-be5d-841e551f4885/3579cd31-f7d1-4b38-82cc-1314e00d3f8a"
-          (reference "#PWR01110") (unit 1)
+          (reference "#PWR01210") (unit 1)
         )
       )
@@
   (symbol (lib_id "power:+3.3V") (at 156.845 69.85 0) (unit 1)
     (in_bom yes) (on_board yes) (dnp no) (fields_autoplaced)
-    (property "Reference" "#PWR01107" (at 156.845 73.66 0)
+    (property "Reference" "#PWR01207" (at 156.845 73.66 0)
       (effects (font (size 1.27 1.27)) hide)
     )
@@
       (project "kleinvoet"
         (path "/4185c36c-c66e-4dbd-be5d-841e551f4885/3579cd31-f7d1-4b38-82cc-1314e00d3f8a"
-          (reference "#PWR01107") (unit 1)
+          (reference "#PWR01207") (unit 1)
         )
       )
@@
   (symbol (lib_id "power:GND") (at 83.185 92.075 0) (unit 1)
     (in_bom yes) (on_board yes) (dnp no) (fields_autoplaced)
-    (property "Reference" "#PWR01102" (at 83.185 98.425 0)
+    (property "Reference" "#PWR01202" (at 83.185 98.425 0)
       (effects (font (size 1.27 1.27)) hide)
     )
@@
       (project "kleinvoet"
         (path "/4185c36c-c66e-4dbd-be5d-841e551f4885/3579cd31-f7d1-4b38-82cc-1314e00d3f8a"
-          (reference "#PWR01102") (unit 1)
+          (reference "#PWR01202") (unit 1)
         )
       )
@@
   (symbol (lib_id "grootvoet:LIS2MDL") (at 99.06 78.105 0) (unit 1)
     (in_bom no) (on_board yes) (dnp yes) (fields_autoplaced)
-    (property "Reference" "U1101" (at 101.0159 90.551 0)
+    (property "Reference" "U1201" (at 101.0159 90.551 0)
       (effects (font (size 1.27 1.27)) (justify left))
     )
@@
       (project "kleinvoet"
         (path "/4185c36c-c66e-4dbd-be5d-841e551f4885/3579cd31-f7d1-4b38-82cc-1314e00d3f8a"
-          (reference "U1101") (unit 1)
+          (reference "U1201") (unit 1)
         )
       )
@@
   (symbol (lib_id "power:GND") (at 156.845 84.455 0) (unit 1)
     (in_bom yes) (on_board yes) (dnp no) (fields_autoplaced)
-    (property "Reference" "#PWR01108" (at 156.845 90.805 0)
+    (property "Reference" "#PWR01208" (at 156.845 90.805 0)
       (effects (font (size 1.27 1.27)) hide)
     )
@@
       (project "kleinvoet"
         (path "/4185c36c-c66e-4dbd-be5d-841e551f4885/3579cd31-f7d1-4b38-82cc-1314e00d3f8a"
-          (reference "#PWR01108") (unit 1)
+          (reference "#PWR01208") (unit 1)
         )
       )
@@
         )
         (path "/4185c36c-c66e-4dbd-be5d-841e551f4885/3579cd31-f7d1-4b38-82cc-1314e00d3f8a"
-          (reference "R1101") (unit 1)
+          (reference "R1201") (unit 1)
         )
       )
@@
   (symbol (lib_id "power:+3.3V") (at 145.415 70.485 0) (unit 1)
     (in_bom yes) (on_board yes) (dnp no) (fields_autoplaced)
-    (property "Reference" "#PWR01105" (at 145.415 74.295 0)
+    (property "Reference" "#PWR01205" (at 145.415 74.295 0)
       (effects (font (size 1.27 1.27)) hide)
     )
@@
       (project "kleinvoet"
         (path "/4185c36c-c66e-4dbd-be5d-841e551f4885/3579cd31-f7d1-4b38-82cc-1314e00d3f8a"
-          (reference "#PWR01105") (unit 1)
+          (reference "#PWR01205") (unit 1)
         )
       )
@@
         )
         (path "/4185c36c-c66e-4dbd-be5d-841e551f4885/3579cd31-f7d1-4b38-82cc-1314e00d3f8a"
-          (reference "C1102") (unit 1)
+          (reference "C1202") (unit 1)
         )
       )
@@
   (symbol (lib_id "Device:C_Small") (at 83.185 85.09 0) (mirror x) (unit 1)
     (in_bom yes) (on_board yes) (dnp yes)
-    (property "Reference" "C1101" (at 80.01 84.4486 0)
+    (property "Reference" "C1201" (at 80.01 84.4486 0)
       (effects (font (size 1.27 1.27)) (justify right))
     )
@@
       (effects (font (size 1.27 1.27)) (justify right))
     )
-    (property "Footprint" "" (at 83.185 85.09 0)
+    (property "Footprint" "Capacitor_SMD:C_0603_1608Metric_Pad1.08x0.95mm_HandSolder" (at 83.185 85.09 0)
       (effects (font (size 1.27 1.27)) hide)
     )
@@
       (project "kleinvoet"
         (path "/4185c36c-c66e-4dbd-be5d-841e551f4885/3579cd31-f7d1-4b38-82cc-1314e00d3f8a"
-          (reference "C1101") (unit 1)
+          (reference "C1201") (unit 1)
         )
       )
@@
   (symbol (lib_id "power:+3.3V") (at 168.275 69.85 0) (unit 1)
     (in_bom yes) (on_board yes) (dnp no) (fields_autoplaced)
-    (property "Reference" "#PWR01109" (at 168.275 73.66 0)
+    (property "Reference" "#PWR01209" (at 168.275 73.66 0)
       (effects (font (size 1.27 1.27)) hide)
     )
@@
       (project "kleinvoet"
         (path "/4185c36c-c66e-4dbd-be5d-841e551f4885/3579cd31-f7d1-4b38-82cc-1314e00d3f8a"
-          (reference "#PWR01109") (unit 1)
-        )
-      )
+          (reference "#PWR01209") (unit 1)
+        )
+      )

Commit message: (sch) change passives to 0402
Parts:
- R1: footprint Resistor_SMD:R_0603_1608Metric_Pad0.98x0.95mm_HandSolder -> Resistor_SMD:R_0402_1005Metric; MPN RC0603JR-0710KL -> RT0402FRE1310KL
- U1201: value LIS2MDL -> LIS3MDL; MPN LIS2MDL -> DNP; Mfr. STMicroelectronics -> DNP
Changed lines of the file:
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@@
       (effects (font (size 1.27 1.27)) (justify left))
     )
-    (property "Value" "LIS2MDL" (at 101.0159 93.091 0)
+    (property "Value" "LIS3MDL" (at 101.0159 93.091 0)
       (effects (font (size 1.27 1.27)) (justify left))
     )
@@
       (effects (font (size 1.27 1.27)) hide)
     )
-    (property "MPN" "LIS2MDL" (at 99.06 78.105 0)
+    (property "MPN" "DNP" (at 99.06 78.105 0)
       (effects (font (size 1.27 1.27)) hide)
     )
-    (property "Mfr." "STMicroelectronics" (at 99.06 78.105 0)
+    (property "Mfr." "DNP" (at 99.06 78.105 0)
       (effects (font (size 1.27 1.27)) hide)
     )
@@
       (effects (font (size 1.27 1.27)) (justify left))
     )
-    (property "Footprint" "Resistor_SMD:R_0603_1608Metric_Pad0.98x0.95mm_HandSolder" (at 82.55 69.85 0)
+    (property "Footprint" "Resistor_SMD:R_0402_1005Metric" (at 82.55 69.85 0)
       (effects (font (size 1.27 1.27)) hide)
     )
@@
       (effects (font (size 1.27 1.27)) hide)
     )
-    (property "MPN" "RC0603JR-0710KL" (at 82.55 69.85 0)
+    (property "MPN" "RT0402FRE1310KL" (at 82.55 69.85 0)
       (effects (font (size 1.27 1.27)) hide)
     )

Commit message: (pcb) initial layout
Parts:
- C1201: footprint Capacitor_SMD:C_0603_1608Metric_Pad1.08x0.95mm_HandSolder -> Capacitor_SMD:C_0402_1005Metric_Pad0.74x0.62mm_HandSolder
- C2: value 10u -> 1u; footprint Capacitor_SMD:C_0805_2012Metric_Pad1.18x1.45mm_HandSolder -> Capacitor_SMD:C_0603_1608Metric; MPN C0805C106K9PACTU -> (none)
- CB1: footprint Capacitor_SMD:C_0603_1608Metric_Pad1.08x0.95mm_HandSolder -> Capacitor_SMD:C_0402_1005Metric; MPN C0603C104M5RACTU -> C0402C104K8PACTU
Changed lines of the file:
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@@
       (effects (font (size 1.27 1.27)) (justify left))
     )
-    (property "Footprint" "Capacitor_SMD:C_0603_1608Metric_Pad1.08x0.95mm_HandSolder" (at 145.415 77.47 0)
+    (property "Footprint" "Capacitor_SMD:C_0402_1005Metric" (at 145.415 77.47 0)
       (effects (font (size 1.27 1.27)) hide)
     )
@@
       (effects (font (size 1.27 1.27)) hide)
     )
-    (property "MPN" "C0603C104M5RACTU" (at 145.415 77.47 0)
+    (property "MPN" "C0402C104K8PACTU" (at 145.415 77.47 0)
       (effects (font (size 1.27 1.27)) hide)
     )
@@
       (effects (font (size 1.27 1.27)) (justify left))
     )
-    (property "Footprint" "Capacitor_SMD:C_0603_1608Metric_Pad1.08x0.95mm_HandSolder" (at 156.845 77.47 0)
+    (property "Footprint" "Capacitor_SMD:C_0402_1005Metric" (at 156.845 77.47 0)
       (effects (font (size 1.27 1.27)) hide)
     )
@@
       (effects (font (size 1.27 1.27)) hide)
     )
-    (property "MPN" "C0603C104M5RACTU" (at 156.845 77.47 0)
+    (property "MPN" "C0402C104K8PACTU" (at 156.845 77.47 0)
       (effects (font (size 1.27 1.27)) hide)
     )
@@
       (effects (font (size 1.27 1.27)) (justify left))
     )
-    (property "Value" "10u" (at 171.45 78.105 0)
-      (effects (font (size 1.27 1.27)) (justify left))
-    )
-    (property "Footprint" "Capacitor_SMD:C_0805_2012Metric_Pad1.18x1.45mm_HandSolder" (at 168.275 77.47 0)
+    (property "Value" "1u" (at 171.45 78.105 0)
+      (effects (font (size 1.27 1.27)) (justify left))
+    )
+    (property "Footprint" "Capacitor_SMD:C_0603_1608Metric" (at 168.275 77.47 0)
       (effects (font (size 1.27 1.27)) hide)
     )
@@
       (effects (font (size 1.27 1.27)) hide)
     )
-    (property "MPN" "C0805C106K9PACTU" (at 168.275 77.47 0)
+    (property "MPN" "" (at 168.275 77.47 0)
       (effects (font (size 1.27 1.27)) hide)
     )
@@
       (effects (font (size 1.27 1.27)) (justify right))
     )
-    (property "Footprint" "Capacitor_SMD:C_0603_1608Metric_Pad1.08x0.95mm_HandSolder" (at 83.185 85.09 0)
-      (effects (font (size 1.27 1.27)) hide)
-    )
+    (property "Footprint" "Capacitor_SMD:C_0402_1005Metric_Pad0.74x0.62mm_HandSolder" (at 83.185 85.09 0)
+      (effects (font (size 1.27 1.27)) hide)
+    )
