File: array.kicad_sch (KiCad schematic)
At the start: 18 parts

Commit message: Big commit for the day
Parts:
- renumbered C14 to C?, C15 to C?, CB9 to CB?, CB8 to CB?, CB7 to CB?, CB6 to CB?, CB13 to CB?, CB12 to CB?, CB11 to CB?, CB10 to CB?
Changed lines of the file:
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@@
   (symbol (lib_id "Device:C_Small") (at 25.4 148.59 0) (unit 1)
     (in_bom yes) (on_board yes) (dnp no)
-    (property "Reference" "C14" (at 27.7368 147.4216 0)
+    (property "Reference" "C?" (at 27.7368 147.4216 0)
       (effects (font (size 1.27 1.27)) (justify left))
     )
@@
   (symbol (lib_id "Device:C_Small") (at 34.29 148.59 0) (unit 1)
     (in_bom yes) (on_board yes) (dnp no)
-    (property "Reference" "C15" (at 36.6268 147.4216 0)
+    (property "Reference" "C?" (at 36.6268 147.4216 0)
       (effects (font (size 1.27 1.27)) (justify left))
     )
@@
   (symbol (lib_id "Device:C_Small") (at 27.94 33.02 0) (unit 1)
     (in_bom yes) (on_board yes) (dnp no)
-    (property "Reference" "CB9" (at 30.2768 31.8516 0)
+    (property "Reference" "CB?" (at 30.2768 31.8516 0)
       (effects (font (size 1.27 1.27)) (justify left))
     )
@@
   (symbol (lib_id "Device:C_Small") (at 26.67 62.23 0) (unit 1)
     (in_bom yes) (on_board yes) (dnp no)
-    (property "Reference" "CB8" (at 29.0068 61.0616 0)
+    (property "Reference" "CB?" (at 29.0068 61.0616 0)
       (effects (font (size 1.27 1.27)) (justify left))
     )
@@
   (symbol (lib_id "Device:C_Small") (at 25.4 91.44 0) (unit 1)
     (in_bom yes) (on_board yes) (dnp no)
-    (property "Reference" "CB7" (at 27.7368 90.2716 0)
+    (property "Reference" "CB?" (at 27.7368 90.2716 0)
       (effects (font (size 1.27 1.27)) (justify left))
     )
@@
   (symbol (lib_id "Device:C_Small") (at 24.13 120.65 0) (unit 1)
     (in_bom yes) (on_board yes) (dnp no)
-    (property "Reference" "CB6" (at 26.4668 119.4816 0)
+    (property "Reference" "CB?" (at 26.4668 119.4816 0)
       (effects (font (size 1.27 1.27)) (justify left))
     )
@@
   (symbol (lib_id "Device:C_Small") (at 81.28 33.02 0) (unit 1)
     (in_bom yes) (on_board yes) (dnp no)
-    (property "Reference" "CB13" (at 83.6168 31.8516 0)
+    (property "Reference" "CB?" (at 83.6168 31.8516 0)
       (effects (font (size 1.27 1.27)) (justify left))
     )
@@
   (symbol (lib_id "Device:C_Small") (at 80.01 62.23 0) (unit 1)
     (in_bom yes) (on_board yes) (dnp no)
-    (property "Reference" "CB12" (at 82.3468 61.0616 0)
+    (property "Reference" "CB?" (at 82.3468 61.0616 0)
       (effects (font (size 1.27 1.27)) (justify left))
     )
@@
   (symbol (lib_id "Device:C_Small") (at 78.74 91.44 0) (unit 1)
     (in_bom yes) (on_board yes) (dnp no)
-    (property "Reference" "CB11" (at 81.0768 90.2716 0)
+    (property "Reference" "CB?" (at 81.0768 90.2716 0)
       (effects (font (size 1.27 1.27)) (justify left))
     )
@@
   (symbol (lib_id "Device:C_Small") (at 77.47 120.65 0) (unit 1)
     (in_bom yes) (on_board yes) (dnp no)
-    (property "Reference" "CB10" (at 79.8068 119.4816 0)
-      (effects (font (size 1.27 1.27)) (justify left))
-    )
+    (property "Reference" "CB?" (at 79.8068 119.4816 0)
+      (effects (font (size 1.27 1.27)) (justify left))
+    )

Commit message: (bc) large commit with spice experiments
Parts:
- gave numbers to parts that had none: 10

Commit message: (bc) new summation preamp & seperate power net
Connections:
- net GND: no longer CB25.2
Other:
- moved on the sheet: C53

Commit message: (sch) relabel
Parts:
- renumbered C52 to C1301, C53 to C1302, CB19 to CB1301, CB20 to CB1302, CB21 to CB1303, CB22 to CB1304, CB23 to CB1305, CB24 to CB1306, CB25 to CB1307, CB26 to CB1308, MK1 to MK1301, MK2 to MK1302, MK3 to MK1303, MK4 to MK1304, MK5 to MK1305, MK6 to MK1306, MK7 to MK1307, MK8 to MK1308

Commit message: (bc) finish up ERC
Connections:
- net GND: now also CB1307.2
Changed lines of the file:
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@@
+    )
+  )
+  (symbol (lib_id "grootvoet:GND_SENSOR") (at 80.01 64.77 0) (unit 1)
+    (in_bom yes) (on_board yes) (dnp no) (fields_autoplaced)
+    (property "Reference" "#PWR0215" (at 80.01 71.12 0)
+      (effects (font (size 1.27 1.27)) hide)
+    )
+    (property "Value" "GND_SENSOR" (at 80.01 69.215 0)
+      (effects (font (size 1.27 1.27)))
+    )
+    (property "Footprint" "" (at 80.01 64.77 0)
+      (effects (font (size 1.27 1.27)) hide)
+    )
+    (property "Datasheet" "" (at 80.01 64.77 0)
+      (effects (font (size 1.27 1.27)) hide)
+    )
+    (pin "1")
+    (instances
+      (project "kleinvoet"
+        (path "/4185c36c-c66e-4dbd-be5d-841e551f4885/b53619ea-788f-4bc9-9946-594014d7d22c"
+          (reference "#PWR0215") (unit 1)
+        )
+        (path "/4185c36c-c66e-4dbd-be5d-841e551f4885/b53619ea-788f-4bc9-9946-594014d7d22c/00000000-0000-0000-0000-00005fa63e4d"
+          (reference "#PWR01421") (unit 1)
+        )
+      )
     )
   )

Commit message: (hk) asign footprints
Parts:
- renumbered C1301 to C1401, C1302 to C1402, CB1301 to CB1401, CB1302 to CB1402, CB1303 to CB1403, CB1304 to CB1404, CB1305 to CB1405, CB1306 to CB1406, CB1307 to CB1407, CB1308 to CB1408, MK1301 to MK1401, MK1302 to MK1402, MK1303 to MK1403, MK1304 to MK1404, MK1305 to MK1405, MK1306 to MK1406, MK1307 to MK1407, MK1308 to MK1408

Commit message: (pcb) initial layout
Parts:
- CB1401, CB1402, CB1403, CB1404, CB1405, CB1406, CB1407, CB1408: footprint Capacitor_SMD:C_0603_1608Metric_Pad1.08x0.95mm_HandSolder -> Capacitor_SMD:C_0402_1005Metric; MPN C0603C104M5RACTU -> C0402C104K8PACTU
Changed lines of the file:
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@@
       (effects (font (size 1.27 1.27)) (justify left))
     )
-    (property "Footprint" "Capacitor_SMD:C_0603_1608Metric_Pad1.08x0.95mm_HandSolder" (at 27.94 33.02 0)
+    (property "Footprint" "Capacitor_SMD:C_0402_1005Metric" (at 27.94 33.02 0)
       (effects (font (size 1.27 1.27)) hide)
     )
@@
       (effects (font (size 1.27 1.27)) hide)
     )
-    (property "MPN" "C0603C104M5RACTU" (at 27.94 33.02 0)
+    (property "MPN" "C0402C104K8PACTU" (at 27.94 33.02 0)
       (effects (font (size 1.27 1.27)) hide)
     )
@@
       (effects (font (size 1.27 1.27)) (justify left))
     )
-    (property "Footprint" "Capacitor_SMD:C_0603_1608Metric_Pad1.08x0.95mm_HandSolder" (at 26.67 62.23 0)
+    (property "Footprint" "Capacitor_SMD:C_0402_1005Metric" (at 26.67 62.23 0)
       (effects (font (size 1.27 1.27)) hide)
     )
@@
       (effects (font (size 1.27 1.27)) hide)
     )
-    (property "MPN" "C0603C104M5RACTU" (at 26.67 62.23 0)
+    (property "MPN" "C0402C104K8PACTU" (at 26.67 62.23 0)
       (effects (font (size 1.27 1.27)) hide)
     )
@@
       (effects (font (size 1.27 1.27)) (justify left))
     )
-    (property "Footprint" "Capacitor_SMD:C_0603_1608Metric_Pad1.08x0.95mm_HandSolder" (at 25.4 91.44 0)
+    (property "Footprint" "Capacitor_SMD:C_0402_1005Metric" (at 25.4 91.44 0)
       (effects (font (size 1.27 1.27)) hide)
     )
@@
       (effects (font (size 1.27 1.27)) hide)
     )
-    (property "MPN" "C0603C104M5RACTU" (at 25.4 91.44 0)
+    (property "MPN" "C0402C104K8PACTU" (at 25.4 91.44 0)
       (effects (font (size 1.27 1.27)) hide)
     )
@@
       (effects (font (size 1.27 1.27)) (justify left))
     )
-    (property "Footprint" "Capacitor_SMD:C_0603_1608Metric_Pad1.08x0.95mm_HandSolder" (at 24.13 120.65 0)
+    (property "Footprint" "Capacitor_SMD:C_0402_1005Metric" (at 24.13 120.65 0)
       (effects (font (size 1.27 1.27)) hide)
     )
@@
       (effects (font (size 1.27 1.27)) hide)
     )
-    (property "MPN" "C0603C104M5RACTU" (at 24.13 120.65 0)
+    (property "MPN" "C0402C104K8PACTU" (at 24.13 120.65 0)
       (effects (font (size 1.27 1.27)) hide)
     )
@@
       (effects (font (size 1.27 1.27)) (justify left))
     )
-    (property "Footprint" "Capacitor_SMD:C_0603_1608Metric_Pad1.08x0.95mm_HandSolder" (at 81.28 33.02 0)
+    (property "Footprint" "Capacitor_SMD:C_0402_1005Metric" (at 81.28 33.02 0)
       (effects (font (size 1.27 1.27)) hide)
     )
@@
       (effects (font (size 1.27 1.27)) hide)
     )
-    (property "MPN" "C0603C104M5RACTU" (at 81.28 33.02 0)
+    (property "MPN" "C0402C104K8PACTU" (at 81.28 33.02 0)
       (effects (font (size 1.27 1.27)) hide)
     )
@@
       (effects (font (size 1.27 1.27)) (justify left))
     )
-    (property "Footprint" "Capacitor_SMD:C_0603_1608Metric_Pad1.08x0.95mm_HandSolder" (at 80.01 62.23 0)
+    (property "Footprint" "Capacitor_SMD:C_0402_1005Metric" (at 80.01 62.23 0)
       (effects (font (size 1.27 1.27)) hide)
     )
@@
       (effects (font (size 1.27 1.27)) hide)
     )
-    (property "MPN" "C0603C104M5RACTU" (at 80.01 62.23 0)
+    (property "MPN" "C0402C104K8PACTU" (at 80.01 62.23 0)
       (effects (font (size 1.27 1.27)) hide)
     )
@@
       (effects (font (size 1.27 1.27)) (justify left))
     )
-    (property "Footprint" "Capacitor_SMD:C_0603_1608Metric_Pad1.08x0.95mm_HandSolder" (at 78.74 91.44 0)
+    (property "Footprint" "Capacitor_SMD:C_0402_1005Metric" (at 78.74 91.44 0)
       (effects (font (size 1.27 1.27)) hide)
     )
@@
       (effects (font (size 1.27 1.27)) hide)
     )
-    (property "MPN" "C0603C104M5RACTU" (at 78.74 91.44 0)
+    (property "MPN" "C0402C104K8PACTU" (at 78.74 91.44 0)
       (effects (font (size 1.27 1.27)) hide)
     )
@@
       (effects (font (size 1.27 1.27)) (justify left))
     )
-    (property "Footprint" "Capacitor_SMD:C_0603_1608Metric_Pad1.08x0.95mm_HandSolder" (at 77.47 120.65 0)
+    (property "Footprint" "Capacitor_SMD:C_0402_1005Metric" (at 77.47 120.65 0)
       (effects (font (size 1.27 1.27)) hide)
     )
@@
       (effects (font (size 1.27 1.27)) hide)
     )
-    (property "MPN" "C0603C104M5RACTU" (at 77.47 120.65 0)
-      (effects (font (size 1.27 1.27)) hide)
-    )
+    (property "MPN" "C0402C104K8PACTU" (at 77.47 120.65 0)
+      (effects (font (size 1.27 1.27)) hide)
+    )

Commit message: (sch) update title block
Other:
- company: (none) -> Department of Electrical and Electronic Engineering - Stellenbosch University
- title: (none) -> Kleinvoet
Changed lines of the file:
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@@
 (kicad_sch (version 20230121) (generator eeschema)
   (paper "A4")
+  (title_block
+    (title "Kleinvoet")
+    (date "2023-04-12")
+    (rev "C")
+    (company "Department of Electrical and Electronic Engineering - Stellenbosch University")
+    (comment 1 "Digital Signal Processing Laboratory")
+    (comment 2 "Author: CM Geldenhuys <cmgeldenhuys@sun.ac.za>")
+    (comment 3 "Project: Kleinvoet")
+    (comment 4 "License: CERN-OHL-S-2.0")
+  )
   (hierarchical_label "MK6" (shape input) (at 111.76 63.5 0) (fields_autoplaced)
     (effects (font (size 1.27 1.27)) (justify left))
