File: array.kicad_sch (KiCad schematic)
At the start: 18 parts

Commit message: replace passives with 0402
Parts:
- C1401, C1402: footprint Capacitor_SMD:C_0603_1608Metric_Pad1.08x0.95mm_HandSolder -> Capacitor_SMD:C_0402_1005Metric; MPN C0603C105K8RACTU -> C0402C105K9PACTU
Changed lines of the file:
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@@
       (effects (font (size 1.27 1.27)) (justify left))
     )
-    (property "Footprint" "Capacitor_SMD:C_0603_1608Metric_Pad1.08x0.95mm_HandSolder" (at 25.4 148.59 0)
+    (property "Footprint" "Capacitor_SMD:C_0402_1005Metric" (at 25.4 148.59 0)
       (effects (font (size 1.27 1.27)) hide)
     )
@@
       (effects (font (size 1.27 1.27)) hide)
     )
-    (property "MPN" "C0603C105K8RACTU" (at 25.4 148.59 0)
+    (property "MPN" "C0402C105K9PACTU" (at 25.4 148.59 0)
       (effects (font (size 1.27 1.27)) hide)
     )
@@
       (effects (font (size 1.27 1.27)) (justify left))
     )
-    (property "Footprint" "Capacitor_SMD:C_0603_1608Metric_Pad1.08x0.95mm_HandSolder" (at 38.735 148.59 0)
+    (property "Footprint" "Capacitor_SMD:C_0402_1005Metric" (at 38.735 148.59 0)
       (effects (font (size 1.27 1.27)) hide)
     )
@@
       (effects (font (size 1.27 1.27)) hide)
     )
-    (property "MPN" "C0603C105K8RACTU" (at 38.735 148.59 0)
+    (property "MPN" "C0402C105K9PACTU" (at 38.735 148.59 0)
       (effects (font (size 1.27 1.27)) hide)
     )

Commit message: (sch) rough layout sensorboard
Parts:
- added C1501, C1503, C1505, C1506, C1507, C1508: 1u, Capacitor_SMD:C_0402_1005Metric, symbol Device:C_Small
Connections:
- net +1V8: now also C1501.1, C1503.1, C1505.1, C1506.1, C1507.1, C1508.1
- net GND: now also C1501.2, C1503.2, C1505.2, C1506.2, C1507.2, C1508.2

Commit message: (pcb) finalise sensorboard layout
Connections:
- net MK1: now also MK1406.1 (OUTPUT); no longer MK1403.1 (OUTPUT)
- net MK3: now also MK1408.1 (OUTPUT); no longer MK1401.1 (OUTPUT)
- net MK4: now also MK1403.1 (OUTPUT); no longer MK1405.1 (OUTPUT)
- net MK5: now also MK1405.1 (OUTPUT); no longer MK1406.1 (OUTPUT)
- net MK6: now also MK1401.1 (OUTPUT); no longer MK1407.1 (OUTPUT)
- net MK7: now also MK1407.1 (OUTPUT); no longer MK1408.1 (OUTPUT)
Changed lines of the file:
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@@
     (comment 4 "License: CERN-OHL-S-2.0")
   )
-  (hierarchical_label "MK6" (shape input) (at 111.76 63.5 0) (fields_autoplaced)
+  (hierarchical_label "MK6" (shape input) (at 55.88 121.92 0) (fields_autoplaced)
     (effects (font (size 1.27 1.27)) (justify left))
   )
-  (hierarchical_label "MK4" (shape input) (at 109.22 121.92 0) (fields_autoplaced)
+  (hierarchical_label "MK4" (shape input) (at 58.42 63.5 0) (fields_autoplaced)
     (effects (font (size 1.27 1.27)) (justify left))
   )
@@
     (effects (font (size 1.27 1.27)) (justify left))
   )
-  (hierarchical_label "MK5" (shape input) (at 110.49 92.71 0) (fields_autoplaced)
+  (hierarchical_label "MK5" (shape input) (at 109.22 121.92 0) (fields_autoplaced)
     (effects (font (size 1.27 1.27)) (justify left))
   )
-  (hierarchical_label "MK1" (shape input) (at 58.42 63.5 0) (fields_autoplaced)
+  (hierarchical_label "MK1" (shape input) (at 110.49 92.71 0) (fields_autoplaced)
     (effects (font (size 1.27 1.27)) (justify left))
   )
-  (hierarchical_label "MK3" (shape input) (at 55.88 121.92 0) (fields_autoplaced)
+  (hierarchical_label "MK3" (shape input) (at 113.03 34.29 0) (fields_autoplaced)
     (effects (font (size 1.27 1.27)) (justify left))
   )
-  (hierarchical_label "MK7" (shape input) (at 113.03 34.29 0) (fields_autoplaced)
+  (hierarchical_label "MK7" (shape input) (at 111.76 63.5 0) (fields_autoplaced)
     (effects (font (size 1.27 1.27)) (justify left))
   )

Commit message: (sch) fix board seperate net labels
Connections:
- net GND renamed GND_SENSOR
