File: ADC_Interface.kicad_sch (KiCad schematic)
At the start: 39 parts, among them U401 ADAU1978, U402 TLV333, X401 12.288MHz

Commit message: (sch) clean up items for BOM
Parts:
- TP406, TP407: now not fitted; now left out of the parts list
Changed lines of the file:
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@@
   )
   (symbol (lib_id "Connector:TestPoint") (at 104.775 135.255 90) (unit 1)
-    (in_bom yes) (on_board yes) (dnp no)
+    (in_bom no) (on_board yes) (dnp yes)
     (property "Reference" "TP406" (at 102.9462 130.302 90)
       (effects (font (size 1.27 1.27)))
@@
       (effects (font (size 1.27 1.27)) hide)
     )
+    (property "MPN" "" (at 104.775 135.255 0)
+      (effects (font (size 1.27 1.27)) hide)
+    )
+    (property "Mfr." "" (at 104.775 135.255 0)
+      (effects (font (size 1.27 1.27)) hide)
+    )
     (pin "1")
     (instances
@@
   )
   (symbol (lib_id "Connector:TestPoint") (at 104.775 142.875 90) (unit 1)
-    (in_bom yes) (on_board yes) (dnp no)
+    (in_bom no) (on_board yes) (dnp yes)
     (property "Reference" "TP407" (at 102.9462 137.922 90)
       (effects (font (size 1.27 1.27)))
@@
       (effects (font (size 1.27 1.27)) hide)
     )
+    (property "MPN" "" (at 104.775 142.875 0)
+      (effects (font (size 1.27 1.27)) hide)
+    )
+    (property "Mfr." "" (at 104.775 142.875 0)
+      (effects (font (size 1.27 1.27)) hide)
+    )

Commit message: (sch) exclude mounting holes & JP from BOM
Parts:
- JP401, JP402: now left out of the parts list
Changed lines of the file:
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@@
   )
   (symbol (lib_id "Jumper:SolderJumper_3_Bridged12") (at 276.86 106.68 270) (mirror x) (unit 1)
-    (in_bom yes) (on_board yes) (dnp no)
+    (in_bom no) (on_board yes) (dnp no)
     (property "Reference" "JP402" (at 278.5872 105.5116 90)
       (effects (font (size 1.27 1.27)) (justify left))
@@
     )
     (property "Datasheet" "~" (at 276.86 106.68 0)
+      (effects (font (size 1.27 1.27)) hide)
+    )
+    (property "MPN" "" (at 276.86 106.68 0)
+      (effects (font (size 1.27 1.27)) hide)
+    )
+    (property "Mfr." "" (at 276.86 106.68 0)
       (effects (font (size 1.27 1.27)) hide)
     )
@@
   )
   (symbol (lib_id "Jumper:SolderJumper_3_Bridged12") (at 266.7 109.22 270) (mirror x) (unit 1)
-    (in_bom yes) (on_board yes) (dnp no)
+    (in_bom no) (on_board yes) (dnp no)
     (property "Reference" "JP401" (at 268.4272 108.0516 90)
       (effects (font (size 1.27 1.27)) (justify left))
@@
       (effects (font (size 1.27 1.27)) hide)
     )
+    (property "MPN" "" (at 266.7 109.22 0)
+      (effects (font (size 1.27 1.27)) hide)
+    )
+    (property "Mfr." "" (at 266.7 109.22 0)
+      (effects (font (size 1.27 1.27)) hide)
+    )
