File: ADC_Frontend.kicad_sch (KiCad schematic)
At the start: 23 parts, among them U701 THS4551xRGT

Commit message: (sch) fix THS4551 3D model
Parts:
- U701: footprint Package_DFN_QFN:VQFN-16-1EP_3x3mm_P0.5mm_EP1.68x1.68mm_ThermalVias -> grootvoet:VQFN-16-1EP_3x3mm_P0.5mm_EP1.68x1.68mm_ThermalVias
Changed lines of the file:
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@@
       (effects (font (size 1.27 1.27)) (justify left))
     )
-    (property "Footprint" "Package_DFN_QFN:VQFN-16-1EP_3x3mm_P0.5mm_EP1.68x1.68mm_ThermalVias" (at 134.62 119.38 0)
+    (property "Footprint" "grootvoet:VQFN-16-1EP_3x3mm_P0.5mm_EP1.68x1.68mm_ThermalVias" (at 134.62 119.38 0)
       (effects (font (size 1.27 1.27)) hide)
     )
@@
       (effects (font (size 1.27 1.27)) (justify left))
     )
-    (property "Footprint" "Package_DFN_QFN:VQFN-16-1EP_3x3mm_P0.5mm_EP1.68x1.68mm_ThermalVias" (at 163.195 55.245 0)
-      (effects (font (size 1.27 1.27)) hide)
-    )
+    (property "Footprint" "grootvoet:VQFN-16-1EP_3x3mm_P0.5mm_EP1.68x1.68mm_ThermalVias" (at 163.195 55.245 0)
+      (effects (font (size 1.27 1.27)) hide)
+    )

Commit message: (sch) run DRC
Other:
- moved on the sheet: C701, C703, R701, R702

Commit message: (sch) consoldate BOM
Parts:
- C704: value DNP -> PH/DNP
- C709, C711: MPN (none) -> C0402C103K3RAC7411; Mfr. Murata -> KEMET
- U701: MPN (none) -> THS4551IRGTR; Mfr. (none) -> Texas Instruments
Changed lines of the file:
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@@
       (effects (font (size 1.27 1.27)) hide)
     )
-    (property "MPN" "" (at 195.58 93.98 0)
-      (effects (font (size 1.27 1.27)) hide)
-    )
-    (property "Mfr." "Murata" (at 195.58 93.98 0)
+    (property "MPN" "C0402C103K3RAC7411" (at 195.58 93.98 0)
+      (effects (font (size 1.27 1.27)) hide)
+    )
+    (property "Mfr." "KEMET" (at 195.58 93.98 0)
       (effects (font (size 1.27 1.27)) hide)
     )
@@
       (effects (font (size 1.27 1.27)) hide)
     )
-    (property "MPN" "" (at 195.58 144.78 0)
-      (effects (font (size 1.27 1.27)) hide)
-    )
-    (property "Mfr." "Murata" (at 195.58 144.78 0)
+    (property "MPN" "C0402C103K3RAC7411" (at 195.58 144.78 0)
+      (effects (font (size 1.27 1.27)) hide)
+    )
+    (property "Mfr." "KEMET" (at 195.58 144.78 0)
       (effects (font (size 1.27 1.27)) hide)
     )
@@
       (effects (font (size 1.27 1.27)) hide)
     )
-    (property "MPN" "" (at 134.62 119.38 0)
-      (effects (font (size 1.27 1.27)) hide)
-    )
-    (property "Mfr." "" (at 134.62 119.38 0)
+    (property "MPN" "THS4551IRGTR" (at 134.62 119.38 0)
+      (effects (font (size 1.27 1.27)) hide)
+    )
+    (property "Mfr." "Texas Instruments" (at 134.62 119.38 0)
       (effects (font (size 1.27 1.27)) hide)
     )
@@
       (effects (font (size 1.27 1.27)) (justify right))
     )
-    (property "Value" "DNP" (at 111.9632 120.523 0)
+    (property "Value" "PH/DNP" (at 111.9632 120.523 0)
       (effects (font (size 1.27 1.27)) (justify right))
     )
@@
       (effects (font (size 1.27 1.27)) hide)
     )
-    (property "MPN" "" (at 163.195 55.245 0)
-      (effects (font (size 1.27 1.27)) hide)
-    )
-    (property "Mfr." "" (at 163.195 55.245 0)
-      (effects (font (size 1.27 1.27)) hide)
-    )
+    (property "MPN" "THS4551IRGTR" (at 163.195 55.245 0)
+      (effects (font (size 1.27 1.27)) hide)
+    )
+    (property "Mfr." "Texas Instruments" (at 163.195 55.245 0)
+      (effects (font (size 1.27 1.27)) hide)
+    )

Commit message: (sch) change diff cap due to unavailable
Parts:
- C703: footprint Capacitor_SMD:C_0402_1005Metric -> Capacitor_SMD:C_0805_2012Metric; MPN GRM1555C1H272GE01D -> GRM2165C1H273JA01D
Changed lines of the file:
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@@
       (effects (font (size 1.27 1.27)) (justify right))
     )
-    (property "Footprint" "Capacitor_SMD:C_0402_1005Metric" (at 85.09 119.38 0)
+    (property "Footprint" "Capacitor_SMD:C_0805_2012Metric" (at 85.09 119.38 0)
       (effects (font (size 1.27 1.27)) hide)
     )
@@
       (effects (font (size 1.27 1.27)) hide)
     )
-    (property "MPN" "GRM1555C1H272GE01D" (at 85.09 119.38 0)
+    (property "MPN" "GRM2165C1H273JA01D" (at 85.09 119.38 0)
       (effects (font (size 1.27 1.27)) hide)
     )

Commit message: (sch) change 10n single-end cap to NG0
Parts:
- C709, C711: MPN C0402C103K3RAC7411 -> GRM1555CYA103GE01D; Mfr. KEMET -> Murata
Changed lines of the file:
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@@
       (effects (font (size 1.27 1.27)) hide)
     )
-    (property "MPN" "C0402C103K3RAC7411" (at 195.58 93.98 0)
+    (property "MPN" "GRM1555CYA103GE01D" (at 195.58 93.98 0)
       (effects (font (size 1.27 1.27)) hide)
     )
-    (property "Mfr." "KEMET" (at 195.58 93.98 0)
+    (property "Mfr." "Murata" (at 195.58 93.98 0)
       (effects (font (size 1.27 1.27)) hide)
     )
@@
       (effects (font (size 1.27 1.27)) hide)
     )
-    (property "MPN" "C0402C103K3RAC7411" (at 195.58 144.78 0)
+    (property "MPN" "GRM1555CYA103GE01D" (at 195.58 144.78 0)
       (effects (font (size 1.27 1.27)) hide)
     )
-    (property "Mfr." "KEMET" (at 195.58 144.78 0)
+    (property "Mfr." "Murata" (at 195.58 144.78 0)
       (effects (font (size 1.27 1.27)) hide)
     )

Commit message: (pcb) fix cap footprint & reroute
Parts:
- C710: footprint Capacitor_SMD:C_0402_1005Metric -> Capacitor_SMD:C_1206_3216Metric; MPN C0402C104K8PACTU -> GRM3195C1H104JA05D; Mfr. KEMET -> Murata
Changed lines of the file:
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@@
       (effects (font (size 1.27 1.27)) (justify left))
     )
-    (property "Footprint" "Capacitor_SMD:C_0402_1005Metric" (at 195.58 119.38 0)
+    (property "Footprint" "Capacitor_SMD:C_1206_3216Metric" (at 195.58 119.38 0)
       (effects (font (size 1.27 1.27)) hide)
     )
@@
       (effects (font (size 1.27 1.27)) hide)
     )
-    (property "MPN" "C0402C104K8PACTU" (at 195.58 119.38 0)
+    (property "MPN" "GRM3195C1H104JA05D" (at 195.58 119.38 0)
       (effects (font (size 1.27 1.27)) hide)
     )
-    (property "Mfr." "KEMET" (at 195.58 119.38 0)
+    (property "Mfr." "Murata" (at 195.58 119.38 0)
       (effects (font (size 1.27 1.27)) hide)
     )

Commit message: (fix) component MPN 0603/0402
Parts:
- R707, R708: value 14.7E -> 15E; MPN RT0603FRE0714R7L -> RT0402FRE0715RL
Changed lines of the file:
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@@
       (effects (font (size 1.27 1.27)))
     )
-    (property "Value" "14.7E" (at 153.67 98.933 90)
+    (property "Value" "15E" (at 153.67 98.933 90)
       (effects (font (size 1.27 1.27)))
     )
@@
       (effects (font (size 1.27 1.27)) hide)
     )
-    (property "MPN" "RT0603FRE0714R7L" (at 153.67 101.6 0)
+    (property "MPN" "RT0402FRE0715RL" (at 153.67 101.6 0)
       (effects (font (size 1.27 1.27)) hide)
     )
@@
       (effects (font (size 1.27 1.27)))
     )
-    (property "Value" "14.7E" (at 153.67 134.493 90)
+    (property "Value" "15E" (at 153.67 134.493 90)
       (effects (font (size 1.27 1.27)))
     )
@@
       (effects (font (size 1.27 1.27)) hide)
     )
-    (property "MPN" "RT0603FRE0714R7L" (at 153.67 137.16 0)
+    (property "MPN" "RT0402FRE0715RL" (at 153.67 137.16 0)
       (effects (font (size 1.27 1.27)) hide)
     )

Commit message: chore: update kicad version
Parts:
- renumbered C41 to C705, C41 to C712
