File: Sensor_Board/Sensor_Board.kicad_pcb (KiCad board)
At the start: 4 copper layers, 68 x 38 mm, 64 parts, among them J1 Mic_Conn, U1 TLV741PxxDBVx, U2 OPA377xxDBVx, U3 THS4551

Commit message: Finish up board design
Parts:
- added C14: 1u, Capacitor_SMD:C_0603_1608Metric_Pad1.08x0.95mm_HandSolder, B.Cu at (179.0, 115.0)
- added C15: 1u, Capacitor_SMD:C_0603_1608Metric_Pad1.08x0.95mm_HandSolder, B.Cu at (181.0, 115.0)
- TP1: moved to F.Cu
- moved TP1 49.9 mm to (205.9, 132.9)
- moved J1 13.5 mm to (210.1, 121.5), turned to 180 degrees
- moved CB5 1.27 mm to (188.0, 131.5), turned to 90 degrees
- moved CB3 1.24 mm to (189.7, 131.5), turned to 90 degrees
- moved R10 0.28 mm to (172.1, 125.8), turned to 180 degrees
- moved C3 0.10 mm to (191.4, 131.5)
- turned CB12 to 270 degrees
- turned CB9 to 180 degrees
- turned R1 to 90 degrees
Routing:
- net GND: track 7.99 -> 142.4 mm, vias 13 -> 69
- net EN: track 2.15 -> 52.4 mm, vias 0 -> 2
- net +1V8: track 2.66 -> 49.3 mm, vias 7 -> 32
- net +3V3: track 9.76 -> 19.3 mm, vias 7 -> 11
- net VCC: track 0.00 -> 3.83 mm, vias 7 -> 6
- added copper zone on In2.Cu, net +1V8
- added copper zone on B.Cu, net GND
Other:
- outline, holes or cut-outs redrawn
- rule trace_min: 0.09 -> 0.15
- rule via_min_drill: 0.2 -> 0.25
- rule via_min_size: 0.45 -> 0.35
- board text added: "PWR"

Commit message: Add connector
Parts:
- J1: footprint Connector_PinHeader_2.00mm:PinHeader_1x08_P2.00mm_Vertical -> grootvoet:TE_7-215079-8; moved to B.Cu
- moved J1 2.41 mm to (209.1, 119.3), turned to 270 degrees
- turned D1 to 270 degrees
Connections:
- net CAL_GND renamed Net-(J1-Pad7)
- net CAL_SIG renamed Net-(J1-Pad8)
- J1 pad 1: SIG_N -> SIG_P
- J1 pad 2: SIG_P -> SIG_N
- J1 pad 4: VCC -> EN
- J1 pad 5: EN -> GND
- J1 pad 6: CAL_EN -> VCC
Routing:
- net SIG_N: track 2.46 -> 34.3 mm
- net SIG_P: track 2.21 -> 32.0 mm
- net EN: track 52.4 -> 49.9 mm
- net VCC: track 3.83 -> 2.08 mm
- net GND: track 142.4 -> 143.6 mm
- net Net-(D1-Pad1): track 3.36 -> 2.64 mm
Other:
- net class Signal added: clearance 0.2, trace_width 0.25, via_dia 0.8, via_drill 0.4
- board text added: "GND"
- board text added: "RSV"
- board text added: "SEN"
- board text added: "SGN"
- board text added: "SGP"
- board text added: "VCC"

Commit message: Update Sch with new compensation
Parts:
- R14: value 270 -> 210

Commit message: Update Footprint & part num.
Parts:
- C2: footprint Capacitor_SMD:C_0603_1608Metric_Pad1.08x0.95mm_HandSolder -> Capacitor_SMD:C_0805_2012Metric_Pad1.18x1.45mm_HandSolder
- R11, R12, R2, R3, R4, R5, R6, R7, R8, R9: value 2.2k -> 2k2
- R17, R18: value 1k -> 1k0
- R19, R20: value 47 -> 47E
- moved C2 0.08 mm to (210.4, 135.9)
Routing:
- net +3V3: track 19.3 -> 17.9 mm
