File: Sensor_Board/Sensor_Board.kicad_pcb (KiCad board)
At the start: 4 copper layers, 68 x 38 mm, 66 parts, among them J1 Mic_Conn, U1 TLV741PxxDBVx, U2 OPA377xxDBVx, U3 THS4551

Commit message: Add emblem
Parts:
- added G***: LOGO, grootvoet:SU-Emblem, B.Cu at (169.3, 132.9)
- added G***: LOGO, grootvoet:Oliver_SilkScreen_15x15mm, B.Cu at (155.6, 113.4)
Routing:
- net +3V3: track 17.9 -> 21.1 mm, vias 11 -> 10
- net GND: track 143.6 -> 146.3 mm
- net +1V8: track 49.3 -> 49.7 mm, vias 32 -> 30
Other:
- board text added: "CM Geldenhuys <20198329@sun.ac.za> Department of Electronic and Electric Engineering Stellenbosch University"
- board text added: "KLEINVOET"
- board text added: "MEMS Microphone Array Rev. B"

Commit message: Update connector
Parts:
- removed CB2: 100n, Capacitor_SMD:C_0603_1608Metric_Pad1.08x0.95mm_HandSolder
- removed G***: LOGO, grootvoet:SU-Emblem
- removed G***: LOGO, grootvoet:Oliver_SilkScreen_15x15mm
- R1: value 100k -> 10k
- moved J1 8.61 mm to (211.2, 111.0), turned to 90 degrees
Connections:
- J1 pad 1: SIG_P -> Net-(J1-Pad1)
- J1 pad 2: SIG_N -> GND
- J1 pad 3: GND -> SIG_N
- J1 pad 4: EN -> GND
- J1 pad 5: GND -> SIG_P
- J1 pad 6: VCC -> GND
- J1 pad 7: Net-(J1-Pad7) -> VCC
- J1 pad 8: Net-(J1-Pad8) -> GND
- R1 pad 1: VCC -> +3V3
- R1 pad 2: EN -> Net-(R1-Pad2)
- U1 pad 3: EN -> Net-(R1-Pad2)
- U3 pad 3: EN -> +3V3
Routing:
- net EN: track 49.9 -> 0.00 mm, vias 2 -> 0
- net Net-(R1-Pad2): track 0.00 -> 38.6 mm, vias 0 -> 1
- net SIG_P: track 32.0 -> 34.2 mm
- net VCC: track 2.08 -> 0.00 mm
- net GND: track 146.3 -> 145.3 mm
- net SIG_N: track 34.3 -> 35.1 mm

Commit message: Route update conn.
Parts:
- moved R1 1.80 mm to (211.5, 127.2), turned to 270 degrees
Connections:
- R1 pad 1: +3V3 -> VCC
Routing:
- net Net-(R1-Pad2): track 38.6 -> 4.37 mm, vias 1 -> 0
- net SIG_P: track 34.2 -> 39.0 mm
- net SIG_N: track 35.1 -> 39.9 mm
- net +3V3: track 21.1 -> 22.7 mm

Commit message: Misc changes
Parts:
- added G***: LOGO, grootvoet:SU-Emblem, B.Cu at (169.5, 132.9)
- added G***: LOGO, grootvoet:Oliver_SilkScreen_15x15mm, B.Cu at (155.5, 113.5)
Other:
- board text removed: "SEN"

Commit message: Reference panel
Other:
- board outline removed
