File: Sensor_Board/buffer.sch (KiCad schematic (older format))
At the start: 15 parts, among them U2 OPA377xxDBVx

Commit message: Assign footprints
Parts:
- C5: footprint Capacitor_SMD:C_1206_3216Metric_Pad1.33x1.80mm_HandSolder -> Capacitor_SMD:C_0603_1608Metric_Pad1.08x0.95mm_HandSolder; MPN (none) -> C0603C221J5GACTU; Mfr. (none) -> KEMET
- U2: footprint (none) -> Package_TO_SOT_SMD:SOT-23-5
Changed lines of the file:
@@
 F 0 "U2" H 5900 2800 50  0000 L CNN
 F 1 "OPA377xxDBVx" H 5700 2700 50  0000 L CNN
-F 2 "" H 5750 2550 50  0001 C CNN
+F 2 "Package_TO_SOT_SMD:SOT-23-5" H 5750 2550 50  0001 C CNN
 F 3 "" H 5750 2550 50  0001 C CNN
 	1    5400 2950
@@
 F 0 "C5" V 5650 2100 50  0000 C CNN
 F 1 "220p" V 5650 1750 50  0000 C CNN
-F 2 "Capacitor_SMD:C_1206_3216Metric_Pad1.33x1.80mm_HandSolder" H 5600 1950 50  0001 C CNN
+F 2 "Capacitor_SMD:C_0603_1608Metric_Pad1.08x0.95mm_HandSolder" H 5600 1950 50  0001 C CNN
 F 3 "~" H 5600 1950 50  0001 C CNN
-F 4 "" V 5600 1950 50  0001 C CNN "MPN"
-F 5 "" V 5600 1950 50  0001 C CNN "Mfr."
+F 4 "C0603C221J5GACTU" V 5600 1950 50  0001 C CNN "MPN"
+F 5 "KEMET" V 5600 1950 50  0001 C CNN "Mfr."
 F 6 "" V 5600 1950 50  0001 C CNN "Notes"
 	1    5600 1950
@@
 P 4250 2350
 AR Path="/5F9C8C9E" Ref="#PWR?"  Part="1"
-AR Path="/5F9C4001/5F9C8C9E" Ref="#PWR0119"  Part="1"
-F 0 "#PWR0119" H 4250 2100 50  0001 C CNN
+AR Path="/5F9C4001/5F9C8C9E" Ref="#PWR020"  Part="1"
+F 0 "#PWR020" H 4250 2100 50  0001 C CNN
 F 1 "GND" V 4255 2222 50  0000 R CNN
 F 2 "" H 4250 2350 50  0001 C CNN
@@
 P 5550 4400
 AR Path="/5F9C8CA4" Ref="#PWR?"  Part="1"
-AR Path="/5F9C4001/5F9C8CA4" Ref="#PWR0120"  Part="1"
-F 0 "#PWR0120" H 5550 4150 50  0001 C CNN
+AR Path="/5F9C4001/5F9C8CA4" Ref="#PWR022"  Part="1"
+F 0 "#PWR022" H 5550 4150 50  0001 C CNN
 F 1 "GND" H 5555 4227 50  0000 C CNN
 F 2 "" H 5550 4400 50  0001 C CNN
@@
 P 5600 3200
 AR Path="/5F9C8CAA" Ref="#PWR?"  Part="1"
-AR Path="/5F9C4001/5F9C8CAA" Ref="#PWR0121"  Part="1"
-F 0 "#PWR0121" H 5600 2950 50  0001 C CNN
+AR Path="/5F9C4001/5F9C8CAA" Ref="#PWR024"  Part="1"
+F 0 "#PWR024" H 5600 2950 50  0001 C CNN
 F 1 "GND" H 5605 3027 50  0000 C CNN
 F 2 "" H 5600 3200 50  0001 C CNN
@@
 P 5600 2700
 AR Path="/5F9C8CB0" Ref="#PWR?"  Part="1"
-AR Path="/5F9C4001/5F9C8CB0" Ref="#PWR0122"  Part="1"
-F 0 "#PWR0122" H 5600 2550 50  0001 C CNN
+AR Path="/5F9C4001/5F9C8CB0" Ref="#PWR023"  Part="1"
+F 0 "#PWR023" H 5600 2550 50  0001 C CNN
 F 1 "+3V3" H 5615 2873 50  0000 C CNN
 F 2 "" H 5600 2700 50  0001 C CNN
@@
 P 5550 4200
 AR Path="/5F9C8CB6" Ref="#PWR?"  Part="1"
-AR Path="/5F9C4001/5F9C8CB6" Ref="#PWR0123"  Part="1"
-F 0 "#PWR0123" H 5550 4050 50  0001 C CNN
+AR Path="/5F9C4001/5F9C8CB6" Ref="#PWR021"  Part="1"
+F 0 "#PWR021" H 5550 4050 50  0001 C CNN
 F 1 "+3V3" H 5565 4373 50  0000 C CNN
 F 2 "" H 5550 4200 50  0001 C CNN
@@
 Connection ~ 4500 5150
 $Comp
-L power:GND #PWR0124
+L power:GND #PWR019
 U 1 1 5F9DA9AB
 P 3650 5800
-F 0 "#PWR0124" H 3650 5550 50  0001 C CNN
+F 0 "#PWR019" H 3650 5550 50  0001 C CNN
 F 1 "GND" V 3655 5672 50  0000 R CNN
 F 2 "" H 3650 5800 50  0001 C CNN

Commit message: Update Footprint & part num.
Parts:
- R11, R12, R2, R3, R4, R5, R6, R7, R8, R9: value 2.2k -> 2k2; Mfr. Yageo -> Panasonic
Changed lines of the file:
@@
 AR Path="/5F9C4001/5F9C8C68" Ref="R11"  Part="1"
 F 0 "R11" H 4709 2396 50  0000 L CNN
-F 1 "2.2k" H 4709 2305 50  0000 L CNN
+F 1 "2k2" H 4709 2305 50  0000 L CNN
 F 2 "Resistor_SMD:R_0603_1608Metric_Pad0.98x0.95mm_HandSolder" H 4650 2350 50  0001 C CNN
 F 3 "~" H 4650 2350 50  0001 C CNN
 F 4 "" H 4650 2350 50  0001 C CNN "MPN"
-F 5 "Yageo" H 4650 2350 50  0001 C CNN "Mfr."
+F 5 "Panasonic" H 4650 2350 50  0001 C CNN "Mfr."
 	1    4650 2350
 	0    -1   -1   0
@@
 AR Path="/5F9C4001/5F9C8C70" Ref="R12"  Part="1"
 F 0 "R12" V 5650 2500 50  0000 L CNN
-F 1 "2.2k" V 5650 2050 50  0000 L CNN
+F 1 "2k2" V 5650 2050 50  0000 L CNN
 F 2 "Resistor_SMD:R_0603_1608Metric_Pad0.98x0.95mm_HandSolder" H 5600 2350 50  0001 C CNN
 F 3 "~" H 5600 2350 50  0001 C CNN
 F 4 "" H 5600 2350 50  0001 C CNN "MPN"
-F 5 "Yageo" H 5600 2350 50  0001 C CNN "Mfr."
+F 5 "Panasonic" H 5600 2350 50  0001 C CNN "Mfr."
 	1    5600 2350
 	0    -1   -1   0
@@
 AR Path="/5F9C4001/5F9C9C1D" Ref="R2"  Part="1"
 F 0 "R2" H 3909 3096 50  0000 L CNN
-F 1 "2.2k" H 3909 3005 50  0000 L CNN
+F 1 "2k2" H 3909 3005 50  0000 L CNN
 F 2 "Resistor_SMD:R_0603_1608Metric_Pad0.98x0.95mm_HandSolder" H 3850 3050 50  0001 C CNN
 F 3 "~" H 3850 3050 50  0001 C CNN
 F 4 "" H 3850 3050 50  0001 C CNN "MPN"
-F 5 "Yageo" H 3850 3050 50  0001 C CNN "Mfr."
+F 5 "Panasonic" H 3850 3050 50  0001 C CNN "Mfr."
 	1    3850 3050
 	0    -1   -1   0
@@
 AR Path="/5F9C4001/5F9CA170" Ref="R3"  Part="1"
 F 0 "R3" H 3909 3396 50  0000 L CNN
-F 1 "2.2k" H 3909 3305 50  0000 L CNN
+F 1 "2k2" H 3909 3305 50  0000 L CNN
 F 2 "Resistor_SMD:R_0603_1608Metric_Pad0.98x0.95mm_HandSolder" H 3850 3350 50  0001 C CNN
 F 3 "~" H 3850 3350 50  0001 C CNN
 F 4 "" H 3850 3350 50  0001 C CNN "MPN"
-F 5 "Yageo" H 3850 3350 50  0001 C CNN "Mfr."
+F 5 "Panasonic" H 3850 3350 50  0001 C CNN "Mfr."
 	1    3850 3350
 	0    -1   -1   0
@@
 AR Path="/5F9C4001/5F9CB9C2" Ref="R4"  Part="1"
 F 0 "R4" H 3909 3696 50  0000 L CNN
-F 1 "2.2k" H 3909 3605 50  0000 L CNN
+F 1 "2k2" H 3909 3605 50  0000 L CNN
 F 2 "Resistor_SMD:R_0603_1608Metric_Pad0.98x0.95mm_HandSolder" H 3850 3650 50  0001 C CNN
 F 3 "~" H 3850 3650 50  0001 C CNN
 F 4 "" H 3850 3650 50  0001 C CNN "MPN"
-F 5 "Yageo" H 3850 3650 50  0001 C CNN "Mfr."
+F 5 "Panasonic" H 3850 3650 50  0001 C CNN "Mfr."
 	1    3850 3650
 	0    -1   -1   0
@@
 AR Path="/5F9C4001/5F9CB9CA" Ref="R5"  Part="1"
 F 0 "R5" H 3909 3996 50  0000 L CNN
-F 1 "2.2k" H 3909 3905 50  0000 L CNN
+F 1 "2k2" H 3909 3905 50  0000 L CNN
 F 2 "Resistor_SMD:R_0603_1608Metric_Pad0.98x0.95mm_HandSolder" H 3850 3950 50  0001 C CNN
 F 3 "~" H 3850 3950 50  0001 C CNN
 F 4 "" H 3850 3950 50  0001 C CNN "MPN"
-F 5 "Yageo" H 3850 3950 50  0001 C CNN "Mfr."
+F 5 "Panasonic" H 3850 3950 50  0001 C CNN "Mfr."
 	1    3850 3950
 	0    -1   -1   0
@@
 AR Path="/5F9C4001/5F9CD10D" Ref="R6"  Part="1"
 F 0 "R6" H 3909 4296 50  0000 L CNN
-F 1 "2.2k" H 3909 4205 50  0000 L CNN
+F 1 "2k2" H 3909 4205 50  0000 L CNN
 F 2 "Resistor_SMD:R_0603_1608Metric_Pad0.98x0.95mm_HandSolder" H 3850 4250 50  0001 C CNN
 F 3 "~" H 3850 4250 50  0001 C CNN
 F 4 "" H 3850 4250 50  0001 C CNN "MPN"
-F 5 "Yageo" H 3850 4250 50  0001 C CNN "Mfr."
+F 5 "Panasonic" H 3850 4250 50  0001 C CNN "Mfr."
 	1    3850 4250
 	0    -1   -1   0
@@
 AR Path="/5F9C4001/5F9CD115" Ref="R7"  Part="1"
 F 0 "R7" H 3909 4596 50  0000 L CNN
-F 1 "2.2k" H 3909 4505 50  0000 L CNN
+F 1 "2k2" H 3909 4505 50  0000 L CNN
 F 2 "Resistor_SMD:R_0603_1608Metric_Pad0.98x0.95mm_HandSolder" H 3850 4550 50  0001 C CNN
 F 3 "~" H 3850 4550 50  0001 C CNN
 F 4 "" H 3850 4550 50  0001 C CNN "MPN"
-F 5 "Yageo" H 3850 4550 50  0001 C CNN "Mfr."
+F 5 "Panasonic" H 3850 4550 50  0001 C CNN "Mfr."
 	1    3850 4550
 	0    -1   -1   0
@@
 AR Path="/5F9C4001/5F9CD11D" Ref="R8"  Part="1"
 F 0 "R8" H 3909 4896 50  0000 L CNN
-F 1 "2.2k" H 3909 4805 50  0000 L CNN
+F 1 "2k2" H 3909 4805 50  0000 L CNN
 F 2 "Resistor_SMD:R_0603_1608Metric_Pad0.98x0.95mm_HandSolder" H 3850 4850 50  0001 C CNN
 F 3 "~" H 3850 4850 50  0001 C CNN
 F 4 "" H 3850 4850 50  0001 C CNN "MPN"
-F 5 "Yageo" H 3850 4850 50  0001 C CNN "Mfr."
+F 5 "Panasonic" H 3850 4850 50  0001 C CNN "Mfr."
 	1    3850 4850
 	0    -1   -1   0
@@
 AR Path="/5F9C4001/5F9CD125" Ref="R9"  Part="1"
 F 0 "R9" H 3909 5196 50  0000 L CNN
-F 1 "2.2k" H 3909 5105 50  0000 L CNN
+F 1 "2k2" H 3909 5105 50  0000 L CNN
 F 2 "Resistor_SMD:R_0603_1608Metric_Pad0.98x0.95mm_HandSolder" H 3850 5150 50  0001 C CNN
 F 3 "~" H 3850 5150 50  0001 C CNN
 F 4 "" H 3850 5150 50  0001 C CNN "MPN"
-F 5 "Yageo" H 3850 5150 50  0001 C CNN "Mfr."
+F 5 "Panasonic" H 3850 5150 50  0001 C CNN "Mfr."
 	1    3850 5150
 	0    -1   -1   0

Commit message: Update BOM
Parts:
- R10: Mfr. Yageo -> (none)
- R11, R12, R2, R3, R4, R5, R6, R7, R8, R9: MPN (none) -> ERJ-3EKF2201V
- U2: MPN (none) -> OPA377AIDBVR; Mfr. (none) -> Texas Instruments
Changed lines of the file:
@@
 F 2 "Package_TO_SOT_SMD:SOT-23-5" H 5750 2550 50  0001 C CNN
 F 3 "" H 5750 2550 50  0001 C CNN
+F 4 "OPA377AIDBVR" H 5400 2950 50  0001 C CNN "MPN"
+F 5 "Texas Instruments" H 5400 2950 50  0001 C CNN "Mfr."
 	1    5400 2950
 	1    0    0    -1
@@
 F 2 "Resistor_SMD:R_0603_1608Metric_Pad0.98x0.95mm_HandSolder" H 4650 2350 50  0001 C CNN
 F 3 "~" H 4650 2350 50  0001 C CNN
-F 4 "" H 4650 2350 50  0001 C CNN "MPN"
+F 4 "ERJ-3EKF2201V" H 4650 2350 50  0001 C CNN "MPN"
 F 5 "Panasonic" H 4650 2350 50  0001 C CNN "Mfr."
 	1    4650 2350
@@
 F 2 "Resistor_SMD:R_0603_1608Metric_Pad0.98x0.95mm_HandSolder" H 5600 2350 50  0001 C CNN
 F 3 "~" H 5600 2350 50  0001 C CNN
-F 4 "" H 5600 2350 50  0001 C CNN "MPN"
+F 4 "ERJ-3EKF2201V" H 5600 2350 50  0001 C CNN "MPN"
 F 5 "Panasonic" H 5600 2350 50  0001 C CNN "Mfr."
 	1    5600 2350
@@
 F 2 "Resistor_SMD:R_0603_1608Metric_Pad0.98x0.95mm_HandSolder" H 3850 3050 50  0001 C CNN
 F 3 "~" H 3850 3050 50  0001 C CNN
-F 4 "" H 3850 3050 50  0001 C CNN "MPN"
+F 4 "ERJ-3EKF2201V" H 3850 3050 50  0001 C CNN "MPN"
 F 5 "Panasonic" H 3850 3050 50  0001 C CNN "Mfr."
 	1    3850 3050
@@
 F 2 "Resistor_SMD:R_0603_1608Metric_Pad0.98x0.95mm_HandSolder" H 3850 3350 50  0001 C CNN
 F 3 "~" H 3850 3350 50  0001 C CNN
-F 4 "" H 3850 3350 50  0001 C CNN "MPN"
+F 4 "ERJ-3EKF2201V" H 3850 3350 50  0001 C CNN "MPN"
 F 5 "Panasonic" H 3850 3350 50  0001 C CNN "Mfr."
 	1    3850 3350
@@
 F 2 "Resistor_SMD:R_0603_1608Metric_Pad0.98x0.95mm_HandSolder" H 3850 3650 50  0001 C CNN
 F 3 "~" H 3850 3650 50  0001 C CNN
-F 4 "" H 3850 3650 50  0001 C CNN "MPN"
+F 4 "ERJ-3EKF2201V" H 3850 3650 50  0001 C CNN "MPN"
 F 5 "Panasonic" H 3850 3650 50  0001 C CNN "Mfr."
 	1    3850 3650
@@
 F 2 "Resistor_SMD:R_0603_1608Metric_Pad0.98x0.95mm_HandSolder" H 3850 3950 50  0001 C CNN
 F 3 "~" H 3850 3950 50  0001 C CNN
-F 4 "" H 3850 3950 50  0001 C CNN "MPN"
+F 4 "ERJ-3EKF2201V" H 3850 3950 50  0001 C CNN "MPN"
 F 5 "Panasonic" H 3850 3950 50  0001 C CNN "Mfr."
 	1    3850 3950
@@
 F 2 "Resistor_SMD:R_0603_1608Metric_Pad0.98x0.95mm_HandSolder" H 3850 4250 50  0001 C CNN
 F 3 "~" H 3850 4250 50  0001 C CNN
-F 4 "" H 3850 4250 50  0001 C CNN "MPN"
+F 4 "ERJ-3EKF2201V" H 3850 4250 50  0001 C CNN "MPN"
 F 5 "Panasonic" H 3850 4250 50  0001 C CNN "Mfr."
 	1    3850 4250
@@
 F 2 "Resistor_SMD:R_0603_1608Metric_Pad0.98x0.95mm_HandSolder" H 3850 4550 50  0001 C CNN
 F 3 "~" H 3850 4550 50  0001 C CNN
-F 4 "" H 3850 4550 50  0001 C CNN "MPN"
+F 4 "ERJ-3EKF2201V" H 3850 4550 50  0001 C CNN "MPN"
 F 5 "Panasonic" H 3850 4550 50  0001 C CNN "Mfr."
 	1    3850 4550
@@
 F 2 "Resistor_SMD:R_0603_1608Metric_Pad0.98x0.95mm_HandSolder" H 3850 4850 50  0001 C CNN
 F 3 "~" H 3850 4850 50  0001 C CNN
-F 4 "" H 3850 4850 50  0001 C CNN "MPN"
+F 4 "ERJ-3EKF2201V" H 3850 4850 50  0001 C CNN "MPN"
 F 5 "Panasonic" H 3850 4850 50  0001 C CNN "Mfr."
 	1    3850 4850
@@
 F 2 "Resistor_SMD:R_0603_1608Metric_Pad0.98x0.95mm_HandSolder" H 3850 5150 50  0001 C CNN
 F 3 "~" H 3850 5150 50  0001 C CNN
-F 4 "" H 3850 5150 50  0001 C CNN "MPN"
+F 4 "ERJ-3EKF2201V" H 3850 5150 50  0001 C CNN "MPN"
 F 5 "Panasonic" H 3850 5150 50  0001 C CNN "Mfr."
 	1    3850 5150
@@
 F 3 "~" H 3850 5800 50  0001 C CNN
 F 4 "" H 3850 5800 50  0001 C CNN "MPN"
-F 5 "Yageo" H 3850 5800 50  0001 C CNN "Mfr."
+F 5 "" H 3850 5800 50  0001 C CNN "Mfr."
 	1    3850 5800
 	0    -1   -1   0
