File: Sensor_Board/Microphone_Sensor.sch (KiCad schematic (older format))
At the start: 31 parts, among them J4 Mic_Conn, U4 MAX4063

Commit message: Merge 'feature/mic-board'
Split out Sensor_board to own project for easier panelising later.
Allows also for better independent development.

Squashed commit of the following:
===============================================
commit 5c89ddf7514428c762fb7c211bc44fe947092eb1
Author: CM Geldenhuys <20198329@sun.ac.za>
Date:   Wed Oct 21 14:34:31 2020 +0200

    Add emblem

commit bbe0a53b49b0ec3aa4e2f65424c556ce99509fe4
Author: CM Geldenhuys <20198329@sun.ac.za>
Date:   Wed Oct 21 11:03:40 2020 +0200

    Misc.

commit b3172de48a622d4a7c8e9fb13a381d32a0990437
Author: CM Geldenhuys <20198329@sun.ac.za>
Date:   Wed Oct 21 08:26:42 2020 +0200

    Update BOM

commit e4c5b39694adfe3b823840b4cd3bc00d306b52fc
Author: CM Geldenhuys <20198329@sun.ac.za>
Date:   Wed Oct 21 07:26:34 2020 +0200

    Update Footprint & part num.

commit 6125562d7501cc555d98682860bdd64678a2fa40
Author: CM Geldenhuys <20198329@sun.ac.za>
Date:   Tue Oct 20 15:41:10 2020 +0200

    Misc. TODOs

commit 1431b8ace7af2c4960b7d9361ce6fcca694d3a38
Author: CM Geldenhuys <20198329@sun.ac.za>
Date:   Tue Oct 20 11:22:04 2020 +0200

    Update passives (fuse + Vsense)

commit 8105b403ec058cf7267c739b2e244ad8880c475f
Author: CM Geldenhuys <20198329@sun.ac.za>
Date:   Tue Oct 20 11:02:06 2020 +0200

    Flip GPS labels

commit f34b34dca70ce235e33188df7f6c69707ad79c9c
Author: CM Geldenhuys <20198329@sun.ac.za>
Date:   Tue Oct 20 10:58:45 2020 +0200

    Swap out ST-Link Conn

commit 1669b3f99c1cffa6c87811843550b346cfb9297e
Author: CM Geldenhuys <20198329@sun.ac.za>
Date:   Tue Oct 20 09:57:40 2020 +0200

    Update Sch with new compensation

commit dde033bb3cbd48a104931da2f1a7f681a8f96ac4
Author: CM Geldenhuys <20198329@sun.ac.za>
Date:   Tue Oct 20 09:55:04 2020 +0200

    Compensate for preamp loading on ADC driver

commit 2ddbd04fb1deccaa72131771362207bd14115936
Author: CM Geldenhuys <20198329@sun.ac.za>
Date:   Tue Oct 20 09:38:09 2020 +0200

    Compensate for buffer output impedance

commit 2f74ea7d6b171bacb6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
Parts:
- removed C20: 1u, Capacitor_SMD:C_0603_1608Metric_Pad1.05x0.95mm_HandSolder, symbol Device:C_Small
- removed C22: 47u, Capacitor_SMD:C_1206_3216Metric_Pad1.42x1.75mm_HandSolder, symbol Device:C_Small
- removed C23: 10p, Capacitor_SMD:C_0603_1608Metric_Pad1.05x0.95mm_HandSolder, symbol Device:C_Small
- removed R30: 1k, Resistor_SMD:R_0603_1608Metric_Pad1.05x0.95mm_HandSolder, symbol Device:R_Small
- removed R31, R32: 27, Resistor_SMD:R_0603_1608Metric_Pad1.05x0.95mm_HandSolder, symbol Device:R_Small
- removed R33, R34: 100k, Resistor_SMD:R_0603_1608Metric_Pad1.05x0.95mm_HandSolder, symbol Device:R_Small
- removed U4: MAX4063, grootvoet:TQFN-16-T1644++4, symbol grootvoet:MAX4063
- added 220p, 220p?: C_Small, symbol Device:C_Small
- added C?: 220p, Capacitor_SMD:C_1206_3216Metric_Pad1.33x1.80mm_HandSolder, symbol Device:C_Small
- added C?: 1u, Capacitor_SMD:C_0603_1608Metric_Pad1.08x0.95mm_HandSolder, symbol Device:C_Small
- added C? (x2): 2.7n, symbol Device:C_Small
- added C?: PH, symbol Device:C_Small
- added C?: 18n, symbol Device:C_Small
- added CB? (x3): 100n, Capacitor_SMD:C_0603_1608Metric_Pad1.08x0.95mm_HandSolder, symbol Device:C_Small
- added R? (x2): 2.2k, Resistor_SMD:R_0603_1608Metric_Pad0.98x0.95mm_HandSolder, symbol Device:R_Small
- added R? (x2): 100k, Resistor_SMD:R_0603_1608Metric_Pad0.98x0.95mm_HandSolder, symbol Device:R_Small
- added R? (x2): 270, symbol Device:R_Small
- added R? (x2): 330, symbol Device:R_Small
- added R? (x2): 1k, symbol Device:R_Small
- added R? (x2): 47, symbol Device:R_Small
- added U?: OPA377xxDBVx, symbol grootvoet:OPA377xxDBVx
- added U?: THS4551, symbol grootvoet:THS4551
- C21: footprint Capacitor_SMD:C_1206_3216Metric_Pad1.42x1.75mm_HandSolder -> Capacitor_SMD:C_1206_3216Metric_Pad1.33x1.80mm_HandSolder
- C24, C25, C26, C27, CB18, CB19, CB20, CB21, CB22: footprint Capacitor_SMD:C_0603_1608Metric_Pad1.05x0.95mm_HandSolder -> Capacitor_SMD:C_0603_1608Metric_Pad1.08x0.95mm_HandSolder
- R35, R36, R37, R38: footprint Resistor_SMD:R_0603_1608Metric_Pad1.05x0.95mm_HandSolder -> Resistor_SMD:R_0603_1608Metric_Pad0.98x0.95mm_HandSolder
Connections:
- net labels added: VBuffer, VCM
- net labels removed: OUT_N, OUT_P
- wire segments 57 -> 110
Other:
- note added: "Buffer + Summer Amp"
- note added: "Preamplifier + LPF + Line Driver"
- note removed: "27 Ohm resistors lower the chance of \nocilations due to frequency domain \ninstability."
- note removed: "See Datasheet MAX4063"
- note removed: "Signal Conditioning"
- moved on the sheet: C2, C5, C6, C7, C8, CB1, CB2, CB3, CB4, CB5, FB1, H1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
