File: Sensor_Board/array.sch (KiCad schematic (older format))
At the start: 16 parts

Commit message: Assign footprints
Parts:
- renumbered CB7 to CB6, CB8 to CB7, CB9 to CB8, CB6 to CB9, MK2 to MK1, MK3 to MK2, MK4 to MK3, MK1 to MK4

Commit message: Finish up board design
Parts:
- added C14, C15: 1u, Capacitor_SMD:C_0603_1608Metric_Pad1.08x0.95mm_HandSolder, symbol Device:C_Small
Connections:
- net +1V8: now also C14.1, C15.1
- net GND: now also C14.2, C15.2
Changed lines of the file:
@@
+	1    0    0    -1
+$EndComp
+$Comp
+L Device:C_Small C?
+U 1 1 5F8A4374
+P 1000 5850
+AR Path="/5EE5ECAD/5EECE6B8/5F8A4374" Ref="C?"  Part="1"
+AR Path="/5EE5ECAD/5EF21991/5F8A4374" Ref="C?"  Part="1"
+AR Path="/5EE5ECAD/5EF33EA2/5F8A4374" Ref="C?"  Part="1"
+AR Path="/5EE5ECAD/5EF4C631/5F8A4374" Ref="C?"  Part="1"
+AR Path="/5EE5ECAD/5F0013E5/5F8A4374" Ref="C?"  Part="1"
+AR Path="/5EE5ECAD/5F0090C7/5F8A4374" Ref="C?"  Part="1"
+AR Path="/5F803BE9/5F8A4374" Ref="C?"  Part="1"
+AR Path="/5F8A4374" Ref="C?"  Part="1"
+AR Path="/5FA63E4D/5F8A4374" Ref="C14"  Part="1"
+F 0 "C14" H 1092 5896 50  0000 L CNN
+F 1 "1u" H 1092 5805 50  0000 L CNN
+F 2 "Capacitor_SMD:C_0603_1608Metric_Pad1.08x0.95mm_HandSolder" H 1000 5850 50  0001 C CNN
+F 3 "~" H 1000 5850 50  0001 C CNN
+F 4 "C0603C105K8RACTU" H 1000 5850 50  0001 C CNN "MPN"
+F 5 "KEMET" H 1000 5850 50  0001 C CNN "Mfr."
+	1    1000 5850
+	1    0    0    -1
+$EndComp
+$Comp
+L power:GND #PWR?
+U 1 1 5F8A437A
+P 1000 5950
+AR Path="/5F8A437A" Ref="#PWR?"  Part="1"
+AR Path="/5FA63E4D/5F8A437A" Ref="#PWR066"  Part="1"
+F 0 "#PWR066" H 1000 5700 50  0001 C CNN
+F 1 "GND" H 1005 5777 50  0000 C CNN
+F 2 "" H 1000 5950 50  0001 C CNN
+F 3 "" H 1000 5950 50  0001 C CNN
+	1    1000 5950
+	1    0    0    -1
+$EndComp
+$Comp
+L Device:C_Small C?
+U 1 1 5F8A47E8
+P 1350 5850
+AR Path="/5EE5ECAD/5EECE6B8/5F8A47E8" Ref="C?"  Part="1"
+AR Path="/5EE5ECAD/5EF21991/5F8A47E8" Ref="C?"  Part="1"
+AR Path="/5EE5ECAD/5EF33EA2/5F8A47E8" Ref="C?"  Part="1"
+AR Path="/5EE5ECAD/5EF4C631/5F8A47E8" Ref="C?"  Part="1"
+AR Path="/5EE5ECAD/5F0013E5/5F8A47E8" Ref="C?"  Part="1"
+AR Path="/5EE5ECAD/5F0090C7/5F8A47E8" Ref="C?"  Part="1"
+AR Path="/5F803BE9/5F8A47E8" Ref="C?"  Part="1"
+AR Path="/5F8A47E8" Ref="C?"  Part="1"
+AR Path="/5FA63E4D/5F8A47E8" Ref="C15"  Part="1"
+F 0 "C15" H 1442 5896 50  0000 L CNN
+F 1 "1u" H 1442 5805 50  0000 L CNN
+F 2 "Capacitor_SMD:C_0603_1608Metric_Pad1.08x0.95mm_HandSolder" H 1350 5850 50  0001 C CNN
+F 3 "~" H 1350 5850 50  0001 C CNN
+F 4 "C0603C105K8RACTU" H 1350 5850 50  0001 C CNN "MPN"
+F 5 "KEMET" H 1350 5850 50  0001 C CNN "Mfr."
+	1    1350 5850
+	1    0    0    -1
+$EndComp
+$Comp
+L power:GND #PWR?
+U 1 1 5F8A47EE
+P 1350 5950
+AR Path="/5F8A47EE" Ref="#PWR?"  Part="1"
+AR Path="/5FA63E4D/5F8A47EE" Ref="#PWR068"  Part="1"
+F 0 "#PWR068" H 1350 5700 50  0001 C CNN
+F 1 "GND" H 1355 5777 50  0000 C CNN
+F 2 "" H 1350 5950 50  0001 C CNN
+F 3 "" H 1350 5950 50  0001 C CNN
+	1    1350 5950
+	1    0    0    -1
+$EndComp
+$Comp
+L power:+1V8 #PWR065
+U 1 1 5F8A4AF2
+P 1000 5750
+F 0 "#PWR065" H 1000 5600 50  0001 C CNN
+F 1 "+1V8" H 1015 5923 50  0000 C CNN
+F 2 "" H 1000 5750 50  0001 C CNN
+F 3 "" H 1000 5750 50  0001 C CNN
+	1    1000 5750
+	1    0    0    -1
+$EndComp
+$Comp
+L power:+1V8 #PWR067
+U 1 1 5F8A4CB5
+P 1350 5750
+F 0 "#PWR067" H 1350 5600 50  0001 C CNN
+F 1 "+1V8" H 1365 5923 50  0000 C CNN
+F 2 "" H 1350 5750 50  0001 C CNN
+F 3 "" H 1350 5750 50  0001 C CNN
+	1    1350 5750
 	1    0    0    -1
 $EndComp

Commit message: Update ICS40300 MPN
Parts:
- MK1, MK2, MK3, MK4, MK5, MK6, MK7, MK8: MPN (none) -> ICS-40300; Mfr. (none) -> TDK InvenSense
Changed lines of the file:
@@
 F 2 "grootvoet:MEMS_Mic_ICS-40300" H 1800 1250 50  0001 C CNN
 F 3 "https://www.mouser.co.za/ProductDetail/TDK-InvenSense/ICS-40300?qs=%2Fha2pyFadujzJsvx64xsUNdAo4Ph4hwqMvEiGbKRLds%3D" H 1800 1250 50  0001 C CNN
+F 4 "ICS-40300" H 1850 1350 50  0001 C CNN "MPN"
+F 5 "TDK InvenSense" H 1850 1350 50  0001 C CNN "Mfr."
 	1    1850 1350
 	1    0    0    -1
@@
 F 2 "grootvoet:MEMS_Mic_ICS-40300" H 1750 2400 50  0001 C CNN
 F 3 "https://www.mouser.co.za/ProductDetail/TDK-InvenSense/ICS-40300?qs=%2Fha2pyFadujzJsvx64xsUNdAo4Ph4hwqMvEiGbKRLds%3D" H 1750 2400 50  0001 C CNN
+F 4 "ICS-40300" H 1800 2500 50  0001 C CNN "MPN"
+F 5 "TDK InvenSense" H 1800 2500 50  0001 C CNN "Mfr."
 	1    1800 2500
 	1    0    0    -1
@@
 F 2 "grootvoet:MEMS_Mic_ICS-40300" H 1700 3550 50  0001 C CNN
 F 3 "https://www.mouser.co.za/ProductDetail/TDK-InvenSense/ICS-40300?qs=%2Fha2pyFadujzJsvx64xsUNdAo4Ph4hwqMvEiGbKRLds%3D" H 1700 3550 50  0001 C CNN
+F 4 "ICS-40300" H 1750 3650 50  0001 C CNN "MPN"
+F 5 "TDK InvenSense" H 1750 3650 50  0001 C CNN "Mfr."
 	1    1750 3650
 	1    0    0    -1
@@
 F 2 "grootvoet:MEMS_Mic_ICS-40300" H 1650 4700 50  0001 C CNN
 F 3 "https://www.mouser.co.za/ProductDetail/TDK-InvenSense/ICS-40300?qs=%2Fha2pyFadujzJsvx64xsUNdAo4Ph4hwqMvEiGbKRLds%3D" H 1650 4700 50  0001 C CNN
+F 4 "ICS-40300" H 1700 4800 50  0001 C CNN "MPN"
+F 5 "TDK InvenSense" H 1700 4800 50  0001 C CNN "Mfr."
 	1    1700 4800
 	1    0    0    -1
@@
 F 2 "grootvoet:MEMS_Mic_ICS-40300" H 3900 1250 50  0001 C CNN
 F 3 "https://www.mouser.co.za/ProductDetail/TDK-InvenSense/ICS-40300?qs=%2Fha2pyFadujzJsvx64xsUNdAo4Ph4hwqMvEiGbKRLds%3D" H 3900 1250 50  0001 C CNN
+F 4 "ICS-40300" H 3950 1350 50  0001 C CNN "MPN"
+F 5 "TDK InvenSense" H 3950 1350 50  0001 C CNN "Mfr."
 	1    3950 1350
 	1    0    0    -1
@@
 F 2 "grootvoet:MEMS_Mic_ICS-40300" H 3850 2400 50  0001 C CNN
 F 3 "https://www.mouser.co.za/ProductDetail/TDK-InvenSense/ICS-40300?qs=%2Fha2pyFadujzJsvx64xsUNdAo4Ph4hwqMvEiGbKRLds%3D" H 3850 2400 50  0001 C CNN
+F 4 "ICS-40300" H 3900 2500 50  0001 C CNN "MPN"
+F 5 "TDK InvenSense" H 3900 2500 50  0001 C CNN "Mfr."
 	1    3900 2500
 	1    0    0    -1
@@
 F 2 "grootvoet:MEMS_Mic_ICS-40300" H 3800 3550 50  0001 C CNN
 F 3 "https://www.mouser.co.za/ProductDetail/TDK-InvenSense/ICS-40300?qs=%2Fha2pyFadujzJsvx64xsUNdAo4Ph4hwqMvEiGbKRLds%3D" H 3800 3550 50  0001 C CNN
+F 4 "ICS-40300" H 3850 3650 50  0001 C CNN "MPN"
+F 5 "TDK InvenSense" H 3850 3650 50  0001 C CNN "Mfr."
 	1    3850 3650
 	1    0    0    -1
@@
 F 2 "grootvoet:MEMS_Mic_ICS-40300" H 3750 4700 50  0001 C CNN
 F 3 "https://www.mouser.co.za/ProductDetail/TDK-InvenSense/ICS-40300?qs=%2Fha2pyFadujzJsvx64xsUNdAo4Ph4hwqMvEiGbKRLds%3D" H 3750 4700 50  0001 C CNN
+F 4 "ICS-40300" H 3800 4800 50  0001 C CNN "MPN"
+F 5 "TDK InvenSense" H 3800 4800 50  0001 C CNN "Mfr."
 	1    3800 4800
 	1    0    0    -1
