File: Sensor_Board/preamp.sch (KiCad schematic (older format))
At the start: 16 parts, among them U3 THS4551

Commit message: Assign footprints
Parts:
- C12: renamed from 220p1; value C_Small -> 220p; footprint (none) -> Capacitor_SMD:C_0603_1608Metric_Pad1.08x0.95mm_HandSolder
- C13: renamed from 220p2; value C_Small -> 220p; footprint (none) -> Capacitor_SMD:C_0603_1608Metric_Pad1.08x0.95mm_HandSolder
- C6, C8, C9: footprint (none) -> Capacitor_SMD:C_0603_1608Metric_Pad1.08x0.95mm_HandSolder
- C7, R13, R14, R15, R16, R17, R18, R19, R20: footprint (none) -> Resistor_SMD:R_0603_1608Metric_Pad0.98x0.95mm_HandSolder
- U3: footprint (none) -> grootvoet:WQFN-10_RUN
Changed lines of the file:
@@
 F 0 "U3" H 5867 3411 50  0000 C CNN
 F 1 "THS4551" H 5867 3320 50  0000 C CNN
-F 2 "" H 5800 3600 50  0001 C CNN
+F 2 "grootvoet:WQFN-10_RUN" H 5800 3600 50  0001 C CNN
 F 3 "" H 5800 3600 50  0001 C CNN
 	1    5400 3850
@@
 F 0 "R13" V 3704 3150 50  0000 C CNN
 F 1 "270" V 3795 3150 50  0000 C CNN
-F 2 "" H 3900 3150 50  0001 C CNN
+F 2 "Resistor_SMD:R_0603_1608Metric_Pad0.98x0.95mm_HandSolder" H 3900 3150 50  0001 C CNN
 F 3 "~" H 3900 3150 50  0001 C CNN
 	1    3900 3150
@@
 F 0 "R15" V 4254 3150 50  0000 C CNN
 F 1 "330" V 4345 3150 50  0000 C CNN
-F 2 "" H 4450 3150 50  0001 C CNN
+F 2 "Resistor_SMD:R_0603_1608Metric_Pad0.98x0.95mm_HandSolder" H 4450 3150 50  0001 C CNN
 F 3 "~" H 4450 3150 50  0001 C CNN
 	1    4450 3150
@@
 F 0 "R17" V 5704 2750 50  0000 C CNN
 F 1 "1k" V 5795 2750 50  0000 C CNN
-F 2 "" H 5900 2750 50  0001 C CNN
+F 2 "Resistor_SMD:R_0603_1608Metric_Pad0.98x0.95mm_HandSolder" H 5900 2750 50  0001 C CNN
 F 3 "~" H 5900 2750 50  0001 C CNN
 	1    5900 2750
@@
 F 0 "R19" V 6154 3150 50  0000 C CNN
 F 1 "47" V 6245 3150 50  0000 C CNN
-F 2 "" H 6350 3150 50  0001 C CNN
+F 2 "Resistor_SMD:R_0603_1608Metric_Pad0.98x0.95mm_HandSolder" H 6350 3150 50  0001 C CNN
 F 3 "~" H 6350 3150 50  0001 C CNN
 	1    6350 3150
@@
 F 0 "C8" V 5421 3150 50  0000 C CNN
 F 1 "2.7n" V 5512 3150 50  0000 C CNN
-F 2 "" H 5650 3150 50  0001 C CNN
+F 2 "Capacitor_SMD:C_0603_1608Metric_Pad1.08x0.95mm_HandSolder" H 5650 3150 50  0001 C CNN
 F 3 "~" H 5650 3150 50  0001 C CNN
 	1    5650 3150
@@
 F 0 "C7" H 4792 3896 50  0000 L CNN
 F 1 "PH" H 4792 3805 50  0000 L CNN
-F 2 "" H 4700 3850 50  0001 C CNN
+F 2 "Resistor_SMD:R_0603_1608Metric_Pad0.98x0.95mm_HandSolder" H 4700 3850 50  0001 C CNN
 F 3 "~" H 4700 3850 50  0001 C CNN
 	1    4700 3850
@@
 F 0 "C6" H 4242 3896 50  0000 L CNN
 F 1 "18n" H 4242 3805 50  0000 L CNN
-F 2 "" H 4150 3850 50  0001 C CNN
+F 2 "Capacitor_SMD:C_0603_1608Metric_Pad1.08x0.95mm_HandSolder" H 4150 3850 50  0001 C CNN
 F 3 "~" H 4150 3850 50  0001 C CNN
 	1    4150 3850
@@
 AR Path="/5F803BE9/5F9FD205" Ref="220p?"  Part="1"
 AR Path="/5F9FD205" Ref="220p?"  Part="1"
-AR Path="/5F9ED899/5F9FD205" Ref="220p1"  Part="1"
-F 0 "220p1" H 4242 2796 50  0000 L CNN
-F 1 "C_Small" H 4242 2705 50  0000 L CNN
-F 2 "" H 4150 2750 50  0001 C CNN
+AR Path="/5F9ED899/5F9FD205" Ref="C12"  Part="1"
+F 0 "C12" H 4242 2796 50  0000 L CNN
+F 1 "220p" H 4242 2705 50  0000 L CNN
+F 2 "Capacitor_SMD:C_0603_1608Metric_Pad1.08x0.95mm_HandSolder" H 4150 2750 50  0001 C CNN
 F 3 "~" H 4150 2750 50  0001 C CNN
 	1    4150 2750
@@
 F 0 "R14" V 3704 4550 50  0000 C CNN
 F 1 "270" V 3795 4550 50  0000 C CNN
-F 2 "" H 3900 4550 50  0001 C CNN
+F 2 "Resistor_SMD:R_0603_1608Metric_Pad0.98x0.95mm_HandSolder" H 3900 4550 50  0001 C CNN
 F 3 "~" H 3900 4550 50  0001 C CNN
 	1    3900 4550
@@
 F 0 "R16" V 4254 4550 50  0000 C CNN
 F 1 "330" V 4345 4550 50  0000 C CNN
-F 2 "" H 4450 4550 50  0001 C CNN
+F 2 "Resistor_SMD:R_0603_1608Metric_Pad0.98x0.95mm_HandSolder" H 4450 4550 50  0001 C CNN
 F 3 "~" H 4450 4550 50  0001 C CNN
 	1    4450 4550
@@
 F 0 "R18" V 5704 4950 50  0000 C CNN
 F 1 "1k" V 5795 4950 50  0000 C CNN
-F 2 "" H 5900 4950 50  0001 C CNN
+F 2 "Resistor_SMD:R_0603_1608Metric_Pad0.98x0.95mm_HandSolder" H 5900 4950 50  0001 C CNN
 F 3 "~" H 5900 4950 50  0001 C CNN
 	1    5900 4950
@@
 F 0 "R20" V 6154 4550 50  0000 C CNN
 F 1 "47" V 6245 4550 50  0000 C CNN
-F 2 "" H 6350 4550 50  0001 C CNN
+F 2 "Resistor_SMD:R_0603_1608Metric_Pad0.98x0.95mm_HandSolder" H 6350 4550 50  0001 C CNN
 F 3 "~" H 6350 4550 50  0001 C CNN
 	1    6350 4550
@@
 F 0 "C9" V 5421 4550 50  0000 C CNN
 F 1 "2.7n" V 5512 4550 50  0000 C CNN
-F 2 "" H 5650 4550 50  0001 C CNN
+F 2 "Capacitor_SMD:C_0603_1608Metric_Pad1.08x0.95mm_HandSolder" H 5650 4550 50  0001 C CNN
 F 3 "~" H 5650 4550 50  0001 C CNN
 	1    5650 4550
@@
 AR Path="/5F803BE9/5F9FD244" Ref="220p?"  Part="1"
 AR Path="/5F9FD244" Ref="220p?"  Part="1"
-AR Path="/5F9ED899/5F9FD244" Ref="220p2"  Part="1"
-F 0 "220p2" H 4242 4996 50  0000 L CNN
-F 1 "C_Small" H 4242 4905 50  0000 L CNN
-F 2 "" H 4150 4950 50  0001 C CNN
+AR Path="/5F9ED899/5F9FD244" Ref="C13"  Part="1"
+F 0 "C13" H 4058 4904 50  0000 R CNN
+F 1 "220p" H 4058 4995 50  0000 R CNN
+F 2 "Capacitor_SMD:C_0603_1608Metric_Pad1.08x0.95mm_HandSolder" H 4150 4950 50  0001 C CNN
 F 3 "~" H 4150 4950 50  0001 C CNN
 	1    4150 4950
@@
 IN
 $Comp
-L power:+3V3 #PWR0125
+L power:+3V3 #PWR027
 U 1 1 5FA050B6
 P 5600 3450
-F 0 "#PWR0125" H 5600 3300 50  0001 C CNN
+F 0 "#PWR027" H 5600 3300 50  0001 C CNN
 F 1 "+3V3" H 5615 3623 50  0000 C CNN
 F 2 "" H 5600 3450 50  0001 C CNN
@@
 $EndComp
 $Comp
-L power:GND #PWR0126
+L power:GND #PWR028
 U 1 1 5FA0546B
 P 5600 4200
-F 0 "#PWR0126" H 5600 3950 50  0001 C CNN
+F 0 "#PWR028" H 5600 3950 50  0001 C CNN
 F 1 "GND" H 5605 4027 50  0000 C CNN
 F 2 "" H 5600 4200 50  0001 C CNN
@@
 $EndComp
 $Comp
-L power:+3V3 #PWR0127
+L power:+3V3 #PWR029
 U 1 1 5FA09046
 P 6450 3750
-F 0 "#PWR0127" H 6450 3600 50  0001 C CNN
+F 0 "#PWR029" H 6450 3600 50  0001 C CNN
 F 1 "+3V3" H 6465 3923 50  0000 C CNN
 F 2 "" H 6450 3750 50  0001 C CNN
@@
 $EndComp
 $Comp
-L power:GND #PWR0128
+L power:GND #PWR030
 U 1 1 5FA093A8
 P 6450 3950
-F 0 "#PWR0128" H 6450 3700 50  0001 C CNN
+F 0 "#PWR030" H 6450 3700 50  0001 C CNN
 F 1 "GND" H 6455 3777 50  0000 C CNN
 F 2 "" H 6450 3950 50  0001 C CNN
@@
 VOCM
 $Comp
-L power:GND #PWR0129
+L power:GND #PWR026
 U 1 1 5FA12CD8
 P 4150 5150
-F 0 "#PWR0129" H 4150 4900 50  0001 C CNN
+F 0 "#PWR026" H 4150 4900 50  0001 C CNN
 F 1 "GND" H 4155 4977 50  0000 C CNN
 F 2 "" H 4150 5150 50  0001 C CNN
@@
 	4150 2550 4150 2650
 $Comp
-L power:GND #PWR0130
+L power:GND #PWR025
 U 1 1 5FA13112
 P 4150 2550
-F 0 "#PWR0130" H 4150 2300 50  0001 C CNN
+F 0 "#PWR025" H 4150 2300 50  0001 C CNN
 F 1 "GND" H 4155 2377 50  0000 C CNN
 F 2 "" H 4150 2550 50  0001 C CNN

Commit message: Update Sch with new compensation
Parts:
- R14: value 270 -> 210
Changed lines of the file:
@@
 AR Path="/5F9ED899/5F9FD226" Ref="R14"  Part="1"
 F 0 "R14" V 3704 4550 50  0000 C CNN
-F 1 "270" V 3795 4550 50  0000 C CNN
+F 1 "210" V 3795 4550 50  0000 C CNN
 F 2 "Resistor_SMD:R_0603_1608Metric_Pad0.98x0.95mm_HandSolder" H 3900 4550 50  0001 C CNN
 F 3 "~" H 3900 4550 50  0001 C CNN

Commit message: Update Footprint & part num.
Parts:
- C12, C13: MPN (none) -> C0603C221J5GACTU; Mfr. (none) -> KEMET
- R13, R14, R15, R16: Mfr. (none) -> Panasonic
- R17, R18: value 1k -> 1k0; MPN (none) -> ERJ-3RBD102V; Mfr. (none) -> Panasonic
- R19, R20: value 47 -> 47E; Mfr. (none) -> Panasonic
Changed lines of the file:
@@
 F 2 "Resistor_SMD:R_0603_1608Metric_Pad0.98x0.95mm_HandSolder" H 3900 3150 50  0001 C CNN
 F 3 "~" H 3900 3150 50  0001 C CNN
+F 4 "Panasonic" H 3900 3150 50  0001 C CNN "Mfr."
 	1    3900 3150
 	0    1    1    0
@@
 F 2 "Resistor_SMD:R_0603_1608Metric_Pad0.98x0.95mm_HandSolder" H 4450 3150 50  0001 C CNN
 F 3 "~" H 4450 3150 50  0001 C CNN
+F 4 "Panasonic" H 4450 3150 50  0001 C CNN "Mfr."
 	1    4450 3150
 	0    1    1    0
@@
 AR Path="/5F9ED899/5F9FD1E7" Ref="R17"  Part="1"
 F 0 "R17" V 5704 2750 50  0000 C CNN
-F 1 "1k" V 5795 2750 50  0000 C CNN
+F 1 "1k0" V 5795 2750 50  0000 C CNN
 F 2 "Resistor_SMD:R_0603_1608Metric_Pad0.98x0.95mm_HandSolder" H 5900 2750 50  0001 C CNN
 F 3 "~" H 5900 2750 50  0001 C CNN
+F 4 "ERJ-3RBD102V" H 5900 2750 50  0001 C CNN "MPN"
+F 5 "Panasonic" H 5900 2750 50  0001 C CNN "Mfr."
 	1    5900 2750
 	0    1    1    0
@@
 AR Path="/5F9ED899/5F9FD1ED" Ref="R19"  Part="1"
 F 0 "R19" V 6154 3150 50  0000 C CNN
-F 1 "47" V 6245 3150 50  0000 C CNN
+F 1 "47E" V 6245 3150 50  0000 C CNN
 F 2 "Resistor_SMD:R_0603_1608Metric_Pad0.98x0.95mm_HandSolder" H 6350 3150 50  0001 C CNN
 F 3 "~" H 6350 3150 50  0001 C CNN
+F 4 "Panasonic" H 6350 3150 50  0001 C CNN "Mfr."
 	1    6350 3150
 	0    1    1    0
@@
 F 2 "Capacitor_SMD:C_0603_1608Metric_Pad1.08x0.95mm_HandSolder" H 4150 2750 50  0001 C CNN
 F 3 "~" H 4150 2750 50  0001 C CNN
+F 4 "C0603C221J5GACTU" H 4150 2750 50  0001 C CNN "MPN"
+F 5 "KEMET" H 4150 2750 50  0001 C CNN "Mfr."
 	1    4150 2750
 	1    0    0    -1
@@
 F 2 "Resistor_SMD:R_0603_1608Metric_Pad0.98x0.95mm_HandSolder" H 3900 4550 50  0001 C CNN
 F 3 "~" H 3900 4550 50  0001 C CNN
+F 4 "Panasonic" H 3900 4550 50  0001 C CNN "Mfr."
 	1    3900 4550
 	0    1    -1   0
@@
 F 2 "Resistor_SMD:R_0603_1608Metric_Pad0.98x0.95mm_HandSolder" H 4450 4550 50  0001 C CNN
 F 3 "~" H 4450 4550 50  0001 C CNN
+F 4 "Panasonic" H 4450 4550 50  0001 C CNN "Mfr."
 	1    4450 4550
 	0    1    -1   0
@@
 AR Path="/5F9ED899/5F9FD232" Ref="R18"  Part="1"
 F 0 "R18" V 5704 4950 50  0000 C CNN
-F 1 "1k" V 5795 4950 50  0000 C CNN
+F 1 "1k0" V 5795 4950 50  0000 C CNN
 F 2 "Resistor_SMD:R_0603_1608Metric_Pad0.98x0.95mm_HandSolder" H 5900 4950 50  0001 C CNN
 F 3 "~" H 5900 4950 50  0001 C CNN
+F 4 "ERJ-3RBD102V" H 5900 4950 50  0001 C CNN "MPN"
+F 5 "Panasonic" H 5900 4950 50  0001 C CNN "Mfr."
 	1    5900 4950
 	0    1    -1   0
@@
 AR Path="/5F9ED899/5F9FD238" Ref="R20"  Part="1"
 F 0 "R20" V 6154 4550 50  0000 C CNN
-F 1 "47" V 6245 4550 50  0000 C CNN
+F 1 "47E" V 6245 4550 50  0000 C CNN
 F 2 "Resistor_SMD:R_0603_1608Metric_Pad0.98x0.95mm_HandSolder" H 6350 4550 50  0001 C CNN
 F 3 "~" H 6350 4550 50  0001 C CNN
+F 4 "Panasonic" H 6350 4550 50  0001 C CNN "Mfr."
 	1    6350 4550
 	0    1    -1   0
@@
 F 2 "Capacitor_SMD:C_0603_1608Metric_Pad1.08x0.95mm_HandSolder" H 4150 4950 50  0001 C CNN
 F 3 "~" H 4150 4950 50  0001 C CNN
+F 4 "C0603C221J5GACTU" H 4150 4950 50  0001 C CNN "MPN"
+F 5 "KEMET" H 4150 4950 50  0001 C CNN "Mfr."
 	1    4150 4950
 	1    0    0    1

Commit message: Update BOM
Parts:
- C6: MPN (none) -> CC0603JRX7R8BB183; Mfr. (none) -> Yageo
- C8, C9: MPN (none) -> CC0603JRX7R9BB272; Mfr. (none) -> Yageo
- R13: MPN (none) -> ERJ-3EKF2700V
- R14: MPN (none) -> ERJ-3EKF2100V
- R15, R16: MPN (none) -> ERJ-3EKF3300V
- R17, R18: MPN ERJ-3RBD102V -> ERJ-3EKF1001V
- R19, R20: MPN (none) -> ERJ-3EKF47R0V
- U3: MPN (none) -> THS4551IRUNR; Mfr. (none) -> Texas Instruments
Changed lines of the file:
@@
 F 2 "grootvoet:WQFN-10_RUN" H 5800 3600 50  0001 C CNN
 F 3 "" H 5800 3600 50  0001 C CNN
+F 4 "THS4551IRUNR" H 5400 3850 50  0001 C CNN "MPN"
+F 5 "Texas Instruments" H 5400 3850 50  0001 C CNN "Mfr."
 	1    5400 3850
 	1    0    0    -1
@@
 F 3 "~" H 3900 3150 50  0001 C CNN
 F 4 "Panasonic" H 3900 3150 50  0001 C CNN "Mfr."
+F 5 "ERJ-3EKF2700V" H 3900 3150 50  0001 C CNN "MPN"
 	1    3900 3150
 	0    1    1    0
@@
 F 3 "~" H 4450 3150 50  0001 C CNN
 F 4 "Panasonic" H 4450 3150 50  0001 C CNN "Mfr."
+F 5 "ERJ-3EKF3300V" H 4450 3150 50  0001 C CNN "MPN"
 	1    4450 3150
 	0    1    1    0
@@
 F 2 "Resistor_SMD:R_0603_1608Metric_Pad0.98x0.95mm_HandSolder" H 5900 2750 50  0001 C CNN
 F 3 "~" H 5900 2750 50  0001 C CNN
-F 4 "ERJ-3RBD102V" H 5900 2750 50  0001 C CNN "MPN"
+F 4 "ERJ-3EKF1001V" H 5900 2750 50  0001 C CNN "MPN"
 F 5 "Panasonic" H 5900 2750 50  0001 C CNN "Mfr."
 	1    5900 2750
@@
 F 3 "~" H 6350 3150 50  0001 C CNN
 F 4 "Panasonic" H 6350 3150 50  0001 C CNN "Mfr."
+F 5 "ERJ-3EKF47R0V" H 6350 3150 50  0001 C CNN "MPN"
 	1    6350 3150
 	0    1    1    0
@@
 F 2 "Capacitor_SMD:C_0603_1608Metric_Pad1.08x0.95mm_HandSolder" H 5650 3150 50  0001 C CNN
 F 3 "~" H 5650 3150 50  0001 C CNN
+F 4 "CC0603JRX7R9BB272" H 5650 3150 50  0001 C CNN "MPN"
+F 5 "Yageo" H 5650 3150 50  0001 C CNN "Mfr."
 	1    5650 3150
 	0    1    1    0
@@
 F 2 "Capacitor_SMD:C_0603_1608Metric_Pad1.08x0.95mm_HandSolder" H 4150 3850 50  0001 C CNN
 F 3 "~" H 4150 3850 50  0001 C CNN
+F 4 "CC0603JRX7R8BB183" H 4150 3850 50  0001 C CNN "MPN"
+F 5 "Yageo" H 4150 3850 50  0001 C CNN "Mfr."
 	1    4150 3850
 	1    0    0    -1
@@
 F 3 "~" H 3900 4550 50  0001 C CNN
 F 4 "Panasonic" H 3900 4550 50  0001 C CNN "Mfr."
+F 5 "ERJ-3EKF2100V" H 3900 4550 50  0001 C CNN "MPN"
 	1    3900 4550
 	0    1    -1   0
@@
 F 3 "~" H 4450 4550 50  0001 C CNN
 F 4 "Panasonic" H 4450 4550 50  0001 C CNN "Mfr."
+F 5 "ERJ-3EKF3300V" H 4450 4550 50  0001 C CNN "MPN"
 	1    4450 4550
 	0    1    -1   0
@@
 F 2 "Resistor_SMD:R_0603_1608Metric_Pad0.98x0.95mm_HandSolder" H 5900 4950 50  0001 C CNN
 F 3 "~" H 5900 4950 50  0001 C CNN
-F 4 "ERJ-3RBD102V" H 5900 4950 50  0001 C CNN "MPN"
+F 4 "ERJ-3EKF1001V" H 5900 4950 50  0001 C CNN "MPN"
 F 5 "Panasonic" H 5900 4950 50  0001 C CNN "Mfr."
 	1    5900 4950
@@
 F 3 "~" H 6350 4550 50  0001 C CNN
 F 4 "Panasonic" H 6350 4550 50  0001 C CNN "Mfr."
+F 5 "ERJ-3EKF47R0V" H 6350 4550 50  0001 C CNN "MPN"
 	1    6350 4550
 	0    1    -1   0
@@
 F 2 "Capacitor_SMD:C_0603_1608Metric_Pad1.08x0.95mm_HandSolder" H 5650 4550 50  0001 C CNN
 F 3 "~" H 5650 4550 50  0001 C CNN
+F 4 "CC0603JRX7R9BB272" H 5650 4550 50  0001 C CNN "MPN"
+F 5 "Yageo" H 5650 4550 50  0001 C CNN "Mfr."
 	1    5650 4550
 	0    1    -1   0

Commit message: Update connector
Connections:
- net ~PD is gone; now on net +3V3: U3.3 (~PD)
Changed lines of the file:
@@
 	1    0    0    -1
 $EndComp
-Text HLabel 5700 3500 1    50   Input ~ 0
-~PD
 Wire Wire Line
 	5700 3500 5700 3550
@@
 	-1   0    0    1
 $EndComp
+Wire Wire Line
+	5700 3500 5600 3500
+Connection ~ 5600 3500
 $EndSCHEMATC
