File: Sensor_Board/Sensor_Board.sch (KiCad schematic (older format))
At the start: 16 parts, among them J1 Mic_Conn, U1 TLV741PxxDBVx

Commit message: Route update conn.
Connections:
- net +3V3: no longer R1.1
- net VCC: now also R1.1
Other:
- moved on the sheet: R1
Changed lines of the file:
@@
 F0 "Preamplifier" 50
 F1 "preamp.sch" 50
-F3 "SIG_P" I R 6450 2250 50
-F4 "SIG_N" I R 6450 2450 50
-F5 "~IN" I L 5700 2250 50
-F6 "IN" I L 5700 2450 50
-F7 "VOCM" I R 6450 2650 50
+F2 "SIG_P" I R 6450 2250 50
+F3 "SIG_N" I R 6450 2450 50
+F4 "~IN" I L 5700 2250 50
+F5 "IN" I L 5700 2450 50
+F6 "VOCM" I R 6450 2650 50
 $EndSheet
 $Comp
@@
 	1    0    0    -1
 $EndComp
-Wire Wire Line
-	3800 5200 3600 5200
 Wire Wire Line
 	3200 5200 3200 5150
@@
 L Device:R_Small R?
 U 1 1 5F976175
-P 3600 5300
+P 3700 5500
 AR Path="/5EE5ECAD/5EECE6B8/5F976175" Ref="R?"  Part="1"
 AR Path="/5EE5ECAD/5EF21991/5F976175" Ref="R?"  Part="1"
@@
 AR Path="/5F803BE9/5F976175" Ref="R?"  Part="1"
 AR Path="/5F976175" Ref="R1"  Part="1"
-F 0 "R1" H 3659 5346 50  0000 L CNN
-F 1 "10k" H 3659 5255 50  0000 L CNN
-F 2 "Resistor_SMD:R_0603_1608Metric_Pad0.98x0.95mm_HandSolder" H 3600 5300 50  0001 C CNN
-F 3 "~" H 3600 5300 50  0001 C CNN
-F 4 "" H 3600 5300 50  0001 C CNN "MPN"
-F 5 "Yageo" H 3600 5300 50  0001 C CNN "Mfr."
-	1    3600 5300
-	1    0    0    -1
-$EndComp
-Connection ~ 3600 5200
-Wire Wire Line
-	3600 5200 3200 5200
-Wire Wire Line
-	3800 5400 3600 5400
+F 0 "R1" H 3759 5546 50  0000 L CNN
+F 1 "10k" H 3759 5455 50  0000 L CNN
+F 2 "Resistor_SMD:R_0603_1608Metric_Pad0.98x0.95mm_HandSolder" H 3700 5500 50  0001 C CNN
+F 3 "~" H 3700 5500 50  0001 C CNN
+F 4 "" H 3700 5500 50  0001 C CNN "MPN"
+F 5 "Yageo" H 3700 5500 50  0001 C CNN "Mfr."
+	1    3700 5500
+	-1   0    0    1
+$EndComp
+Wire Wire Line
+	3800 5400 3700 5400
 $Comp
 L power:GND #PWR0102
@@
 Wire Wire Line
 	6050 5200 6500 5200
+Wire Wire Line
+	3200 5200 3800 5200
+$Comp
+L power:VCC #PWR?
+U 1 1 5FA121ED
+P 3700 5600
+F 0 "#PWR?" H 3700 5450 50  0001 C CNN
+F 1 "VCC" V 3715 5727 50  0000 L CNN
+F 2 "" H 3700 5600 50  0001 C CNN
+F 3 "" H 3700 5600 50  0001 C CNN
+	1    3700 5600
+	-1   0    0    1
+$EndComp
 $EndSCHEMATC

Commit message: Add 10k MPN
Parts:
- R1: MPN (none) -> RC0603JR-0710KL
Changed lines of the file:
@@
 F 2 "Resistor_SMD:R_0603_1608Metric_Pad0.98x0.95mm_HandSolder" H 3700 5500 50  0001 C CNN
 F 3 "~" H 3700 5500 50  0001 C CNN
-F 4 "" H 3700 5500 50  0001 C CNN "MPN"
+F 4 "RC0603JR-0710KL" H 3700 5500 50  0001 C CNN "MPN"
 F 5 "Yageo" H 3700 5500 50  0001 C CNN "Mfr."
 	1    3700 5500
@@
 	3200 5200 3800 5200
 $Comp
-L power:VCC #PWR?
+L power:VCC #PWR0105
 U 1 1 5FA121ED
 P 3700 5600
-F 0 "#PWR?" H 3700 5450 50  0001 C CNN
+F 0 "#PWR0105" H 3700 5450 50  0001 C CNN
 F 1 "VCC" V 3715 5727 50  0000 L CNN
 F 2 "" H 3700 5600 50  0001 C CNN

Commit message: (bc) add sensorboard changes
Parts:
- FB1: symbol Device:Ferrite_Bead_Small -> Sensor_Board-rescue:Ferrite_Bead_Small-Device
